File: Full Boards/Main Control Unit/Main Control Unit.kicad_pcb (KiCad board)
At the start: 4 copper layers, 350 x 200 mm, 402 parts, among them J1 Optional Bond, J2 Future Use, J3 Conn_01x02_Pin, Q1 DMN6075S, Q10 DMN6075S, Q11 BSS314PE, Q12 DMN6075S, Q13 BSS314PE, Q14 DMN6075S, Q15 DMN6075S, Q2 BSS314PE, Q3 DMN6075S, Q4 BSS314PE, Q5 DMN6075S, Q6 DMN6075S, Q7 DMN6075S, Q8 DMN6075S, Q9 BSS314PE, SW1 Boot, SW2 Reset, T1 760390014, T2 760390014

Commit message: Crashed while validating custom desgin rules. Comitting to record changes to this point.
Signed-off-by: digimer <digital.mermaid@gmail.com>
Parts:
- removed DE2: L17H2110127, mr-stuff:Amphenol_L17H2110127
- added DE3: L777SDE09PA4CH4F, mr-stuff:Amphenol_L777SDE09PA4CH4F, F.Cu at (371.3, 290.3)
- added TB6: 1862411, mr-stuff:Phoenix Contact 1862411, F.Cu at (125.9, 374.3)
- added TB7: 1862411, mr-stuff:Phoenix Contact 1862411, F.Cu at (74.6, 416.8)
- added TB8: 1862411, mr-stuff:Phoenix Contact 1862411, F.Cu at (28.1, 366.8)
- moved C63 347.4 mm to (181.9, 268.1)
- moved C62 339.8 mm to (189.6, 268.1)
- moved TVS20 339.5 mm to (181.9, 274.7), turned to 90 degrees
- moved TVS33 335.7 mm to (173.5, 275.9), turned to -90 degrees
- moved TVS19 333.0 mm to (189.6, 274.7), turned to 90 degrees
- moved C61 332.3 mm to (197.3, 268.1)
- moved TVS18 326.5 mm to (197.3, 274.7), turned to 90 degrees
- moved C64 324.2 mm to (205.0, 268.1)
- moved R103 322.2 mm to (172.0, 272.9), turned to 90 degrees
- moved R102 318.7 mm to (175.0, 272.9), turned to 90 degrees
- moved C78 316.8 mm to (172.0, 261.9), turned to -90 degrees
- moved C65 316.5 mm to (212.7, 268.1)
- moved TVS21 315.8 mm to (205.0, 274.7), turned to 90 degrees
- moved C77 313.1 mm to (175.0, 261.9), turned to 90 degrees
- moved R76 312.0 mm to (178.1, 276.9), turned to 90 degrees
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Other:
- board text added: "Muirgen - Main Control Unit v1.6.4 - Prototype - 01 © The Digital Mermaid - 2026"
- board text removed: "Muirgen - Main Control Unit v1.5.4 - Prototype - 02 © The Digital Mermaid - 2026"

Commit message: v1.6.4 change log;
* 1. Refactored DA1's pinout to reduce the risk of salt tracking providing power to the "foot switch" we use to kill propulsion.

Signed-off-by: digimer <digital.mermaid@gmail.com>
Parts:
- moved C83 8.89 mm to (179.5, 294.4)
- moved DB1 8.89 mm to (225.3, 282.3)
- moved OI4 8.80 mm to (283.6, 261.6)
- moved R51 8.80 mm to (283.6, 254.5)
- moved R52 8.80 mm to (283.6, 268.7)
- moved C81 7.86 mm to (268.2, 272.5)
- moved C82 7.86 mm to (271.2, 272.5)
- moved R106 7.86 mm to (268.2, 265.3)
- moved R107 7.86 mm to (271.2, 265.3)
- moved TVS35 7.86 mm to (269.7, 268.3)
- moved C79 7.77 mm to (279.5, 272.5)
- moved C80 7.77 mm to (276.5, 272.5)
- moved R104 7.77 mm to (279.5, 265.3)
- moved R105 7.77 mm to (276.5, 265.3)
- moved TVS34 7.77 mm to (277.9, 268.3)
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Routing:
- net M5KW_GND: track 0.00 -> 85.0 mm
- net /M5KW_REGEN_DAC_PLUG: track 0.00 -> 77.3 mm
- net /M5KW_THROTTLE_DAC_PLUG: track 0.00 -> 75.3 mm
- net /M5KW_FOOT_SW_CTRL: track 0.00 -> 61.7 mm
- net M10KW_GND: track 0.00 -> 54.7 mm
- net /M5KW_HIGH_SW_CTRL: track 0.00 -> 42.3 mm
- net /M5KW_LOW_SW_CTRL: track 0.00 -> 36.9 mm
- net /M10KW_THROTTLE_DAC_PLUG: track 0.00 -> 32.4 mm
- net /M10KW_REGEN_DAC_PLUG: track 0.00 -> 28.1 mm
- net /M10KW_LOW_SW_CTRL: track 0.00 -> 24.0 mm
- net /M10KW_HIGH_SW_CTRL: track 0.00 -> 23.7 mm
- net /M10KW_FOOT_SW_CTRL: track 0.00 -> 21.6 mm
- net +3.3V: vias 0 -> 1
