File: Full Boards/Main Control Unit/Main Control Unit.kicad_pcb (KiCad board)
At the start: 4 copper layers, 350 x 200 mm, 405 parts, among them J1 Optional Bond, J2 Future Use, J3 Conn_01x02_Pin, Q1 DMN6075S, Q10 DMN6075S, Q11 BSS314PE, Q12 DMN6075S, Q13 BSS314PE, Q14 DMN6075S, Q15 DMN6075S, Q2 BSS314PE, Q3 DMN6075S, Q4 BSS314PE, Q5 DMN6075S, Q6 DMN6075S, Q7 DMN6075S, Q8 DMN6075S, Q9 BSS314PE, SW1 Boot, SW2 Reset, T1 760390014, T2 760390014

Commit message: Changes post crash.
Signed-off-by: digimer <digital.mermaid@gmail.com>
Parts:
- moved J2 19.9 mm to (283.7, 241.2), turned to 90 degrees
- moved R44 8.45 mm to (270.0, 239.2), turned to 0 degrees
Routing:
- net Net-(IOX1-P6): track 0.00 -> 18.4 mm
- net Net-(IOX1-P7): track 0.00 -> 13.3 mm
- net /MOTOR_I2C_SCL: track 0.00 -> 11.9 mm
- net /MOTOR_I2C_SDA: track 0.00 -> 10.8 mm
- net GND: track 1.49 -> 8.73 mm, vias 1 -> 2
- net Net-(IOX1-~{INT}): track 0.00 -> 4.85 mm
- net +3.3V: track 0.00 -> 1.39 mm, vias 1 -> 2

Commit message: Pre-crash save
Signed-off-by: digimer <digital.mermaid@gmail.com>
Parts:
- moved C86 90.2 mm to (390.3, 292.8), turned to -90 degrees
- moved C84 55.5 mm to (297.5, 283.7), turned to 0 degrees
- moved C85 54.3 mm to (350.5, 286.4), turned to -90 degrees
- moved ICT1 44.7 mm to (91.1, 273.7)
- moved PTC1 44.7 mm to (101.2, 274.9)
- moved TB1 44.7 mm to (115.5, 288.8)
- moved H1 35.0 mm to (165.5, 105.5)
- moved H3 35.0 mm to (434.5, 105.5)
- moved H4 35.0 mm to (165.5, 250.0)
- moved H6 35.0 mm to (435.0, 250.0)
- moved H7 35.0 mm to (165.5, 294.5)
- moved H9 35.0 mm to (434.5, 294.5)
- moved FID1 26.9 mm to (438.0, 112.0)
- moved FID2 26.6 mm to (438.0, 289.0)
- moved FID3 26.6 mm to (162.0, 289.0)
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Routing:
- net GND_SHIP: track 0.00 -> 110.9 mm
- net /THROTTLE_PORT_POT_IN_PLUG: track 0.00 -> 57.4 mm
- net /THROTTLE_STBD_POT_IN_PLUG: track 0.00 -> 52.3 mm
- net /M10KW_REGEN_POT_IN_PLUG: track 0.00 -> 49.2 mm, vias 0 -> 1
- net /M10KW_MOTOR_SELECT_IN_PLUG: track 0.00 -> 48.3 mm
- net /M5KW_REGEN_POT_IN_PLUG: track 0.00 -> 46.4 mm, vias 0 -> 1
- net /M5KW_MOTOR_SELECT_IN_PLUG: track 0.00 -> 42.5 mm, vias 0 -> 1
- net /M10KW_ENABLE_IN_PLUG: track 0.00 -> 39.8 mm, vias 0 -> 1
- net /M5KW_ENABLE_IN_PLUG: track 0.00 -> 34.8 mm, vias 0 -> 1
- net /M5KW_SPEED_HIGH_IN_PLUG: track 0.00 -> 34.6 mm
- net /M10KW_SPEED_LOW_IN_PLUG: track 0.00 -> 34.6 mm, vias 0 -> 1
- net /M5KW_SPEED_LOW_IN_PLUG: track 0.00 -> 30.9 mm, vias 0 -> 1
- net /M10KW_SPEED_HIGH_IN_PLUG: track 0.00 -> 29.3 mm
- net GND_SH25F: track 0.00 -> 10.8 mm, vias 0 -> 1
- net +3.3V_A: track 0.00 -> 9.94 mm
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Other:
- board size 350 x 200 mm -> 280 x 200 mm
