File: Full Boards/Main Control Unit/Main Control Unit.kicad_sch (KiCad schematic)
At the start: 408 parts, among them J1 Optional Bond, J2 Future Use, J3 Conn_01x02_Pin, Q1 DMN6075S, Q10 DMN6075S, Q11 BSS314PE, Q12 DMN6075S, Q13 BSS314PE, Q14 DMN6075S, Q15 DMN6075S, Q2 BSS314PE, Q3 DMN6075S, Q4 BSS314PE, Q5 DMN6075S, Q6 DMN6075S, Q7 DMN6075S, Q8 DMN6075S, Q9 BSS314PE, SW1 Boot, SW2 Reset, T1 760390014, T2 760390014

Commit message: Fixed a couple Part metadata values.
Signed-off-by: digimer <digital.mermaid@gmail.com>
Parts:
- FB1: Part Würth 782853601 -> Wurth 782853601
- LS1: value TI PCA9306IDCURQ1 -> PCA9306IDCURQ1; Part Texas Instruments PCA9306IDCURQ1 -> TI PCA9306IDCURQ1
- PTC1: Part LittelFuse AHEF100 -> Littelfuse AHEF100
- TVS1: Part LittelFuse SLD22-018 -> Littelfuse SLD22-018

Commit message: Fixed the Newhaven Display symbol, missing Part.
Signed-off-by: digimer <digital.mermaid@gmail.com>
Parts:
- LCD1: Part (none) -> Newhaven Display NHD-0216K3Z-NS(RGB)-FBW-V3
Changed lines of the file:
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@@
+			)
+		)
+		(property "Part" "Newhaven Display NHD-0216K3Z-NS(RGB)-FBW-V3"
+			(at 367.03 73.66 0)
+			(hide yes)
+			(show_name no)
+			(do_not_autoplace no)
+			(effects
+				(font
+					(size 1.27 1.27)
+				)
 			)
 		)

Commit message: Added Part to headers. Marked TPs as DNP.
Signed-off-by: digimer <digital.mermaid@gmail.com>
Parts:
- DE2: footprint mr-stuff:Amphenol_L777SDE09PA4CH4F -> mr-stuff:Amphenol L777SDE09PA4CH4F
- J1, J3: Part (none) -> Amphenol 68001-416HLF
- J2, TP1, TP10, TP13, TP14, TP2, TP3, TP4, TP5, TP6, TP8, TP9: Part (none) -> Amphenol 68001-416HLF; now not fitted

Commit message: Added a part for SWD1
Signed-off-by: digimer <digital.mermaid@gmail.com>
Parts:
- SWD1: Part (none) -> Sullins GRPB052VWVN-RC
Changed lines of the file:
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@@
 			)
 		)
-		(property "Arrow Part Number" ""
+		(property "Part" "Sullins GRPB052VWVN-RC"
 			(at 306.07 302.26 0)
 			(hide yes)
-			(show_name no)
-			(do_not_autoplace no)
-			(effects
-				(font
-					(size 1.27 1.27)
-				)
-			)
-		)
-		(property "Arrow Price/Stock" ""
-			(at 306.07 302.26 0)
-			(hide yes)
-			(show_name no)
-			(do_not_autoplace no)
-			(effects
-				(font
-					(size 1.27 1.27)
-				)
-			)
-		)
-		(property "Height" ""
-			(at 306.07 302.26 0)
-			(hide yes)
-			(show_name no)
-			(do_not_autoplace no)
-			(effects
-				(font
-					(size 1.27 1.27)
-				)
-			)
-		)
-		(property "Manufacturer_Name" ""
-			(at 306.07 302.26 0)
-			(hide yes)
-			(show_name no)
-			(do_not_autoplace no)
-			(effects
-				(font
-					(size 1.27 1.27)
-				)
-			)
-		)
-		(property "Manufacturer_Part_Number" ""
-			(at 306.07 302.26 0)
-			(hide yes)
-			(show_name no)
-			(do_not_autoplace no)
-			(effects
-				(font
-					(size 1.27 1.27)
-				)
-			)
-		)
-		(property "Mouser Part Number" ""
-			(at 306.07 302.26 0)
-			(hide yes)
-			(show_name no)
-			(do_not_autoplace no)
-			(effects
-				(font
-					(size 1.27 1.27)
-				)
-			)
-		)
-		(property "Mouser Price/Stock" ""
-			(at 306.07 302.26 0)
-			(hide yes)

Commit message: Corrected the right-hand speaker header part.
Signed-off-by: digimer <digital.mermaid@gmail.com>
Parts:
- J3: Part Amphenol 68001-416HLF -> Sullins PRPC040SBAN-M71RC
Changed lines of the file:
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@@
 			)
 		)
-		(property "Part" "Amphenol 68001-416HLF"
+		(property "Part" "Sullins PRPC040SBAN-M71RC"
 			(at 365.76 185.42 90)
 			(hide yes)
@@
 			)
 		)
-		(property "Arrow Part Number" ""
-			(at 308.61 123.19 0)
-			(hide yes)
-			(show_name no)
-			(do_not_autoplace no)
-			(effects
-				(font
-					(size 1.27 1.27)
-				)
-			)
-		)
-		(property "Arrow Price/Stock" ""
-			(at 308.61 123.19 0)
-			(hide yes)
-			(show_name no)
-			(do_not_autoplace no)
-			(effects
-				(font
-					(size 1.27 1.27)
-				)
-			)
-		)
-		(property "Height" ""
-			(at 308.61 123.19 0)
-			(hide yes)
-			(show_name no)
-			(do_not_autoplace no)
-			(effects
-				(font
-					(size 1.27 1.27)
-				)
-			)
-		)
-		(property "Manufacturer_Name" ""
-			(at 308.61 123.19 0)
-			(hide yes)
-			(show_name no)
-			(do_not_autoplace no)
-			(effects
-				(font
-					(size 1.27 1.27)
-				)
-			)
-		)
-		(property "Manufacturer_Part_Number" ""
-			(at 308.61 123.19 0)
-			(hide yes)
-			(show_name no)
-			(do_not_autoplace no)
-			(effects
-				(font
-					(size 1.27 1.27)
-				)
-			)
-		)
-		(property "Mouser Part Number" ""
-			(at 308.61 123.19 0)
-			(hide yes)
-			(show_name no)
-			(do_not_autoplace no)
-			(effects
-				(font
-					(size 1.27 1.27)
-				)
-			)
-		)
-		(property "Mouser Price/Stock" ""
-			(at 308.61 123.19 0)
-			(hide yes)
-			(show_name no)
-			(do_not_autoplace no)
-			(effects
-				(font
-					(size 1.27 1.27)
-				)
-			)
-		)
 		(pin "2"
 		)
@@
 			(hide yes)
 			(show_name no)
-			(do_not_autoplace no)
-			(effects
-				(font
-					(size 1.27 1.27)
-				)
-			)
-		)
-		(property "Arrow Part Number" ""
-			(at 307.34 181.61 0)
-			(hide yes)
-			(show_name no)
-			(do_not_autoplace no)
-			(effects
-				(font
-					(size 1.27 1.27)
-				)
-			)
-		)
-		(property "Arrow Price/Stock" ""
-			(at 307.34 181.61 0)
-			(hide yes)
-			(show_name no)
-			(do_not_autoplace no)
-			(effects
-				(font
-					(size 1.27 1.27)
-				)
-			)
-		)
-		(property "Height" ""
-			(at 307.34 181.61 0)
-			(hide yes)
-			(show_name no)
-			(do_not_autoplace no)
-			(effects
-				(font
-					(size 1.27 1.27)
-				)
-			)
-		)
-		(property "Manufacturer_Name" ""
-			(at 307.34 181.61 0)
-			(hide yes)
-			(show_name no)
-			(do_not_autoplace no)
-			(effects
-				(font
-					(size 1.27 1.27)
-				)
-			)
-		)
-		(property "Manufacturer_Part_Number" ""
-			(at 307.34 181.61 0)
-			(hide yes)
-			(show_name no)
-			(do_not_autoplace no)
-			(effects
-				(font
-					(size 1.27 1.27)
-				)
-			)
-		)
-		(property "Mouser Part Number" ""
-			(at 307.34 181.61 0)
-			(hide yes)
-			(show_name no)
-			(do_not_autoplace no)
-			(effects
-				(font
-					(size 1.27 1.27)
-				)
-			)
-		)
-		(property "Mouser Price/Stock" ""
-			(at 307.34 181.61 0)
-			(hide yes)
-			(show_name no)
