File: Full Boards/Main Control Unit/Main Control Unit.kicad_sch (KiCad schematic)
At the start: 408 parts, among them J1 Optional Bond, J2 Future Use, J3 Conn_01x02_Pin, Q1 DMN6075S, Q10 DMN6075S, Q11 BSS314PE, Q12 DMN6075S, Q13 BSS314PE, Q14 DMN6075S, Q15 DMN6075S, Q2 BSS314PE, Q3 DMN6075S, Q4 BSS314PE, Q5 DMN6075S, Q6 DMN6075S, Q7 DMN6075S, Q8 DMN6075S, Q9 BSS314PE, SW1 Boot, SW2 Reset, T1 760390014, T2 760390014

Commit message: Changed MT to Microchip to prevent ambiguity or confusion with MT-prefixed part numbers.
Signed-off-by: digimer <digital.mermaid@gmail.com>
Parts:
- DAC1: Part MT MCP4726A0T-E/CH -> Microchip MCP4726A0T-E/CH
- DAC2: Part MT MCP4726A1T-E/CH -> Microchip MCP4726A1T-E/CH
- DAC3: Part MT MCP4726A2T-E/CH -> Microchip MCP4726A2T-E/CH
- DAC4: Part MT MCP4726A3T-E/CH -> Microchip MCP4726A3T-E/CH

Commit message: Fixed a difference in the part number format for the CMC chokes.
Signed-off-by: digimer <digital.mermaid@gmail.com>
Parts:
- CMC1, CMC2, CMC3: Part TDK ACT12101012PTL00 -> TDK ACT1210-101-2P-TL00
Changed lines of the file:
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@@
 			)
 		)
-		(property "Part" "TDK ACT12101012PTL00"
-			(at 63.5 57.15 0)
-			(hide yes)
-			(show_name no)
-			(do_not_autoplace no)
-			(effects
-				(font
-					(size 1.27 1.27)
-				)
-			)
-		)
-		(property "Arrow Part Number" ""
-			(at 63.5 57.15 0)
-			(hide yes)
-			(show_name no)
-			(do_not_autoplace no)
-			(effects
-				(font
-					(size 1.27 1.27)
-				)
-			)
-		)
-		(property "Arrow Price/Stock" ""
-			(at 63.5 57.15 0)
-			(hide yes)
-			(show_name no)
-			(do_not_autoplace no)
-			(effects
-				(font
-					(size 1.27 1.27)
-				)
-			)
-		)
-		(property "Height" ""
-			(at 63.5 57.15 0)
-			(hide yes)
-			(show_name no)
-			(do_not_autoplace no)
-			(effects
-				(font
-					(size 1.27 1.27)
-				)
-			)
-		)
-		(property "Manufacturer_Name" ""
-			(at 63.5 57.15 0)
-			(hide yes)
-			(show_name no)
-			(do_not_autoplace no)
-			(effects
-				(font
-					(size 1.27 1.27)
-				)
-			)
-		)
-		(property "Manufacturer_Part_Number" ""
-			(at 63.5 57.15 0)
-			(hide yes)
-			(show_name no)
-			(do_not_autoplace no)
-			(effects
-				(font
-					(size 1.27 1.27)
-				)
-			)
-		)
-		(property "Mouser Part Number" ""
-			(at 63.5 57.15 0)
-			(hide yes)
-			(show_name no)
-			(do_not_autoplace no)
-			(effects
-				(font
-					(size 1.27 1.27)
-				)
-			)
-		)
-		(property "Mouser Price/Stock" ""
+		(property "Part" "TDK ACT1210-101-2P-TL00"
 			(at 63.5 57.15 0)
 			(hide yes)
@@
 			)
 		)
-		(property "Part" "TDK ACT12101012PTL00"
-			(at 144.78 322.58 0)
-			(hide yes)
-			(show_name no)
-			(do_not_autoplace no)
-			(effects
-				(font
-					(size 1.27 1.27)
-				)
-			)
-		)
-		(property "Arrow Part Number" ""
-			(at 144.78 322.58 0)
-			(hide yes)
-			(show_name no)
-			(do_not_autoplace no)
-			(effects
-				(font
-					(size 1.27 1.27)
-				)
-			)
-		)
-		(property "Arrow Price/Stock" ""
-			(at 144.78 322.58 0)
-			(hide yes)
-			(show_name no)
-			(do_not_autoplace no)
-			(effects
-				(font
-					(size 1.27 1.27)
-				)
-			)
-		)
-		(property "Height" ""
-			(at 144.78 322.58 0)
-			(hide yes)
-			(show_name no)
-			(do_not_autoplace no)
-			(effects
-				(font
-					(size 1.27 1.27)
-				)
-			)
-		)
-		(property "Manufacturer_Name" ""
-			(at 144.78 322.58 0)
-			(hide yes)
-			(show_name no)
-			(do_not_autoplace no)
-			(effects
-				(font
-					(size 1.27 1.27)
-				)
-			)
-		)
-		(property "Manufacturer_Part_Number" ""
-			(at 144.78 322.58 0)
-			(hide yes)
-			(show_name no)
-			(do_not_autoplace no)
-			(effects
-				(font
-					(size 1.27 1.27)
-				)
-			)
-		)
-		(property "Mouser Part Number" ""
-			(at 144.78 322.58 0)
-			(hide yes)
-			(show_name no)
-			(do_not_autoplace no)
-			(effects
-				(font
-					(size 1.27 1.27)
-				)
-			)
-		)
-		(property "Mouser Price/Stock" ""
+		(property "Part" "TDK ACT1210-101-2P-TL00"
 			(at 144.78 322.58 0)
 			(hide yes)
@@
 			)
 		)
-		(property "Part" "TDK ACT12101012PTL00"
-			(at 143.51 238.76 0)
-			(hide yes)
-			(show_name no)
-			(do_not_autoplace no)
-			(effects
-				(font
-					(size 1.27 1.27)
-				)
-			)
-		)
-		(property "Arrow Part Number" ""
-			(at 143.51 238.76 0)
-			(hide yes)
-			(show_name no)
-			(do_not_autoplace no)
-			(effects
-				(font
-					(size 1.27 1.27)
-				)
-			)
-		)
-		(property "Arrow Price/Stock" ""
-			(at 143.51 238.76 0)
-			(hide yes)
-			(show_name no)
-			(do_not_autoplace no)
-			(effects
-				(font
-					(size 1.27 1.27)
-				)
-			)
-		)
-		(property "Height" ""
-			(at 143.51 238.76 0)
-			(hide yes)
-			(show_name no)
-			(do_not_autoplace no)
-			(effects
-				(font
-					(size 1.27 1.27)
-				)
-			)
-		)
-		(property "Manufacturer_Name" ""
-			(at 143.51 238.76 0)
-			(hide yes)
-			(show_name no)
-			(do_not_autoplace no)
-			(effects
-				(font
-					(size 1.27 1.27)
-				)
-			)
-		)
-		(property "Manufacturer_Part_Number" ""
-			(at 143.51 238.76 0)
-			(hide yes)
-			(show_name no)
-			(do_not_autoplace no)
-			(effects
-				(font
-					(size 1.27 1.27)
-				)
-			)
-		)
-		(property "Mouser Part Number" ""
-			(at 143.51 238.76 0)
-			(hide yes)
-			(show_name no)
-			(do_not_autoplace no)
-			(effects
-				(font
-					(size 1.27 1.27)
-				)
-			)
-		)
-		(property "Mouser Price/Stock" ""
+		(property "Part" "TDK ACT1210-101-2P-TL00"
 			(at 143.51 238.76 0)
 			(hide yes)

Commit message: Changed the TDK CGA5L1X7R1E106K160DC to CGA5L1X7R1H106K160AE.
Signed-off-by: digimer <digital.mermaid@gmail.com>
Parts:
- C39, C42, C43, C46, C7: Part TDK CGA5L1X7R1E106K160DC -> TDK CGA5L1X7R1H106K160AE

Commit message: Removed unused metadata fields from the MCU schematic.
Signed-off-by: digimer <digital.mermaid@gmail.com>
Parts:
- RL2: MANUFACTURER TE Connectivity -> (none)

Commit message: More metadata cleanup.
Signed-off-by: digimer <digital.mermaid@gmail.com>
Parts:
- DAC1, DAC2, DAC3, DAC4: Note Part number suffix denotes I2C address (MCP4726A0T-E/CH = 0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 -> (none)
