File: Full Boards/USB-C PD x2/USB-C PD x2.kicad_sch (KiCad schematic)
At the start: 160 parts, among them J1 Conn_02x05_Odd_Even, J2 Conn_01x05_Pin

Commit message: Updated the symbols and footprints for replaced foot prints.
Signed-off-by: digimer <digital.mermaid@gmail.com>
Parts:
- TB1, TB2: value Keystone Electronics 7799 -> 7799; Part (none) -> Keystone 7799
- TVS1: footprint mr-stuff:DIOAD4425W136L885D885 -> mr-stuff:Littelfuse SDL; symbol mr-parts:SLD15-018 -> mr-parts:Littelfuse SLD18-018; Part (none) -> Littelfuse SLD18-018
Connections:
- net +BATT: no longer TB1.2, TB1.3, TB1.4, TB1.5, TB1.6
- net -BATT: no longer TB2.2, TB2.3, TB2.4, TB2.5, TB2.6
Other:
- moved on the sheet: C1, C2, C3, C4, NT10, NT9, PMIC1, R1, R2, R3, R4, TVS1

Commit message: Started adding 'Part' metadata, but may not finish for this board.
Signed-off-by: digimer <digital.mermaid@gmail.com>
Parts:
- C3, C4: MANUFACTURER Panasonic -> (none); MAXIMUM_PACKAGE_HEIGHT 12.8mm -> (none); PARTREV 30-Sep-20 -> (none); Part (none) -> Panasonic EEH-ZU1V331V; STANDARD Manufacturer Recommendations -> (none)
- F1: Part (none) -> Littelfuse 178.6165.0001
- HS1: value Nexperia PSMN1R4-40YLDX -> PSMN1R4-40YLDX; Part (none) -> Nexperia PSMN1R4-40YLDX
- ID1: Arrow Part Number IAUC120N04S6L008ATMA1 -> (none); Arrow Price/Stock https://www.arrow.com/en/products/iauc120n04s6l008atma1/inf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 -> (none); Height 1.1 -> (none); Manufacturer_Name Infineon -> (none); Manufacturer_Part_Number IAUC120N04S6L008ATMA1 -> (none); Mouser Part Number 726-IAUC120N04S6L008 -> (none); Mouser Price/Stock https://www.mouser.co.uk/ProductDetail/Infineon-Technologie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 -> (none); Part (none) -> Infineon IAUC120N04S6L008ATMA1
- PMIC1: MANUFACTURER Analog Devices -> (none); MAXIMUM_PACKAGE_HEIGHT 1.1 mm -> (none); PARTREV F -> (none); Part (none) -> ADI LTC4368; STANDARD IPC 7351B -> (none)
- TB1, TB2: MANUFACTURER Keystone Electronics -> (none); MAXIMUM_PACKAGE_HEIGHT 6.35 mm -> (none); PARTREV C -> (none); STANDARD Manufacturer Recommendations -> (none)
- TVS1: Manufacturer_Name LITTELFUSE -> (none)

Commit message: Created new Infineon IAUC120N04S6L008ATMA1 and updated ID1 to use it. No substantive changes, but makes the footprint match the real part number.
Signed-off-by: digimer <digital.mermaid@gmail.com>
Parts:
- ID1: value Infineon IAUC120N04S6L008ATMA1 -> IAUC120N04S6L008ATMA1; footprint mr-stuff:Infineon IAUC120N06S5N017ATMA1 -> mr-stuff:Infineon IAUC120N04S6L008ATMA1
Changed lines of the file:
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@@
 			)
 		)
-		(property "Value" "Infineon IAUC120N04S6L008ATMA1"
+		(property "Value" "IAUC120N04S6L008ATMA1"
 			(at 109.474 24.384 0)
 			(hide yes)
@@
 			)
 		)
-		(property "Footprint" "mr-stuff:Infineon IAUC120N06S5N017ATMA1"
+		(property "Footprint" "mr-stuff:Infineon IAUC120N04S6L008ATMA1"
 			(at 76.2 -58.09 0)
 			(hide yes)

Commit message: Cleaned up symbol metadata for R1, Wurth 560112132040.
Signed-off-by: digimer <digital.mermaid@gmail.com>
Parts:
- R1: Part (none) -> Wurth 560112132040
Changed lines of the file:
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@@
 			)
 		)
-		(property "Description" "560112132040 1% 0.25W"
+		(property "Description" "1.5 MOhms ±1% 0.25W, 1/4W Chip Resistor 1206 (3216 Metric) Anti-Sulfur Thick Film"
 			(at 27.94 44.45 0)
 			(hide yes)
 			(show_name no)
+			(do_not_autoplace no)
+			(effects
+				(font
+					(size 1.27 1.27)
+				)
+			)
+		)
+		(property "Part" "Wurth 560112132040"
+			(at 27.94 44.45 90)
+			(hide yes)
+			(show_name no)

Commit message: Bumped the Infineon CYPD7272 footprint to use 0.3mm instead of 0.2mm thermal vias.
Signed-off-by: digimer <digital.mermaid@gmail.com>
Parts:
- PD1: footprint Package_DFN_QFN:QFN-68-1EP_8x8mm_P0.4mm_EP5.2x5.2mm_ThermalVias -> mr-stuff:Infineon CYPD727x
Changed lines of the file:
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@@
 			)
 		)
-		(property "Footprint" "Package_DFN_QFN:QFN-68-1EP_8x8mm_P0.4mm_EP5.2x5.2mm_ThermalVias"
+		(property "Footprint" "mr-stuff:Infineon CYPD727x"
 			(at 339.344 156.718 0)
 			(hide yes)

Commit message: Changed the current sense resistor on the PMIC to 1.5mR 6W from 2mR 5W to help increase the trip margin.
Signed-off-by: digimer <digital.mermaid@gmail.com>
Parts:
- R4: value 2mR -> 1.5mR; footprint mr-stuff:Vishay WSLP -> mr-stuff:Vishay WSLF2512; Part Yageo PK2512FKF570R002L -> Vishay WSLF25121L500FEA
Other:
- note added: "Configs: ch0: A, ch1: A - R25 = 0R ch0: A, ch1: B - R25 = 4.7KR ch0: B, ch1: A - R25 = 10KR ch0: B, ch1: B - R25 = DNP A: 5V, 5A rapid response, buck only (Raspberry Pi) B: Slower response, full range (General Purpose) See compensation network notes"
- note removed: "Configs: ch0: A, ch1: A - R20 = 0R ch0: A, ch1: B - R20 = 4.7KR ch0: B, ch1: A - R20 = 10KR ch0: B, ch1: B - R20 = DNP A: 5V, 5A rapid response, buck only (Raspberry Pi) B: Slower response, full range (General Purpose) See compensation network notes"
Changed lines of the file:
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@@
 		)
 	)
-	(text "Configs:\nch0: A, ch1: A - R20 = 0R\nch0: A, ch1: B - R20 = 4.7KR\nch0: B, ch1: A - R20 = 10KR\nch0: B, ch1: B - R20 = DNP\n\nA: 5V, 5A rapid response, buck only (Raspberry Pi)\nB: Slower response, full range (General Purpose)\n\nSee compensation network notes"
+	(text "Configs:\nch0: A, ch1: A - R25 = 0R\nch0: A, ch1: B - R25 = 4.7KR\nch0: B, ch1: A - R25 = 10KR\nch0: B, ch1: B - R25 = DNP\n\nA: 5V, 5A rapid response, buck only (Raspberry Pi)\nB: Slower response, full range (General Purpose)\n\nSee compensation network notes"
 		(exclude_from_sim no)
 		(at 291.846 200.914 0)
@@
 			)
 		)
-		(property "Value" "2mR"
+		(property "Value" "1.5mR"
 			(at 88.646 68.58 90)
 			(show_name no)
@@
 			)
 		)
-		(property "Footprint" "mr-stuff:Vishay WSLP"
+		(property "Footprint" "mr-stuff:Vishay WSLF2512"
 			(at 84.582 68.58 90)
 			(hide yes)
@@
 			)
 		)
-		(property "Datasheet" "https://yageogroup.com/content/datasheet/asset/file/PYU-PK_51_ROHS_L"
+		(property "Datasheet" "https://www.vishay.com/docs/30193/wslf.pdf"
 			(at 86.36 68.58 0)
 			(hide yes)
@@
 			)
 		)
-		(property "Description" "RES 0.002 OHM 1% 5W 2512"
+		(property "Description" "RES 0.0015 OHM 1% 6W 2512"
 			(at 86.36 68.58 0)
 			(hide yes)
@@
 			)
 		)
-		(property "Part" "Yageo PK2512FKF570R002L"
+		(property "Part" "Vishay WSLF25121L500FEA"
 			(at 86.36 68.58 90)
 			(hide yes)

Commit message: Removed C34 (1uF on CLPD7272 VCCD, pin 62). As per the datasheet; "1.8-V core LDO output. Connect a 0.1-µF bypass capacitor to ground. Do not connect anything else to this pin."
Signed-off-by: digimer <digital.mermaid@gmail.com>
Parts:
- removed C34: 1μF, mr-stuff:Kyocera AVX 08051A0R8CAT2A, symbol Device:C
Other:
- moved on the sheet: C35, TP11
Changed lines of the file:
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@@
 	)
 	(junction
-		(at 276.86 90.17)
-		(diameter 0)
-		(color 0 0 0 0)
-	)
-	(junction
 		(at 60.96 160.02)
 		(diameter 0)
@@
 	)
 	(junction
+		(at 283.21 82.55)
+		(diameter 0)
+		(color 0 0 0 0)
+	)
+	(junction
 		(at 298.45 87.63)
 		(diameter 0)
@@
 	)
 	(junction
-		(at 284.48 82.55)
-		(diameter 0)
-		(color 0 0 0 0)
-	)
-	(junction
 		(at 25.4 171.45)
 		(diameter 0)
@@
 	)
 	(junction
-		(at 276.86 82.55)
-		(diameter 0)
-		(color 0 0 0 0)
-	)
-	(junction
 		(at 314.96 60.96)
 		(diameter 0)
@@
 	(wire
 		(pts
+			(xy 283.21 82.55) (xy 298.45 82.55)
+		)
+		(stroke
+			(width 0)
+			(type default)
+		)
+	)
+	(wire
+		(pts
 			(xy 227.33 17.78) (xy 223.52 17.78)
 		)
@@
 	(wire
 		(pts
-			(xy 276.86 82.55) (xy 284.48 82.55)
+			(xy 275.59 82.55) (xy 283.21 82.55)
 		)
 		(stroke
@@
 	(wire
 		(pts
-			(xy 260.35 82.55) (xy 260.35 81.28)
+			(xy 275.59 90.17) (xy 275.59 82.55)
 		)
 		(stroke
@@
 	(wire
 		(pts
-			(xy 276.86 90.17) (xy 270.51 90.17)
+			(xy 283.21 91.44) (xy 283.21 90.17)
 		)
 		(stroke
@@
 	(wire
 		(pts
-			(xy 260.35 82.55) (xy 276.86 82.55)
-		)
-		(stroke
-			(width 0)
-			(type default)
-		)
-	)
-	(wire
-		(pts
 			(xy 81.28 58.42) (xy 76.2 58.42)
 		)
@@
 	(wire
 		(pts
-			(xy 284.48 82.55) (xy 298.45 82.55)
-		)
-		(stroke
-			(width 0)
-			(type default)
-		)
-	)
-	(wire
-		(pts
 			(xy 295.91 100.33) (xy 298.45 100.33)
 		)
@@
 	(wire
 		(pts
+			(xy 275.59 90.17) (xy 271.78 90.17)
+		)
+		(stroke
+			(width 0)
+			(type default)
+		)
+	)
+	(wire
+		(pts
 			(xy 295.91 113.03) (xy 298.45 113.03)
 		)
@@
 	(wire
 		(pts
-			(xy 284.48 90.17) (xy 276.86 90.17)
-		)
-		(stroke
-			(width 0)
-			(type default)
-		)
-	)
-	(wire
-		(pts
 			(xy 91.44 260.35) (xy 91.44 262.89)
 		)
@@
 	)
 	(symbol
-		(lib_id "Device:C")
-		(at 276.86 86.36 180)
-		(unit 1)
-		(body_style 1)
-		(exclude_from_sim no)
-		(in_bom yes)
-		(on_board yes)
-		(in_pos_files yes)
-		(dnp no)
-		(property "Reference" "C34"
-			(at 275.844 84.074 0)
-			(show_name no)
-			(do_not_autoplace no)
-			(effects
-				(font
-					(size 1.27 1.27)
-				)
-				(justify left)
-			)
-		)
-		(property "Value" "1μF"
-			(at 275.59 88.9 0)
-			(show_name no)
-			(do_not_autoplace no)
-			(effects
-				(font
-					(size 1.27 1.27)
-				)
-				(justify left)
-			)
-		)
-		(property "Footprint" "mr-stuff:Kyocera AVX 08051A0R8CAT2A"
-			(at 275.8948 82.55 0)
-			(hide yes)
-			(show_name no)
-			(do_not_autoplace no)
-			(effects
-				(font
-					(size 1.27 1.27)
-				)
-			)
-		)
-		(property "Datasheet" "https://mm.digikey.com/Volume0/opasdata/d220001/medias/docus/6397/AutoMLCC-2952695-DS.pdf"
-			(at 276.86 86.36 0)
-			(hide yes)
-			(show_name no)
-			(do_not_autoplace no)
-			(effects
-				(font
-					(size 1.27 1.27)
-				)
-			)
-		)
-		(property "Description" "Unpolarized capacitor"
-			(at 276.86 86.36 0)
-			(hide yes)
-			(show_name no)
-			(do_not_autoplace no)
-			(effects
-				(font
-					(size 1.27 1.27)
-				)
-			)
-		)
-		(pin "2"
-		)
-		(pin "1"
-		)
-		(instances
-			(project "USB-C PD x2"
-				(path "/5152699f-c39d-4ac5-8e07-bebed783643b"
-					(reference "C34")
-					(unit 1)
-				)
-			)
-		)
-	)
-	(symbol
 		(lib_id "Device:L")
 		(at 157.48 171.45 90)
@@
 	(symbol
 		(lib_id "Connector:TestPoint")
-		(at 260.35 81.28 0)
+		(at 271.78 90.17 0)
 		(unit 1)
 		(body_style 1)
@@
 		(dnp no)
 		(property "Reference" "TP11"
-			(at 258.826 76.2 0)
+			(at 269.748 85.09 0)
 			(show_name no)
 			(do_not_autoplace no)
@@
 		)
 		(property "Value" "TestPoint"
-			(at 262.89 79.2479 0)
+			(at 274.32 88.1379 0)
 			(hide yes)
 			(show_name no)
@@
 		)
 		(property "Footprint" "Connector_PinHeader_1.00mm:PinHeader_1x01_P1.00mm_Vertical"
-			(at 265.43 81.28 0)
+			(at 276.86 90.17 0)
 			(hide yes)
 			(show_name no)
@@
 		)
 		(property "Datasheet" ""
-			(at 265.43 81.28 0)
+			(at 276.86 90.17 0)
 			(hide yes)
 			(show_name no)
@@
 		)
 		(property "Description" "test point"
-			(at 260.35 81.28 0)
+			(at 271.78 90.17 0)
 			(hide yes)
 			(show_name no)
@@
 	(symbol
 		(lib_id "power:-BATT")
-		(at 270.51 90.17 180)
+		(at 283.21 91.44 180)
 		(unit 1)
 		(body_style 1)
@@
 		(dnp no)
 		(property "Reference" "#PWR062"
-			(at 270.51 86.36 0)
+			(at 283.21 87.63 0)
 			(hide yes)
 			(show_name no)
@@
 		)
 		(property "Value" "-BATT"
-			(at 270.51 93.98 0)
+			(at 283.21 95.25 0)
 			(show_name no)
 			(do_not_autoplace no)
@@
 		)
 		(property "Footprint" ""
-			(at 270.51 90.17 0)
+			(at 283.21 91.44 0)
 			(hide yes)
 			(show_name no)
@@
 		)
 		(property "Datasheet" ""
-			(at 270.51 90.17 0)
+			(at 283.21 91.44 0)
 			(hide yes)
 			(show_name no)
@@
 		)
 		(property "Description" "Power symbol creates a global label with name \"-BATT\""
-			(at 270.51 90.17 0)
+			(at 283.21 91.44 0)
 			(hide yes)
 			(show_name no)
@@
 	(symbol
 		(lib_id "Device:C")
-		(at 284.48 86.36 0)
+		(at 283.21 86.36 0)
 		(unit 1)
 		(body_style 1)
@@
 		(dnp no)
 		(property "Reference" "C35"
-			(at 280.162 84.074 0)
+			(at 278.892 84.074 0)
 			(show_name no)
 			(do_not_autoplace no)
@@
 		)
 		(property "Value" "0.1μF"
-			(at 278.384 88.9 0)
+			(at 277.114 88.9 0)
 			(show_name no)
 			(do_not_autoplace no)
@@
 		)
 		(property "Footprint" "mr-stuff:Kyocera AVX 08051A0R8CAT2A"
-			(at 285.4452 90.17 0)
+			(at 284.1752 90.17 0)
 			(hide yes)
 			(show_name no)
@@
 		)
 		(property "Datasheet" "https://datasheets.kyocera-avx.com/FlexitermMLCC.pdf"
-			(at 284.48 86.36 0)
+			(at 283.21 86.36 0)
 			(hide yes)
 			(show_name no)
@@
 		)
 		(property "Description" "Unpolarized capacitor"
-			(at 284.48 86.36 0)
+			(at 283.21 86.36 0)
 			(hide yes)
 			(show_name no)
