File: Full Boards/USB-C PD x2/USB-C PD x2.kicad_sch (KiCad schematic)
At the start: 160 parts, among them J1 Conn_02x05_Odd_Even, J2 Conn_01x05_Pin

Commit message: Fixed the Value field for the TVS diodes.
Signed-off-by: digimer <digital.mermaid@gmail.com>
Parts:
- TVS2, TVS3, TVS4, TVS5, TVS6, TVS7, TVS8, TVS9: value Nexperia PESD24 -> MMBZ27VAL,215
Changed lines of the file:
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@@
 			)
 		)
-		(property "Value" "Nexperia PESD24"
+		(property "Value" "MMBZ27VAL,215"
 			(at 205.994 230.378 0)
 			(hide yes)
@@
 			)
 		)
-		(property "Value" "Nexperia PESD24"
+		(property "Value" "MMBZ27VAL,215"
 			(at 92.964 230.378 0)
 			(hide yes)
@@
 			)
 		)
-		(property "Value" "Nexperia PESD24"
+		(property "Value" "MMBZ27VAL,215"
 			(at 115.824 230.378 0)
 			(hide yes)
@@
 			)
 		)
-		(property "Value" "Nexperia PESD24"
+		(property "Value" "MMBZ27VAL,215"
 			(at 205.994 244.348 0)
 			(hide yes)
@@
 			)
 		)
-		(property "Value" "Nexperia PESD24"
+		(property "Value" "MMBZ27VAL,215"
 			(at 92.964 244.348 0)
 			(hide yes)
@@
 			)
 		)
-		(property "Value" "Nexperia PESD24"
+		(property "Value" "MMBZ27VAL,215"
 			(at 228.854 244.348 0)
 			(hide yes)
@@
 			)
 		)
-		(property "Value" "Nexperia PESD24"
+		(property "Value" "MMBZ27VAL,215"
 			(at 228.854 230.378 0)
 			(hide yes)
@@
 			)
 		)
-		(property "Value" "Nexperia PESD24"
+		(property "Value" "MMBZ27VAL,215"
 			(at 115.824 244.348 0)
 			(hide yes)

Commit message: Removed the packaging component of the LED part numbers.
Signed-off-by: digimer <digital.mermaid@gmail.com>
Parts:
- LED1, LED2, LED3, LED4: Part ams OSRAM LS Q976.01-N1Q2-1-20-R18 -> ams OSRAM LS Q976.01-N1Q2-1
Changed lines of the file:
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@@
 			)
 		)
-		(property "Part" "ams OSRAM LS Q976.01-N1Q2-1-20-R18"
+		(property "Part" "ams OSRAM LS Q976.01-N1Q2-1"
 			(at 270.51 201.93 0)
 			(hide yes)
@@
 			)
 		)
-		(property "Part" "ams OSRAM LS Q976.01-N1Q2-1-20-R18"
+		(property "Part" "ams OSRAM LS Q976.01-N1Q2-1"
 			(at 269.24 226.06 0)
 			(hide yes)
@@
 			)
 		)
-		(property "Part" "ams OSRAM LS Q976.01-N1Q2-1-20-R18"
+		(property "Part" "ams OSRAM LS Q976.01-N1Q2-1"
 			(at 269.24 210.82 0)
 			(hide yes)
@@
 			)
 		)
-		(property "Part" "ams OSRAM LS Q976.01-N1Q2-1-20-R18"
+		(property "Part" "ams OSRAM LS Q976.01-N1Q2-1"
 			(at 269.24 218.44 0)
 			(hide yes)

Commit message: Sync'ed the USB-C PD PCB to the schematic.
Removed test points from the 1212 kicad schematic, as it was unused.

Signed-off-by: digimer <digital.mermaid@gmail.com>
Parts:
- C_OUT_1_0, C_OUT_1_1, C_OUT_2_0, C_OUT_2_1, C_OUT_3_0, C_OUT_3_1: MANUFACTURER Panasonic -> (none); MAXIMUM_PACKAGE_HEIGHT 12.8mm -> (none); PARTREV 30-Sep-20 -> (none); STANDARD Manufacturer Recommendations -> (none)
