File: Full Boards/USB-C PD x2/USB-C PD x2.kicad_pcb (KiCad board)
At the start: 4 copper layers, 96 x 136 mm, 161 parts, among them J1 Conn_02x05_Odd_Even, J2 Conn_01x05_Pin

Commit message: Sync'ed the USB-C PD PCB to the schematic.
Removed test points from the 1212 kicad schematic, as it was unused.

Signed-off-by: digimer <digital.mermaid@gmail.com>
Parts:
- C1: value 0.22μF -> 0.22uF
- C10, C11, C12, C14, C15, C18, C19, C20, C36, C6, C7: value 10μF -> 10uF
- C13, C17, C23, C26, C27, C28, C29, C30, C31, C33, C35, C37, C39, C40, C41, C42, C45, C46, C47, C48, C49, C5, C9: value 0.1μF -> 0.1uF
- C16, C8: value 68µF -> 68uF
- C2: value 3.3nF -> 3300pF
- C3, C4, C_OUT_1_0, C_OUT_1_1, C_OUT_2_0, C_OUT_2_1, C_OUT_3_0, C_OUT_3_1: value 330 µF -> 330 uF
- C32, C38, C43, C44: value 1μF -> 1uF
- Cc1: value 10nF -> 0.01uF
- Cc2: value 470nF -> 0.470uF
- Cp2: value 1.5nF -> 1500pF
- LED1, LED2, LED3, LED4: footprint LED_SMD:LED_0603_1608Metric -> mr-stuff:ams OSRAM LS Q976.01
- PD1: footprint mr-stuff:Infineon CYPD727x -> Package_DFN_QFN:QFN-68-1EP_8x8mm_P0.4mm_EP5.2x5.2mm_ThermalVias
- TVS2, TVS3, TVS4, TVS5, TVS6, TVS7, TVS8, TVS9: value Nexperia PESD24 -> MMBZ27VAL,215; footprint mr-stuff:Nexperia PESD24 -> mr-stuff:Nexperia MMBZ27
Other:
- board text added: "USB-C PD Dual Channel 100w v1.3.3 - Prototype - 01 © The Digital Mermaid - 2026"
- board text removed: "USB-C PD Dual Channel 100w v1.3.2 - Prototype - 01 © The Digital Mermaid - 2026"
