File: Full Boards/Masthead Controller/Masthead Controller.kicad_sch (KiCad schematic)
At the start: 167 parts, among them Q1 2N7002, Q2 2N7002, SW1 SW_MEC_5G, SW2 SW_MEC_5G

Commit message: Updated the metadata for the 300kR resistors on the UVLO voltage divider.
Signed-off-by: digimer <digital.mermaid@gmail.com>
Parts:
- R21, R30: Part (none) -> Yageo AE1206BR-07300KL
Changed lines of the file:
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@@
 			)
 		)
-		(property "Datasheet" ""
+		(property "Datasheet" "https://yageogroup.com/content/datasheet/asset/file/PYU-AE_51_ROHS_L"
 			(at 139.7 106.68 0)
 			(hide yes)
@@
 			)
 		)
-		(property "Description" "Resistor"
+		(property "Description" "300 kOhms ±0.1% 0.333W, 1/3W Chip Resistor 1206 (3216 Metric) Automotive AEC-Q200 Thick Film"
 			(at 139.7 106.68 0)
 			(hide yes)
@@
 			)
 		)
+		(property "Part" "Yageo AE1206BR-07300KL"
+			(at 139.7 106.68 90)
+			(hide yes)
+			(show_name no)
+			(do_not_autoplace no)
+			(effects
+				(font
+					(size 1.27 1.27)
+				)
+			)
+		)
 		(pin "2"
 		)
@@
 			)
 		)
-		(property "Datasheet" ""
+		(property "Datasheet" "https://yageogroup.com/content/datasheet/asset/file/PYU-AE_51_ROHS_L"
 			(at 140.97 35.56 0)
 			(hide yes)
@@
 			)
 		)
-		(property "Description" "Resistor"
+		(property "Description" "300 kOhms ±0.1% 0.333W, 1/3W Chip Resistor 1206 (3216 Metric) Automotive AEC-Q200 Thick Film"
 			(at 140.97 35.56 0)
 			(hide yes)
 			(show_name no)
+			(do_not_autoplace no)
+			(effects
+				(font
+					(size 1.27 1.27)
+				)
+			)
+		)
+		(property "Part" "Yageo AE1206BR-07300KL"
+			(at 140.97 35.56 90)
+			(hide yes)
+			(show_name no)

Commit message: Fixed the metadata on R37 60.4 kOhm resistor.
Signed-off-by: digimer <digital.mermaid@gmail.com>
Parts:
- R37: Part (none) -> Vishay RCA080560K4FKEA
Changed lines of the file:
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@@
 			)
 		)
-		(property "Datasheet" ""
+		(property "Datasheet" "https://www.vishay.com/docs/20037/rcae3.pdf"
 			(at 208.28 125.73 0)
 			(hide yes)
@@
 			)
 		)
-		(property "Description" "Resistor"
+		(property "Description" "60.4 kOhms ±1% 0.125W, 1/8W Chip Resistor 0805 (2012 Metric) Anti-Sulfur, Automotive AEC-Q200 Thick Film"
 			(at 208.28 125.73 0)
 			(hide yes)
 			(show_name no)
+			(do_not_autoplace no)
+			(effects
+				(font
+					(size 1.27 1.27)
+				)
+			)
+		)
+		(property "Part" "Vishay RCA080560K4FKEA"
+			(at 208.28 125.73 90)
+			(hide yes)
+			(show_name no)

Commit message: Fixed reversed pin assignements on the Diodes Inc DMTH6010SK3Q.
Signed-off-by: digimer <digital.mermaid@gmail.com>
Parts:
- NFET1, NFET2: Part (none) -> Diodes Inc. DMTH6010SK3Q-13
Connections:
- net +24V_ISO: now also NFET1.3 (S), NFET2.3 (S); no longer NFET1.2, NFET2.2
- net at C12.2, EF2.1 (IN), EF2.2 (IN)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: now also NFET2.2 (D); no longer NFET2.3
- net at C10.2, EF1.1 (IN), EF1.2 (IN)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: now also NFET1.2 (D); no longer NFET1.3
Changed lines of the file:
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@@
 	)
 	(junction
+		(at 158.75 105.41)
+		(diameter 0)
+		(color 0 0 0 0)
+	)
+	(junction
 		(at 389.89 59.69)
 		(diameter 0)
@@
 	)
 	(junction
-		(at 158.75 105.41)
-		(diameter 0)
-		(color 0 0 0 0)
-	)
-	(junction
 		(at 511.81 119.38)
 		(diameter 0)
@@
 	(wire
 		(pts
-			(xy 158.75 105.41) (xy 161.29 105.41)
-		)
-		(stroke
-			(width 0)
-			(type default)
-		)
-	)
-	(wire
-		(pts
 			(xy 326.39 119.38) (xy 327.66 119.38)
 		)
@@
 	(wire
 		(pts
+			(xy 158.75 105.41) (xy 161.29 105.41)
+		)
+		(stroke
+			(width 0)
+			(type default)
+		)
+	)
+	(wire
+		(pts
 			(xy 67.31 60.96) (xy 76.2 60.96)
 		)
@@
 	)
 	(symbol
+		(lib_name "Diodes Inc DMTH6010SK3Q_1")
+		(lib_id "mr-parts:Diodes Inc DMTH6010SK3Q")
+		(at 158.75 100.33 270)
+		(mirror x)
+		(unit 1)
+		(body_style 1)
+		(exclude_from_sim no)
+		(in_bom yes)
+		(on_board yes)
+		(in_pos_files yes)
+		(dnp no)
+		(property "Reference" "NFET2"
+			(at 155.956 92.964 90)
+			(show_name no)
+			(do_not_autoplace no)
+			(effects
+				(font
+					(size 1.27 1.27)
+				)
+				(justify left)
+			)
+		)
+		(property "Value" "DMTH6010SK3Q"
+			(at 150.876 95.504 90)
+			(show_name no)
+			(do_not_autoplace no)
+			(effects
+				(font
+					(size 1.27 1.27)
+				)
+				(justify left)
+			)
+		)
+		(property "Footprint" "mr-stuff:Diodes Inc DMTH6010SK3Q"
+			(at 158.75 100.33 0)
+			(hide yes)
+			(show_name no)
+			(do_not_autoplace no)
+			(effects
+				(font
+					(size 1.27 1.27)
+				)
+			)
+		)
+		(property "Datasheet" "https://www.diodes.com/datasheet/download/DMTH6010SK3Q.pdf"
+			(at 145.796 100.33 0)
+			(hide yes)
+			(show_name no)
+			(do_not_autoplace no)
+			(effects
+				(font
+					(size 1.27 1.27)
+				)
+			)
+		)
+		(property "Description" "N-Channel 60 V 16.3A (Ta), 70A (Tc) 3.1W (Ta) Surface Mount TO-252-3"
+			(at 158.75 100.33 0)
+			(hide yes)
+			(show_name no)
+			(do_not_autoplace no)
+			(effects
+				(font
+					(size 1.27 1.27)
+				)
+			)
+		)
+		(property "Part" "Diodes Inc. DMTH6010SK3Q-13"
+			(at 158.75 100.33 90)
+			(hide yes)
+			(show_name no)
+			(do_not_autoplace no)
+			(effects
+				(font
+					(size 1.27 1.27)
+				)
+			)
+		)
+		(pin "3"
+		)
+		(pin "2"
+		)
+		(pin "1"
+		)
+		(instances
+			(project "Masthead Controller"
+				(path "/2a070473-cb6e-4844-8f2a-5ea6a35ddb49"
+					(reference "NFET2")
+					(unit 1)
+				)
+			)
+		)
+	)
+	(symbol
 		(lib_id "Device:R")
 		(at 139.7 116.84 0)
@@
 	)
 	(symbol
-		(lib_id "mr-parts:Diodes Inc DMTH6010SK3Q")
-		(at 158.75 100.33 270)
-		(mirror x)
-		(unit 1)
-		(body_style 1)
-		(exclude_from_sim no)
-		(in_bom yes)
-		(on_board yes)
-		(in_pos_files yes)
-		(dnp no)
-		(property "Reference" "NFET2"
-			(at 155.956 92.964 90)
-			(show_name no)
-			(do_not_autoplace no)
-			(effects
-				(font
-					(size 1.27 1.27)
-				)
-				(justify left)
-			)
-		)
-		(property "Value" "DMTH6010SK3Q"
-			(at 150.876 95.504 90)
-			(show_name no)
-			(do_not_autoplace no)
-			(effects
-				(font
-					(size 1.27 1.27)
-				)
-				(justify left)
-			)
-		)
-		(property "Footprint" "mr-stuff:Diodes Inc DMTH6010SK3Q"
-			(at 158.75 100.33 0)
-			(hide yes)
-			(show_name no)
-			(do_not_autoplace no)
-			(effects
-				(font
-					(size 1.27 1.27)
-				)
-			)
-		)
-		(property "Datasheet" "https://www.diodes.com/datasheet/download/DMTH6010SK3Q.pdf"
-			(at 145.796 100.33 0)
-			(hide yes)
-			(show_name no)
-			(do_not_autoplace no)
-			(effects
-				(font
-					(size 1.27 1.27)
-				)
-			)
-		)
-		(property "Description" ""
-			(at 158.75 100.33 0)
-			(hide yes)
-			(show_name no)
-			(do_not_autoplace no)
-			(effects
-				(font
-					(size 1.27 1.27)
-				)
-			)
-		)
-		(pin "3"
-		)
-		(pin "2"
-		)
-		(pin "1"
-		)
-		(instances
-			(project "Masthead Controller"
-				(path "/2a070473-cb6e-4844-8f2a-5ea6a35ddb49"
-					(reference "NFET2")
-					(unit 1)
-				)
-			)
-		)
-	)
-	(symbol
 		(lib_id "mr-parts:AL8861MP-13")
 		(at 378.46 115.57 0)
@@
 	)
 	(symbol
+		(lib_name "Diodes Inc DMTH6010SK3Q_1")
 		(lib_id "mr-parts:Diodes Inc DMTH6010SK3Q")
 		(at 160.02 29.21 270)
@@
 			)
 		)
-		(property "Description" ""
+		(property "Description" "N-Channel 60 V 16.3A (Ta), 70A (Tc) 3.1W (Ta) Surface Mount TO-252-3"
 			(at 160.02 29.21 0)
 			(hide yes)
 			(show_name no)
+			(do_not_autoplace no)
+			(effects
+				(font
+					(size 1.27 1.27)
+				)
+			)
+		)
+		(property "Part" "Diodes Inc. DMTH6010SK3Q-13"
+			(at 160.02 29.21 90)
+			(hide yes)
+			(show_name no)
