File: Full Boards/Masthead Controller/Masthead Controller.kicad_sch (KiCad schematic)
At the start: 184 parts, among them Q1 2N7002, Q2 2N7002, Q3 BSS138P,215, Q4 BSS138P,215, SW1 SW_MEC_5G, SW2 SW_MEC_5G

Commit message: Updated the metadata for the AL8861QMP-13 parts.
Signed-off-by: digimer <digital.mermaid@gmail.com>
Parts:
- DAC1, DAC2, DAC3: Part (none) -> Microchip MCP4728T-E/UN
- LD1, LD10, LD11, LD12, LD2, LD3, LD4, LD5, LD6, LD7, LD8, LD9: Part (none) -> Diodes Inc AL8861QMP-13
- NFET1, NFET2: Part Diodes Inc. DMTH6010SK3Q-13 -> Diodes Inc DMTH6010SK3Q-13
Connections:
- no-connect marks 13 -> 16
Changed lines of the file:
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@@
 	)
 	(no_connect
+		(at 22.86 168.91)
+	)
+	(no_connect
 		(at 78.74 199.39)
 	)
@@
 	)
 	(no_connect
+		(at 0 173.99)
+	)
+	(no_connect
 		(at 78.74 196.85)
 	)
@@
 	)
 	(no_connect
+		(at 95.25 110.49)
+	)
+	(no_connect
 		(at 78.74 184.15)
 	)
@@
 			)
 		)
-		(property "Datasheet" "AL8861MP-13"
+		(property "Datasheet" "https://www.diodes.com/assets/Datasheets/AL8861Q.pdf"
 			(at 384.81 60.198 0)
 			(hide yes)
@@
 			)
 		)
-		(property "Description" ""
+		(property "Description" "LED Driver IC 1 Output DC DC Regulator Step-Down (Buck) Analog, PWM Dimming 1.5A 8-MSOP-EP"
 			(at 384.81 36.83 0)
 			(hide yes)
@@
 			)
 		)
+		(property "Part" "Diodes Inc AL8861QMP-13"
+			(at 384.81 64.77 0)
+			(hide yes)
+			(show_name no)
+			(do_not_autoplace no)
+			(effects
+				(font
+					(size 1.27 1.27)
+				)
+			)
+		)
 		(pin "8"
 		)
@@
 			)
 		)
-		(property "Datasheet" "AL8861MP-13"
+		(property "Datasheet" "https://www.diodes.com/assets/Datasheets/AL8861Q.pdf"
 			(at 276.86 138.938 0)
 			(hide yes)
@@
 			)
 		)
-		(property "Description" ""
+		(property "Description" "LED Driver IC 1 Output DC DC Regulator Step-Down (Buck) Analog, PWM Dimming 1.5A 8-MSOP-EP"
 			(at 276.86 115.57 0)
 			(hide yes)
@@
 			)
 		)
+		(property "Part" "Diodes Inc AL8861QMP-13"
+			(at 276.86 143.51 0)
+			(hide yes)
+			(show_name no)
+			(do_not_autoplace no)
+			(effects
+				(font
+					(size 1.27 1.27)
+				)
+			)
+		)
 		(pin "8"
 		)
@@
 			)
 		)
-		(property "Datasheet" "AL8861MP-13"
+		(property "Datasheet" "https://www.diodes.com/assets/Datasheets/AL8861Q.pdf"
 			(at 384.81 97.028 0)
 			(hide yes)
@@
 			)
 		)
-		(property "Description" ""
+		(property "Description" "LED Driver IC 1 Output DC DC Regulator Step-Down (Buck) Analog, PWM Dimming 1.5A 8-MSOP-EP"
 			(at 384.81 73.66 0)
 			(hide yes)
@@
 			)
 		)
+		(property "Part" "Diodes Inc AL8861QMP-13"
+			(at 384.81 101.6 0)
+			(hide yes)
+			(show_name no)
+			(do_not_autoplace no)
+			(effects
+				(font
+					(size 1.27 1.27)
+				)
+			)
+		)
 		(pin "8"
 		)
@@
 			)
 		)
+		(property "Part" "Microchip MCP4728T-E/UN"
+			(at 198.12 256.54 0)
+			(hide yes)
+			(show_name no)
+			(do_not_autoplace no)
+			(effects
+				(font
+					(size 1.27 1.27)
+				)
+			)
+		)
 		(pin "1"
 		)
@@
 			)
 		)
-		(property "Part" "Diodes Inc. DMTH6010SK3Q-13"
+		(property "Part" "Diodes Inc DMTH6010SK3Q-13"
 			(at 168.91 97.79 90)
 			(hide yes)
@@
 			)
 		)
-		(property "Datasheet" "AL8861MP-13"
+		(property "Datasheet" "https://www.diodes.com/assets/Datasheets/AL8861Q.pdf"
 			(at 276.86 60.198 0)
 			(hide yes)
@@
 			)
 		)
-		(property "Description" ""
+		(property "Description" "LED Driver IC 1 Output DC DC Regulator Step-Down (Buck) Analog, PWM Dimming 1.5A 8-MSOP-EP"
 			(at 276.86 36.83 0)
 			(hide yes)
@@
 			)
 		)
+		(property "Part" "Diodes Inc AL8861QMP-13"
+			(at 276.86 64.77 0)
+			(hide yes)
+			(show_name no)
+			(do_not_autoplace no)
+			(effects
+				(font
+					(size 1.27 1.27)
+				)
+			)
+		)
 		(pin "8"
 		)
@@
 			)
 		)
-		(property "Datasheet" "AL8861MP-13"
+		(property "Datasheet" "https://www.diodes.com/assets/Datasheets/AL8861Q.pdf"
 			(at 488.95 175.768 0)
 			(hide yes)
@@
 			)
 		)
-		(property "Description" ""
+		(property "Description" "LED Driver IC 1 Output DC DC Regulator Step-Down (Buck) Analog, PWM Dimming 1.5A 8-MSOP-EP"
 			(at 488.95 152.4 0)
 			(hide yes)
@@
 			)
 		)
+		(property "Part" "Diodes Inc AL8861QMP-13"
+			(at 488.95 180.34 0)
+			(hide yes)
+			(show_name no)
+			(do_not_autoplace no)
+			(effects
+				(font
+					(size 1.27 1.27)
+				)
+			)
+		)
 		(pin "8"
 		)
@@
 			)
 		)
-		(property "Datasheet" "AL8861MP-13"
+		(property "Datasheet" "https://www.diodes.com/assets/Datasheets/AL8861Q.pdf"
 			(at 488.95 138.938 0)
 			(hide yes)
@@
 			)
 		)
-		(property "Description" ""
+		(property "Description" "LED Driver IC 1 Output DC DC Regulator Step-Down (Buck) Analog, PWM Dimming 1.5A 8-MSOP-EP"
 			(at 488.95 115.57 0)
 			(hide yes)
@@
 			)
 		)
+		(property "Part" "Diodes Inc AL8861QMP-13"
+			(at 488.95 143.51 0)
+			(hide yes)
+			(show_name no)
+			(do_not_autoplace no)
+			(effects
+				(font
+					(size 1.27 1.27)
+				)
+			)
+		)
 		(pin "8"
 		)
@@
 			)
 		)
-		(property "Datasheet" "AL8861MP-13"
+		(property "Datasheet" "https://www.diodes.com/assets/Datasheets/AL8861Q.pdf"
 			(at 492.76 95.758 0)
 			(hide yes)
@@
 			)
 		)
-		(property "Description" ""
+		(property "Description" "LED Driver IC 1 Output DC DC Regulator Step-Down (Buck) Analog, PWM Dimming 1.5A 8-MSOP-EP"
 			(at 492.76 72.39 0)
 			(hide yes)
@@
 			)
 		)
+		(property "Part" "Diodes Inc AL8861QMP-13"
+			(at 492.76 100.33 0)
+			(hide yes)
+			(show_name no)
+			(do_not_autoplace no)
+			(effects
+				(font
+					(size 1.27 1.27)
+				)
+			)
+		)
 		(pin "8"
 		)
@@
 			)
 		)
-		(property "Datasheet" "AL8861MP-13"
+		(property "Datasheet" "https://www.diodes.com/assets/Datasheets/AL8861Q.pdf"
 			(at 384.81 175.768 0)
 			(hide yes)
@@
 			)
 		)
-		(property "Description" ""
+		(property "Description" "LED Driver IC 1 Output DC DC Regulator Step-Down (Buck) Analog, PWM Dimming 1.5A 8-MSOP-EP"
 			(at 384.81 152.4 0)
 			(hide yes)
@@
 			)
 		)
+		(property "Part" "Diodes Inc AL8861QMP-13"
+			(at 384.81 180.34 0)
+			(hide yes)
+			(show_name no)
+			(do_not_autoplace no)
+			(effects
+				(font
+					(size 1.27 1.27)
+				)
+			)
+		)
 		(pin "8"
 		)
@@
 			)
 		)
-		(property "Datasheet" "AL8861MP-13"
+		(property "Datasheet" "https://www.diodes.com/assets/Datasheets/AL8861Q.pdf"
 			(at 384.81 138.938 0)
 			(hide yes)
@@
 			)
 		)
-		(property "Description" ""
+		(property "Description" "LED Driver IC 1 Output DC DC Regulator Step-Down (Buck) Analog, PWM Dimming 1.5A 8-MSOP-EP"
 			(at 384.81 115.57 0)
 			(hide yes)
@@
 			)
 		)
+		(property "Part" "Diodes Inc AL8861QMP-13"
+			(at 384.81 143.51 0)
+			(hide yes)
+			(show_name no)
+			(do_not_autoplace no)
+			(effects
+				(font
+					(size 1.27 1.27)
+				)
+			)
+		)
 		(pin "8"
 		)
@@
 			)
 		)
-		(property "Datasheet" "AL8861MP-13"
+		(property "Datasheet" "https://www.diodes.com/assets/Datasheets/AL8861Q.pdf"
 			(at 276.86 175.768 0)
 			(hide yes)
@@
 			)
 		)
-		(property "Description" ""
+		(property "Description" "LED Driver IC 1 Output DC DC Regulator Step-Down (Buck) Analog, PWM Dimming 1.5A 8-MSOP-EP"
 			(at 276.86 152.4 0)
 			(hide yes)
@@
 			)
 		)
+		(property "Part" "Diodes Inc AL8861QMP-13"
+			(at 276.86 180.34 0)
+			(hide yes)
+			(show_name no)
+			(do_not_autoplace no)
+			(effects
+				(font
+					(size 1.27 1.27)
+				)
+			)
+		)
 		(pin "8"
 		)
@@
 			)
 		)
-		(property "Datasheet" "AL8861MP-13"
+		(property "Datasheet" "https://www.diodes.com/assets/Datasheets/AL8861Q.pdf"
 			(at 492.76 60.198 0)
 			(hide yes)
@@
 			)
 		)
-		(property "Description" ""
+		(property "Description" "LED Driver IC 1 Output DC DC Regulator Step-Down (Buck) Analog, PWM Dimming 1.5A 8-MSOP-EP"
 			(at 492.76 36.83 0)
 			(hide yes)
@@
 			)
 		)
+		(property "Part" "Diodes Inc AL8861QMP-13"
+			(at 492.76 64.77 0)
+			(hide yes)
+			(show_name no)
+			(do_not_autoplace no)
+			(effects
+				(font
+					(size 1.27 1.27)
+				)
+			)
+		)
 		(pin "8"
 		)
@@
 			)
 		)
-		(property "Part" "Diodes Inc. DMTH6010SK3Q-13"
+		(property "Part" "Diodes Inc DMTH6010SK3Q-13"
 			(at 170.18 30.48 90)
 			(hide yes)
@@
 			)
 		)
+		(property "Part" "Microchip MCP4728T-E/UN"
+			(at 198.12 307.34 0)
+			(hide yes)
+			(show_name no)
+			(do_not_autoplace no)
+			(effects
+				(font
+					(size 1.27 1.27)
+				)
+			)
+		)
 		(pin "1"
 		)
@@
 			)
 		)
+		(property "Part" "Microchip MCP4728T-E/UN"
+			(at 198.12 281.94 0)
+			(hide yes)
+			(show_name no)
+			(do_not_autoplace no)
+			(effects
+				(font
+					(size 1.27 1.27)
+				)
+			)
+		)
 		(pin "1"
 		)
@@
 			)
 		)
-		(property "Datasheet" "AL8861MP-13"
+		(property "Datasheet" "https://www.diodes.com/assets/Datasheets/AL8861Q.pdf"
 			(at 276.86 97.028 0)
 			(hide yes)
@@
 			)
 		)
-		(property "Description" ""
+		(property "Description" "LED Driver IC 1 Output DC DC Regulator Step-Down (Buck) Analog, PWM Dimming 1.5A 8-MSOP-EP"
 			(at 276.86 73.66 0)
 			(hide yes)
 			(show_name no)
+			(do_not_autoplace no)
+			(effects
+				(font
+					(size 1.27 1.27)
+				)
+			)
+		)
+		(property "Part" "Diodes Inc AL8861QMP-13"
+			(at 276.86 101.6 0)
+			(hide yes)
+			(show_name no)

Commit message: Added `Part` for the Onsemi NRVBA340NT3G.
Signed-off-by: digimer <digital.mermaid@gmail.com>
Parts:
- D10, D11, D12, D13, D14, D15, D4, D5, D6, D7, D8, D9: Part (none) -> Onsemi NRVBA340NT3G
Changed lines of the file:
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@@
 			)
 		)
+		(property "Part" "Onsemi NRVBA340NT3G"
+			(at 403.86 146.05 0)
+			(hide yes)
+			(show_name no)
+			(do_not_autoplace no)
+			(effects
+				(font
+					(size 1.27 1.27)
+				)
+			)
+		)
 		(pin "2"
 		)
@@
 			)
 		)
+		(property "Part" "Onsemi NRVBA340NT3G"
+			(at 509.27 111.76 0)
+			(hide yes)
+			(show_name no)
+			(do_not_autoplace no)
+			(effects
+				(font
+					(size 1.27 1.27)
+				)
+			)
+		)
 		(pin "2"
 		)
@@
 			)
 		)
+		(property "Part" "Onsemi NRVBA340NT3G"
+			(at 511.81 33.02 0)
+			(hide yes)
+			(show_name no)
+			(do_not_autoplace no)
+			(effects
+				(font
+					(size 1.27 1.27)
+				)
+			)
+		)
 		(pin "2"
 		)
@@
 			)
 		)
+		(property "Part" "Onsemi NRVBA340NT3G"
+			(at 297.18 33.02 0)
+			(hide yes)
+			(show_name no)
+			(do_not_autoplace no)
+			(effects
+				(font
+					(size 1.27 1.27)
+				)
+			)
+		)
 		(pin "2"
 		)
@@
 			)
 		)
+		(property "Part" "Onsemi NRVBA340NT3G"
+			(at 403.86 111.76 0)
+			(hide yes)
+			(show_name no)
+			(do_not_autoplace no)
+			(effects
+				(font
+					(size 1.27 1.27)
+				)
+			)
+		)
 		(pin "2"
 		)
@@
 			)
 		)
+		(property "Part" "Onsemi NRVBA340NT3G"
+			(at 403.86 69.85 0)
+			(hide yes)
+			(show_name no)
+			(do_not_autoplace no)
+			(effects
+				(font
+					(size 1.27 1.27)
+				)
+			)
+		)
 		(pin "2"
 		)
@@
 			)
 		)
+		(property "Part" "Onsemi NRVBA340NT3G"
+			(at 509.27 148.59 0)
+			(hide yes)
+			(show_name no)
+			(do_not_autoplace no)
+			(effects
+				(font
+					(size 1.27 1.27)
+				)
+			)
+		)
 		(pin "2"
 		)
@@
 			)
 		)
+		(property "Part" "Onsemi NRVBA340NT3G"
+			(at 403.86 33.02 0)
+			(hide yes)
+			(show_name no)
+			(do_not_autoplace no)
+			(effects
+				(font
+					(size 1.27 1.27)
+				)
+			)
+		)
 		(pin "2"
 		)
@@
 			)
 		)
+		(property "Part" "Onsemi NRVBA340NT3G"
+			(at 295.91 148.59 0)
+			(hide yes)
+			(show_name no)
+			(do_not_autoplace no)
+			(effects
+				(font
+					(size 1.27 1.27)
+				)
+			)
+		)
 		(pin "2"
 		)
@@
 			)
 		)
+		(property "Part" "Onsemi NRVBA340NT3G"
+			(at 295.91 111.76 0)
+			(hide yes)
+			(show_name no)
+			(do_not_autoplace no)
+			(effects
+				(font
+					(size 1.27 1.27)
+				)
+			)
+		)
 		(pin "2"
 		)
@@
 			)
 		)
+		(property "Part" "Onsemi NRVBA340NT3G"
+			(at 295.91 69.85 0)
+			(hide yes)
+			(show_name no)
+			(do_not_autoplace no)
+			(effects
+				(font
+					(size 1.27 1.27)
+				)
+			)
+		)
 		(pin "2"
 		)
@@
 			(at 511.81 68.58 0)
 			(hide yes)
+			(show_name no)
+			(do_not_autoplace no)
+			(effects
+				(font
+					(size 1.27 1.27)
+				)
+			)
+		)
+		(property "Part" "Onsemi NRVBA340NT3G"
+			(at 511.81 68.58 0)
+			(hide yes)

Commit message: Added `Part` to Phoenix Contact 1862437
Signed-off-by: digimer <digital.mermaid@gmail.com>
Parts:
- TB4, TB5, TB6, TB7, TB8, TB9: Part (none) -> Phoenix Contact 1862437
Changed lines of the file:
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@@
 			)
 		)
+		(property "Part" "Phoenix Contact 1862437"
+			(at 557.53 145.034 0)
+			(hide yes)
+			(show_name no)
+			(do_not_autoplace no)
+			(effects
+				(font
+					(size 1.27 1.27)
+				)
+			)
+		)
 		(pin "5"
 		)
@@
 			)
 		)
+		(property "Part" "Phoenix Contact 1862437"
+			(at 449.58 66.294 0)
+			(hide yes)
+			(show_name no)
+			(do_not_autoplace no)
+			(effects
+				(font
+					(size 1.27 1.27)
+				)
+			)
+		)
 		(pin "5"
 		)
@@
 			)
 		)
+		(property "Part" "Phoenix Contact 1862437"
+			(at 449.58 145.034 0)
+			(hide yes)
+			(show_name no)
+			(do_not_autoplace no)
+			(effects
+				(font
+					(size 1.27 1.27)
+				)
+			)
+		)
 		(pin "5"
 		)
@@
 			)
 		)
+		(property "Part" "Phoenix Contact 1862437"
+			(at 341.63 145.034 0)
+			(hide yes)
+			(show_name no)
+			(do_not_autoplace no)
+			(effects
+				(font
+					(size 1.27 1.27)
+				)
+			)
+		)
 		(pin "5"
 		)
@@
 			)
 		)
+		(property "Part" "Phoenix Contact 1862437"
+			(at 341.63 66.294 0)
+			(hide yes)
+			(show_name no)
+			(do_not_autoplace no)
+			(effects
+				(font
+					(size 1.27 1.27)
+				)
+			)
+		)
 		(pin "5"
 		)
@@
 			(hide yes)
 			(show_name no)
+			(do_not_autoplace no)
+			(effects
+				(font
+					(size 1.27 1.27)
+				)
+			)
+		)
+		(property "Part" "Phoenix Contact 1862437"
+			(at 557.53 66.294 0)
+			(hide yes)
+			(show_name no)

Commit message: Added Part and Footprint for Pheonix Contact 1862440
Signed-off-by: digimer <digital.mermaid@gmail.com>
Parts:
- EF1, EF2: Part (none) -> TI TPS26631PWP
- TB1: Part (none) -> Phoenix Contact 1862440
Changed lines of the file:
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@@
 			)
 		)
+		(property "Part" "TI TPS26631PWP"
+			(at 189.23 151.13 0)
+			(hide yes)
+			(show_name no)
+			(do_not_autoplace no)
+			(effects
+				(font
+					(size 1.27 1.27)
+				)
+			)
+		)
 		(pin "16"
 		)
@@
 			)
 		)
+		(property "Part" "TI TPS26631PWP"
+			(at 189.23 83.82 0)
+			(hide yes)
+			(show_name no)
+			(do_not_autoplace no)
+			(effects
+				(font
+					(size 1.27 1.27)
+				)
+			)
+		)
 		(pin "16"
 		)
@@
 			(hide yes)
 			(show_name no)
+			(do_not_autoplace no)
+			(effects
+				(font
+					(size 1.27 1.27)
+				)
+			)
+		)
+		(property "Part" "Phoenix Contact 1862440"
+			(at 121.92 29.21 0)
+			(hide yes)
+			(show_name no)

Commit message: Added Part to TI TCAN330DR
Signed-off-by: digimer <digital.mermaid@gmail.com>
Parts:
- CAN1: Part (none) -> TI TCAN330DR
- MCU1: Part (none) -> Espressif ESP32-S3-WROOM-1-N16R2
Changed lines of the file:
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@@
 			)
 		)
+		(property "Part" "TI TCAN330DR"
+			(at 59.69 76.2 0)
+			(hide yes)
+			(show_name no)
+			(do_not_autoplace no)
+			(effects
+				(font
+					(size 1.27 1.27)
+				)
+			)
+		)
 		(pin "2"
 		)
@@
 			(at 63.5 199.39 0)
 			(hide yes)
+			(show_name no)
+			(do_not_autoplace no)
+			(effects
+				(font
+					(size 1.27 1.27)
+				)
+			)
+		)
+		(property "Part" "Espressif ESP32-S3-WROOM-1-N16R2"
+			(at 63.5 199.39 0)
+			(hide yes)

Commit message: Added Part for Sensirion SHT41A
Signed-off-by: digimer <digital.mermaid@gmail.com>
Parts:
- HTS1: Part (none) -> Sensirion SHT41A-AW1B-R2
- VR1: Part (none) -> TI TPSM33610S3QRDNRQ1
Connections:
- no-connect marks 16 -> 15
Changed lines of the file:
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@@
 	)
 	(no_connect
-		(at 0 173.99)
-	)
-	(no_connect
 		(at 78.74 196.85)
 	)
@@
 			)
 		)
+		(property "Part" "TI TPSM33610S3QRDNRQ1"
+			(at 58.42 126.238 0)
+			(hide yes)
+			(show_name no)
+			(do_not_autoplace no)
+			(effects
+				(font
+					(size 1.27 1.27)
+				)
+			)
+		)
 		(pin "1"
 		)
@@
 			(hide yes)
 			(show_name no)
+			(do_not_autoplace no)
+			(effects
+				(font
+					(size 1.27 1.27)
+				)
+			)
+		)
+		(property "Part" "Sensirion SHT41A-AW1B-R2"
+			(at 199.39 206.502 0)
+			(hide yes)
+			(show_name no)

Commit message: Added Part to SMCJ33A
Signed-off-by: digimer <digital.mermaid@gmail.com>
Parts:
- TVS1: Part (none) -> Littelfuse SMCJ33A
Connections:
- no-connect marks 15 -> 14
Changed lines of the file:
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@@
 	)
 	(no_connect
-		(at 95.25 110.49)
-	)
-	(no_connect
 		(at 78.74 184.15)
 	)
@@
 			(hide yes)
 			(show_name no)
+			(do_not_autoplace no)
+			(effects
+				(font
+					(size 1.27 1.27)
+				)
+			)
+		)
+		(property "Part" "Littelfuse SMCJ33A"
+			(at 85.09 96.52 0)
+			(hide yes)
+			(show_name no)

Commit message: Fixed the metadata for TI ADS1115BQDGSRQ1
Signed-off-by: digimer <digital.mermaid@gmail.com>
Parts:
- ADC1: value TI ADS1115BQDGSRQ1 -> ADS1115BQDGSRQ1; MANUFACTURER Texas Instruments -> (none); MAXIMUM_PACKAGE_HEIGHT 1.1 mm -> (none); PARTREV D -> (none); Part (none) -> TI ADS1115BQDGSRQ1; STANDARD IPC 7351B -> (none)
Changed lines of the file:
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@@
 			)
 		)
-		(property "Value" "TI ADS1115BQDGSRQ1"
+		(property "Value" "ADS1115BQDGSRQ1"
 			(at 194.31 210.566 0)
 			(show_name no)
@@
 			)
 		)
-		(property "PARTREV" "D"
+		(property "Part" "TI ADS1115BQDGSRQ1"
 			(at 186.69 236.982 0)
 			(hide yes)
 			(show_name no)
-			(do_not_autoplace no)
-			(effects
-				(font
-					(size 1.27 1.27)
-				)
-				(justify bottom)
-			)
-		)
-		(property "STANDARD" "IPC 7351B"
-			(at 194.31 236.982 0)
-			(hide yes)
-			(show_name no)
-			(do_not_autoplace no)
-			(effects
-				(font
-					(size 1.27 1.27)
-				)
-				(justify bottom)
-			)
-		)
-		(property "MAXIMUM_PACKAGE_HEIGHT" "1.1 mm"
-			(at 204.724 236.982 0)
-			(hide yes)
-			(show_name no)
-			(do_not_autoplace no)
-			(effects
-				(font
-					(size 1.27 1.27)
-				)
-				(justify bottom)
-			)
-		)
-		(property "MANUFACTURER" "Texas Instruments"
-			(at 194.31 232.41 0)
-			(hide yes)
-			(show_name no)
