File: Full Boards/Compass Rose/Compass Rose.kicad_pcb (KiCad board)
At the start: 4 copper layers, 170 x 180 mm, 247 parts, among them J1 Program Header, J2 Future Bonding, Q10 2N3904, Q11 AO3401A, Q12 2N3904, Q7 AO3401A, Q8 2N3904, Q9 AO3401A, SW1 SW_MEC_5G, SW2 SW_MEC_5G, U1 ISO1044BD, U2 LM1117MP-5.0, U3 MAX3232, U4 STM32C092KCT6, U5 IS31FL3731-SA, U6 FM24CL64B-G, U7 FM24CL64B-G

Commit message: Started updating the compass rose.
Signed-off-by: digimer <digital.mermaid@gmail.com>
Parts:
- removed G***: LOGO, mr-stuff:cc-by-nc-sa_8mm
Other:
- board text added: "-=] License CERN Open Hardware Licence Weakly Reciprocal Version 2"
- board text added: "NMEA2000 Two-Ring Compass Rose v4.1 - Prototype - 01 © The Digital Mermaid - 2026"
- board text removed: "NMEA2000 Two-Ring Compass Rose v4 - Prototype - 01 © The Digital Mermaid - 2025"
- board text removed: "v4.0"
