File: Full Boards/Battery Display/Battery Display.kicad_pcb (KiCad board)
At the start: 4 copper layers, 110 x 175.2 mm, 196 parts, among them J1 Future Bonding, J2 Program Header, Q1 AO3401A, Q2 2N3904, Q3 AO3401A, Q4 2N3904, Q5 AO3401A, Q6 2N3904, SW1 SW_MEC_5G, SW2 SW_MEC_5G, U1 ISO1044BD, U2 LM1117MP-5.0, U3 STM32C092KCT6, U4 IS31FL3731-SA, U5 MAX3232, U6 FM24CL64B-G, U7 FM24CL64B-G

Commit message: Blanked the PCB, save for the LED section.
Signed-off-by: digimer <digital.mermaid@gmail.com>
Parts:
- removed C12: 0.1uF, mr-stuff:RCE5C1H104J2A2H03B
- removed D145: 1N5822, Diode_THT:D_DO-201AD_P15.24mm_Horizontal
- removed D146: SLD22-018, mr-stuff:DIOAD4425W136L885D885
- removed G***: LOGO, mr-stuff:cc-by-nc-sa_8mm
- removed J1: Future Bonding, Connector_PinHeader_2.54mm:PinHeader_1x03_P2.54mm_Horizontal
- removed J2: Program Header, Connector_PinHeader_2.54mm:PinHeader_1x05_P2.54mm_Horizontal
- removed L1: PA4340.103NLT, mr-stuff:Pulse PA4340.103NLT
- removed LCD1: ~, mr-stuff:NHD-0216K3Z-NS(RGB)-FBW-V3
- removed LR1: NCV8730ASN500T1G, mr-stuff:TSOP-5_483_OSI
- removed N2K1: ~, mr-stuff:M12B-05PMMR
- removed PS1: SPBW06F-05, mr-stuff:SPBW06F05
- removed PTC1: PTC, mr-stuff:AHEF100
- removed Q1, Q3, Q5: AO3401A, Package_TO_SOT_SMD:SOT-23
- removed Q2, Q4, Q6: 2N3904, Package_TO_SOT_THT:TO-92_Inline
- removed R89: 475, Resistor_THT:R_Axial_DIN0207_L6.3mm_D2.5mm_P7.62mm_Horizontal
- removed SW1, SW2: SW_MEC_5G, mr-stuff:SW_TS03-66-50-BK-160-LCR-D-67
- removed TP10, TP12, TP7: +5V_SHIP, Connector_PinHeader_2.54mm:PinHeader_1x01_P2.54mm_Vertical
- removed TP11, TP13, TP8: GND_SHIP, Connector_PinHeader_2.54mm:PinHeader_1x01_P2.54mm_Vertical
- removed TP5: +5V, Connector_PinHeader_2.54mm:PinHeader_1x01_P2.54mm_Vertical
- removed TP6: GND, Connector_PinHeader_2.54mm:PinHeader_1x01_P2.54mm_Vertical
- removed TP9: +3.3V, Connector_PinHeader_2.54mm:PinHeader_1x01_P2.54mm_Vertical
- removed U1: ISO1044BD, Package_SO:SOIC-8_3.9x4.9mm_P1.27mm
- removed U2: LM1117MP-5.0, Package_TO_SOT_SMD:SOT-223-3_TabPin2
- removed U3: STM32C092KCT6, Package_DFN_QFN:QFN-32-1EP_5x5mm_P0.5mm_EP3.45x3.45mm
- removed U4: IS31FL3731-SA, Package_SO:SSOP-28_5.3x10.2mm_P0.65mm
- removed U5: MAX3232, Package_SO:TSSOP-16_4.4x5mm_P0.65mm
- removed U6, U7: FM24CL64B-G, Package_SO:SOIC-8_3.9x4.9mm_P1.27mm
- added C29: 0.1uF, mr-stuff:Kyocera AVX 0805, F.Cu at (221.2, 95.6)
- added C30: 0.1uF, mr-stuff:Kyocera AVX 0805, F.Cu at (221.2, 98.7)
- added C31: 0.1uF, mr-stuff:Kyocera AVX 0805, F.Cu at (221.2, 101.8)
- added C32: 0.1uF, mr-stuff:Kyocera AVX 0805, F.Cu at (225.8, 80.1)
- added CMC1: ACT12101012PTL00, mr-stuff:TDK ACT12101012PTL00, F.Cu at (218.2, 106.2)
- added CPD1: IS31FL3731-SA, Package_SO:SSOP-28_5.3x10.2mm_P0.65mm, F.Cu at (265.8, 64.1)
- added FID1: Fiducial, Fiducial:Fiducial_0.5mm_Mask1.5mm, F.Cu at (229.3, 104.9)
- added FID2: Fiducial, Fiducial:Fiducial_0.5mm_Mask1.5mm, F.Cu at (229.3, 108.0)
- added FID3: Fiducial, Fiducial:Fiducial_0.5mm_Mask1.5mm, F.Cu at (229.3, 111.0)
- added ICT1: ISO1044BD, mr-stuff:TI ISO1044BDR, F.Cu at (265.3, 52.0)
- added IDCB1: SPBW06F-05, mr-stuff:Meanwell SPBW06F05, F.Cu at (245.3, 97.5)
- added J3: Program Header, Connector_PinHeader_2.54mm:PinHeader_1x05_P2.54mm_Horizontal, F.Cu at (196.7, 96.3)
- added J4: Optional Bond, Connector_PinHeader_2.54mm:PinHeader_1x02_P2.54mm_Vertical, F.Cu at (234.9, 105.8)
- added L2: PA4340.103NLT, mr-stuff:Pulse PA4340.103NLT, F.Cu at (252.9, 73.7)
- added LCD2: NHD-0216K3Z-NS(RGB)-FBW-V3, mr-stuff:Newhaven Display NHD-0216K3Z-NS(RGB)-FBW-V3, F.Cu at (220.4, 39.6)
- added LS1: TI PCA9306IDCURQ1, mr-stuff:TI PCA9306, F.Cu at (210.5, 85.6)
- added LVR1: BD450S5FP-CE2, mr-stuff:Rohm BD4xxS5 TO252-3, F.Cu at (265.2, 39.1)
- added LVR2: BD33C0AFP-CE2, mr-stuff:Rohm BD33C0, F.Cu at (264.5, 82.5)
- added MCU1: STM32C092KCT6, mr-stuff:STM STM32C0 LQFP-32, F.Cu at (254.7, 64.1)
- added OX1: 12.60378, Crystal:Crystal_SMD_3225-4Pin_3.2x2.5mm, F.Cu at (205.2, 111.1)
- added PTC2: 0ZCG0110CF2B, mr-stuff:Bel Fuse 0ZCG, F.Cu at (184.1, 110.4)
- added Q10: DMN6075S, Package_TO_SOT_SMD:SOT-23, F.Cu at (192.0, 94.8)
- added Q11: BSS314PE, Package_TO_SOT_SMD:SOT-23, F.Cu at (192.0, 99.2)
- added Q12: DMN6075S, Package_TO_SOT_SMD:SOT-23, F.Cu at (192.0, 103.7)
- added Q7: BSS314PE, Package_TO_SOT_SMD:SOT-23, F.Cu at (192.0, 81.4)
- added Q8: DMN6075S, Package_TO_SOT_SMD:SOT-23, F.Cu at (192.0, 85.9)
- added Q9: BSS314PE, Package_TO_SOT_SMD:SOT-23, F.Cu at (192.0, 90.3)
- added R28: 3.3k, mr-stuff:Stackpole RNCF0805, F.Cu at (205.5, 83.6)
- added R29: 3.3k, mr-stuff:Stackpole RNCF0805, F.Cu at (205.5, 86.6)
- added ROM1: M24C64, mr-stuff:STM M24C64-RMN6P, F.Cu at (266.0, 24.2)
- added ROM2: M24C64, mr-stuff:STM M24C64-RMN6P, F.Cu at (266.0, 30.7)
- added RST1: MAX3232, mr-stuff:TI MAX3232EIPWRQ1, F.Cu at (265.0, 73.4)
- added SD1: VS-30MQ040HM3/5AT, Diode_SMD:D_SMA, F.Cu at (198.5, 111.1)
- added SW3: Boot, mr-stuff:Same Sky TS03-66, F.Cu at (262.7, 95.0)
- added SW4: Reset, mr-stuff:Same Sky TS03-66, F.Cu at (262.7, 102.6)
- added TB1: 1862440, mr-stuff:Phoenix Contact 1862440, F.Cu at (257.0, 87.4)
- C1, C17, C18, C19, C2, C20, C21, C22, C5: footprint mr-stuff:RCE5C1H104J2A2H03B -> mr-stuff:Kyocera AVX 0805; moved to F.Cu
- C10: value 4.7uF -> 10uF; footprint mr-stuff:RCER71E475K2A2H03B -> mr-stuff:Kyocera AVX 1206; moved to F.Cu
- C11: value 0.1uF -> 1nF; footprint mr-stuff:RCE5C1H104J2A2H03B -> mr-stuff:Knowles Syfer 2211JA25; moved to F.Cu
- C13: value 100uF -> 10uF; footprint Capacitor_THT:CP_Radial_D8.0mm_P5.00mm -> mr-stuff:TDK CGA5; moved to F.Cu
- C14: value 100uF -> 22uF; footprint Capacitor_THT:CP_Radial_D8.0mm_P5.00mm -> mr-stuff:Murata GCJ31CR71A; moved to F.Cu
- C15: value 100uF -> 0.1uF; footprint Capacitor_THT:CP_Radial_D8.0mm_P5.00mm -> mr-stuff:Kyocera AVX 0805; moved to F.Cu
- C16: value 1uF -> 0.1uF; footprint Capacitor_THT:C_Rect_L7.2mm_W7.2mm_P5.00mm_FKS2_FKP2_MKS2_MKP2 -> mr-stuff:Kyocera AVX 0805; moved to F.Cu
- C23: value 0.1uF -> 0.01uF; footprint mr-stuff:RCE5C1H104J2A2H03B -> mr-stuff:Kemet C0805X; moved to F.Cu
- C24: value 0.1uF -> 100pF; footprint mr-stuff:RCE5C1H104J2A2H03B -> mr-stuff:Kemet C0805X; moved to F.Cu
- C25, C26, C27: value 0.1uF -> 100uF; footprint mr-stuff:RCE5C1H104J2A2H03B -> Capacitor_THT:CP_Radial_D8.0mm_P3.50mm; moved to F.Cu
- C28: value 0.1uF -> 1uF; footprint mr-stuff:RCE5C1H104J2A2H03B -> mr-stuff:Kemet C1206C; moved to F.Cu
- C3: value 10uF -> 4.7uF; footprint Capacitor_THT:CP_Radial_D8.0mm_P3.50mm -> mr-stuff:Kyocera AVX 1206; moved to F.Cu
- C4: value TDK FA28NP01H152JNU06 -> 0.1uF; footprint mr-stuff:TDK CAPRB500W50L400T250H550 -> mr-stuff:Kyocera AVX 0805; moved to F.Cu
- C6, C7: value 0.1uF -> 16pF; footprint mr-stuff:RCE5C1H104J2A2H03B -> mr-stuff:Kemet C0603X; moved to F.Cu
- C8: value 10uF -> 0.1uF; footprint Capacitor_THT:CP_Radial_D8.0mm_P3.50mm -> mr-stuff:Kyocera AVX 0805; moved to F.Cu
- C9: value 10uF -> 22uF; footprint Capacitor_THT:CP_Radial_D8.0mm_P3.50mm -> mr-stuff:Murata GCJ31CR71A; moved to F.Cu
- DE1: value ~ -> L77SDE09SA4CH4F; moved to F.Cu
- DE2: value ~ -> L777SDE09PA4CH4F; moved to F.Cu
- LED1: renamed from D1; footprint mr-stuff:WP383SURDTK -> mr-stuff:Kingbright WP383SURDTK
- LED10: renamed from D10; footprint mr-stuff:WP383SURDTK -> mr-stuff:Kingbright WP383SURDTK
- LED11: renamed from D11; footprint mr-stuff:WP383SURDTK -> mr-stuff:Kingbright WP383SURDTK
- LED12: renamed from D12; footprint mr-stuff:WP383SURDTK -> mr-stuff:Kingbright WP383SURDTK
- LED13: renamed from D13; footprint mr-stuff:WP383SURDTK -> mr-stuff:Kingbright WP383SURDTK
- LED14: renamed from D14; footprint mr-stuff:WP383SURDTK -> mr-stuff:Kingbright WP383SURDTK
- LED15: renamed from D15; footprint mr-stuff:WP383SURDTK -> mr-stuff:Kingbright WP383SURDTK
- LED16: renamed from D16; footprint mr-stuff:WP383SURDTK -> mr-stuff:Kingbright WP383SURDTK
- LED17: renamed from D17; footprint mr-stuff:WP383SURDTK -> mr-stuff:Kingbright WP383SURDTK
- LED18: renamed from D18; footprint mr-stuff:WP383SURDTK -> mr-stuff:Kingbright WP383SURDTK
- LED19: renamed from D19; footprint mr-stuff:WP383SURDTK -> mr-stuff:Kingbright WP383SURDTK
- LED2: renamed from D2; footprint mr-stuff:WP383SURDTK -> mr-stuff:Kingbright WP383SURDTK
- LED20: renamed from D20; footprint mr-stuff:WP383SURDTK -> mr-stuff:Kingbright WP383SURDTK
- LED21: renamed from D21; footprint mr-stuff:WP383SURDTK -> mr-stuff:Kingbright WP383SURDTK
- LED22: renamed from D22; footprint mr-stuff:WP383SURDTK -> mr-stuff:Kingbright WP383SURDTK
- LED23: renamed from D23; footprint mr-stuff:WP383SURDTK -> mr-stuff:Kingbright WP383SURDTK
- LED24: renamed from D24; footprint mr-stuff:WP383SURDTK -> mr-stuff:Kingbright WP383SURDTK
- LED25: renamed from D25; footprint mr-stuff:WP383SURDTK -> mr-stuff:Kingbright WP383SURDTK
- LED26: renamed from D26; footprint mr-stuff:WP383SURDTK -> mr-stuff:Kingbright WP383SURDTK
- LED27: renamed from D27; footprint mr-stuff:WP383SURDTK -> mr-stuff:Kingbright WP383SURDTK
- LED28: renamed from D28; footprint mr-stuff:WP383SURDTK -> mr-stuff:Kingbright WP383SURDTK
- LED29: renamed from D29; footprint mr-stuff:WP383SURDTK -> mr-stuff:Kingbright WP383SURDTK
- LED3: renamed from D3; footprint mr-stuff:WP383SURDTK -> mr-stuff:Kingbright WP383SURDTK
- LED30: renamed from D30; footprint mr-stuff:WP383SURDTK -> mr-stuff:Kingbright WP383SURDTK
- LED31: renamed from D31; footprint mr-stuff:WP383SURDTK -> mr-stuff:Kingbright WP383SURDTK
- LED32: renamed from D32; footprint mr-stuff:WP383SURDTK -> mr-stuff:Kingbright WP383SURDTK
- LED33: renamed from D33; footprint mr-stuff:WP383SURDTK -> mr-stuff:Kingbright WP383SURDTK
- LED34: renamed from D34; footprint mr-stuff:WP383SURDTK -> mr-stuff:Kingbright WP383SURDTK
- LED35: renamed from D35; footprint mr-stuff:WP383SURDTK -> mr-stuff:Kingbright WP383SURDTK
- LED36: renamed from D36; footprint mr-stuff:WP383SURDTK -> mr-stuff:Kingbright WP383SURDTK
- LED37: renamed from D37; footprint mr-stuff:WP383SURDTK -> mr-stuff:Kingbright WP383SURDTK
- LED38: renamed from D38; footprint mr-stuff:WP383SURDTK -> mr-stuff:Kingbright WP383SURDTK
- LED39: renamed from D39; footprint mr-stuff:WP383SURDTK -> mr-stuff:Kingbright WP383SURDTK
- LED4: renamed from D4; footprint mr-stuff:WP383SURDTK -> mr-stuff:Kingbright WP383SURDTK
- LED40: renamed from D40; footprint mr-stuff:WP383SURDTK -> mr-stuff:Kingbright WP383SURDTK
- LED41: renamed from D41; footprint mr-stuff:WP383SURDTK -> mr-stuff:Kingbright WP383SURDTK
- LED42: renamed from D42; footprint mr-stuff:WP383SURDTK -> mr-stuff:Kingbright WP383SURDTK
- LED43: renamed from D43; footprint mr-stuff:WP383SURDTK -> mr-stuff:Kingbright WP383SURDTK
- LED44: renamed from D44; footprint mr-stuff:WP383SURDTK -> mr-stuff:Kingbright WP383SURDTK
- LED45: renamed from D45; footprint mr-stuff:WP383SURDTK -> mr-stuff:Kingbright WP383SURDTK
- LED46: renamed from D46; footprint mr-stuff:WP383SURDTK -> mr-stuff:Kingbright WP383SURDTK
- LED47: renamed from D47; footprint mr-stuff:WP383SURDTK -> mr-stuff:Kingbright WP383SURDTK
- LED48: renamed from D48; footprint mr-stuff:WP383SURDTK -> mr-stuff:Kingbright WP383SURDTK
- LED49: renamed from D49; footprint mr-stuff:WP383SURDTK -> mr-stuff:Kingbright WP383SURDTK
- LED5: renamed from D5; footprint mr-stuff:WP383SURDTK -> mr-stuff:Kingbright WP383SURDTK
- LED50: renamed from D50; footprint mr-stuff:WP383SURDTK -> mr-stuff:Kingbright WP383SURDTK
- LED51: renamed from D51; footprint mr-stuff:WP383SURDTK -> mr-stuff:Kingbright WP383SURDTK
- LED52: renamed from D52; footprint mr-stuff:WP383SURDTK -> mr-stuff:Kingbright WP383SURDTK
- LED53: renamed from D53; footprint mr-stuff:WP383SURDTK -> mr-stuff:Kingbright WP383SURDTK
- LED54: renamed from D54; footprint mr-stuff:WP383SURDTK -> mr-stuff:Kingbright WP383SURDTK
- LED55: renamed from D55; footprint mr-stuff:WP383SURDTK -> mr-stuff:Kingbright WP383SURDTK
- LED56: renamed from D56; footprint mr-stuff:WP383SURDTK -> mr-stuff:Kingbright WP383SURDTK
- LED57: renamed from D57; footprint mr-stuff:WP383SURDTK -> mr-stuff:Kingbright WP383SURDTK
- LED58: renamed from D58; footprint mr-stuff:WP383SURDTK -> mr-stuff:Kingbright WP383SURDTK
- LED59: renamed from D59; footprint mr-stuff:WP383SURDTK -> mr-stuff:Kingbright WP383SURDTK
- LED6: renamed from D6; footprint mr-stuff:WP383SURDTK -> mr-stuff:Kingbright WP383SURDTK
- LED60: renamed from D60; footprint mr-stuff:WP383SURDTK -> mr-stuff:Kingbright WP383SURDTK
- LED61: renamed from D61; footprint mr-stuff:WP383SURDTK -> mr-stuff:Kingbright WP383SURDTK
- LED62: renamed from D62; footprint mr-stuff:WP383SURDTK -> mr-stuff:Kingbright WP383SURDTK
- LED63: renamed from D63; footprint mr-stuff:WP383SURDTK -> mr-stuff:Kingbright WP383SURDTK
- LED64: renamed from D64; footprint mr-stuff:WP383SURDTK -> mr-stuff:Kingbright WP383SURDTK
- LED65: renamed from D65; footprint mr-stuff:WP383SURDTK -> mr-stuff:Kingbright WP383SURDTK
- LED66: renamed from D66; footprint mr-stuff:WP383SURDTK -> mr-stuff:Kingbright WP383SURDTK
- LED67: renamed from D67; footprint mr-stuff:WP383SURDTK -> mr-stuff:Kingbright WP383SURDTK
- LED68: renamed from D68; footprint mr-stuff:WP383SURDTK -> mr-stuff:Kingbright WP383SURDTK
- LED69: renamed from D69; footprint mr-stuff:WP383SURDTK -> mr-stuff:Kingbright WP383SURDTK
- LED7: renamed from D7; footprint mr-stuff:WP383SURDTK -> mr-stuff:Kingbright WP383SURDTK
- LED70: renamed from D70; footprint mr-stuff:WP383SURDTK -> mr-stuff:Kingbright WP383SURDTK
- LED71: renamed from D71; footprint mr-stuff:WP383SURDTK -> mr-stuff:Kingbright WP383SURDTK
- LED72: renamed from D72; footprint mr-stuff:WP383SURDTK -> mr-stuff:Kingbright WP383SURDTK
- LED73: renamed from D73; footprint mr-stuff:WP383SURDTK -> mr-stuff:Kingbright WP383SURDTK
- LED74: renamed from D74; footprint mr-stuff:WP383SURDTK -> mr-stuff:Kingbright WP383SURDTK
- LED75: renamed from D75; footprint mr-stuff:WP383SURDTK -> mr-stuff:Kingbright WP383SURDTK
- LED76: renamed from D76; footprint mr-stuff:WP383SURDTK -> mr-stuff:Kingbright WP383SURDTK
- LED77: renamed from D77; footprint mr-stuff:WP383SURDTK -> mr-stuff:Kingbright WP383SURDTK
- LED78: renamed from D78; footprint mr-stuff:WP383SURDTK -> mr-stuff:Kingbright WP383SURDTK
- LED79: renamed from D79; footprint mr-stuff:WP383SURDTK -> mr-stuff:Kingbright WP383SURDTK
- LED8: renamed from D8; footprint mr-stuff:WP383SURDTK -> mr-stuff:Kingbright WP383SURDTK
- LED80: renamed from D80; footprint mr-stuff:WP383SURDTK -> mr-stuff:Kingbright WP383SURDTK
- LED81: renamed from D81; footprint mr-stuff:WP383SURDTK -> mr-stuff:Kingbright WP383SURDTK
- LED82: renamed from D82; footprint mr-stuff:WP383SURDTK -> mr-stuff:Kingbright WP383SURDTK
- LED83: renamed from D83; footprint mr-stuff:WP383SURDTK -> mr-stuff:Kingbright WP383SURDTK
- LED84: renamed from D84; footprint mr-stuff:WP383SURDTK -> mr-stuff:Kingbright WP383SURDTK
- LED85: renamed from D85; footprint mr-stuff:WP383SURDTK -> mr-stuff:Kingbright WP383SURDTK
- LED86: renamed from D86; footprint mr-stuff:WP383SURDTK -> mr-stuff:Kingbright WP383SURDTK
- LED87: renamed from D87; footprint mr-stuff:WP383SURDTK -> mr-stuff:Kingbright WP383SURDTK
- LED88: renamed from D88; footprint mr-stuff:WP383SURDTK -> mr-stuff:Kingbright WP383SURDTK
- LED89: renamed from D89; footprint mr-stuff:WP383SURDTK -> mr-stuff:Kingbright WP383SURDTK
- LED9: renamed from D9; footprint mr-stuff:WP383SURDTK -> mr-stuff:Kingbright WP383SURDTK
- LED90: renamed from D90; footprint mr-stuff:WP383SURDTK -> mr-stuff:Kingbright WP383SURDTK
- R1, R18, R2, R4: value 10K -> 10k; footprint Resistor_THT:R_Axial_DIN0207_L6.3mm_D2.5mm_P7.62mm_Horizontal -> mr-stuff:Stackpole RMCA0805; moved to F.Cu
- R10, R6, R8: value 4.7K -> 10k; footprint Resistor_THT:R_Axial_DIN0207_L6.3mm_D2.5mm_P7.62mm_Horizontal -> mr-stuff:Stackpole RMCA0805; moved to F.Cu
- R11: value 3.3K -> 1k; footprint Resistor_THT:R_Axial_DIN0207_L6.3mm_D2.5mm_P7.62mm_Horizontal -> mr-stuff:Stackpole RNCP0805; moved to F.Cu
- R12: value 10K -> 100k; footprint Resistor_THT:R_Axial_DIN0207_L6.3mm_D2.5mm_P7.62mm_Horizontal -> mr-stuff:Stackpole RMCA0805; moved to F.Cu
- R13: value 147 -> 68.1; footprint Resistor_THT:R_Axial_DIN0207_L6.3mm_D2.5mm_P7.62mm_Horizontal -> mr-stuff:Stackpole RNCP0805; moved to F.Cu
- R14: value 1K -> 10k; footprint Resistor_THT:R_Axial_DIN0207_L6.3mm_D2.5mm_P7.62mm_Horizontal -> mr-stuff:Stackpole RMCA0805; moved to F.Cu
- R15: value 10K -> 1k; footprint Resistor_THT:R_Axial_DIN0207_L6.3mm_D2.5mm_P7.62mm_Horizontal -> mr-stuff:Stackpole RNCP0805; moved to F.Cu
- R16: value 63.4 -> 100k; footprint Resistor_THT:R_Axial_DIN0207_L6.3mm_D2.5mm_P7.62mm_Horizontal -> mr-stuff:Stackpole RMCA0805; moved to F.Cu
- R17: value 1K -> 68.1; footprint Resistor_THT:R_Axial_DIN0207_L6.3mm_D2.5mm_P7.62mm_Horizontal -> mr-stuff:Stackpole RNCP0805; moved to F.Cu
- R19: value 63.4 -> 1k; footprint Resistor_THT:R_Axial_DIN0207_L6.3mm_D2.5mm_P7.62mm_Horizontal -> mr-stuff:Stackpole RNCP0805; moved to F.Cu
- R20: value 1K -> 100k; footprint Resistor_THT:R_Axial_DIN0207_L6.3mm_D2.5mm_P7.62mm_Horizontal -> mr-stuff:Stackpole RMCA0805; moved to F.Cu
- R21: value 475 -> 200K; footprint Resistor_THT:R_Axial_DIN0207_L6.3mm_D2.5mm_P7.62mm_Horizontal -> mr-stuff:Yageo AE0805; moved to F.Cu
- R22, R23: value 475 -> 4.7k; footprint Resistor_THT:R_Axial_DIN0207_L6.3mm_D2.5mm_P7.62mm_Horizontal -> mr-stuff:Stackpole RMCA0805; moved to F.Cu
- R24: value 3.3K -> 4.7k; footprint Resistor_THT:R_Axial_DIN0207_L6.3mm_D2.5mm_P7.62mm_Horizontal -> mr-stuff:Stackpole RMCA0805; moved to F.Cu
- R25: value 3.3K -> 20k; footprint Resistor_THT:R_Axial_DIN0207_L6.3mm_D2.5mm_P7.62mm_Horizontal -> mr-stuff:Stackpole RMCA0805; moved to F.Cu
- R26, R27: value 3.3K -> 3.3k; footprint Resistor_THT:R_Axial_DIN0207_L6.3mm_D2.5mm_P7.62mm_Horizontal -> mr-stuff:Stackpole RNCF0805; moved to F.Cu
- R3, R5: value 10K -> 475; footprint Resistor_THT:R_Axial_DIN0207_L6.3mm_D2.5mm_P7.62mm_Horizontal -> mr-stuff:Stackpole RNCP0805; moved to F.Cu
- R7: value 4.7K -> 475; footprint Resistor_THT:R_Axial_DIN0207_L6.3mm_D2.5mm_P7.62mm_Horizontal -> mr-stuff:Stackpole RNCP0805; moved to F.Cu
- R9: value 100K -> 147; footprint Resistor_THT:R_Axial_DIN0207_L6.3mm_D2.5mm_P7.62mm_Horizontal -> mr-stuff:Stackpole RNCP0805; moved to F.Cu
- TDM***: moved to F.Cu
- TP1: value TP_VRAW -> Ship Power; footprint Connector_PinHeader_2.54mm:PinHeader_1x01_P2.54mm_Vertical -> Connector_PinHeader_2.54mm:PinHeader_1x03_P2.54mm_Vertical; moved to F.Cu
- TP2: value GND_SHIP -> Board Power; footprint Connector_PinHeader_2.54mm:PinHeader_1x01_P2.54mm_Vertical -> Connector_PinHeader_2.54mm:PinHeader_1x03_P2.54mm_Vertical; moved to F.Cu
- TP3: value N2K_TX -> IS31 I2C; footprint Connector_PinHeader_2.54mm:PinHeader_1x01_P2.54mm_Vertical -> Connector_PinHeader_2.54mm:PinHeader_1x02_P2.54mm_Vertical; moved to F.Cu
- TP4: value N2K_RX -> Board I2C; footprint Connector_PinHeader_2.54mm:PinHeader_1x01_P2.54mm_Vertical -> Connector_PinHeader_2.54mm:PinHeader_1x02_P2.54mm_Vertical; moved to F.Cu
- TVS1: value PESD3V3L1BA -> SMBJ20A-Q; footprint Diode_SMD:D_SOD-323 -> mr-stuff:Bourns SMBJ20; moved to F.Cu
- TVS2: value PESD3V3L1BA -> PESD2CANFD54VT-QR; footprint Diode_SMD:D_SOD-323 -> mr-stuff:Nexperia PESD2CANFD; moved to F.Cu
- TVS3, TVS4: value PESD3V3L1BA -> TPD2E2U06QDBZRQ1; footprint Diode_SMD:D_SOD-323 -> mr-stuff:TI TPD2E2U06; moved to F.Cu
- moved C23 218.8 mm to (268.0, 108.1)
- moved C24 217.7 mm to (268.0, 111.3)
- moved TP4 208.8 mm to (244.1, 105.8)
- moved TP3 199.7 mm to (239.5, 105.8)
- moved R20 185.6 mm to (230.4, 89.4), turned to 0 degrees
- moved R18 184.2 mm to (230.4, 86.3), turned to 0 degrees
- moved TVS2 178.6 mm to (210.1, 81.5), turned to 0 degrees
- moved R25 176.8 mm to (230.4, 101.8)
- moved R4 175.7 mm to (225.8, 89.4)
- moved R22 173.0 mm to (230.4, 92.5), turned to 0 degrees
- moved R16 172.7 mm to (230.4, 83.2), turned to 0 degrees
- moved C1 172.6 mm to (216.6, 80.1), turned to 0 degrees
- moved R3 170.6 mm to (196.7, 80.7)
- moved R21 170.1 mm to (209.9, 92.4), turned to 0 degrees
- moved R27 167.0 mm to (205.5, 80.7), turned to 0 degrees
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Connections:
- C1 pad 1: +3.3V -> GND
- C1 pad 2: GND -> +3.3V
- C10 pad 1: +3.3V -> V_RAW
- C10 pad 2: GND -> GND_SHIP
- C11 pad 1: +3.3V -> GND_SHIP
- C13 pad 1: +5V -> GND
- C13 pad 2: GND -> +5V
- C14 pad 1: +5V -> GND
- C14 pad 2: GND -> +3.3V
- C15 pad 1: +5V -> Net-(RST1-C1-)
- C15 pad 2: GND -> Net-(RST1-C1+)
- C16 pad 1: +5V -> Net-(RST1-VS+)
- C16 pad 2: GND -> +3.3V
- C17 pad 1: +5V -> GND
- C17 pad 2: GND -> +3.3V
- C18 pad 2: GND -> Net-(RST1-C2+)
- C19 pad 1: Net-(U5-C1+) -> GND
- C2 pad 1: +5V_SHIP -> GND_SHIP
- C2 pad 2: GND_SHIP -> +5V_SHIP
- C20 pad 1: Net-(U5-C2+) -> GND
- C20 pad 2: Net-(U5-C2-) -> /LCD_PGUP_IN
- C21 pad 1: +3.3V -> GND
- C21 pad 2: Net-(U5-VS+) -> /LCD_PGDOWN_IN
- C22 pad 1: Net-(U5-VS-) -> GND
- C22 pad 2: GND -> /DISPLAY_ON_IN
- C23 pad 1: +3.3V -> GND
- C23 pad 2: GND -> Net-(LS1-EN)
- C24 pad 1: +3.3V -> GND
- C24 pad 2: GND -> Net-(LS1-EN)
- C25 pad 1: /BRIGHTNESS_POT_IN -> +5V
- C26 pad 1: /LCD_PGUP_IN -> +5V
- C27 pad 1: /LCD_PGDOWN_IN -> +5V
- C28 pad 1: /DISPLAY_ON_IN -> +5V
- C3 pad 1: V_RAW -> +3.3V
- C3 pad 2: GND_SHIP -> GND
- C4 pad 1: +5V -> GND
- C4 pad 2: Net-(PS1-+VIN) -> +3.3V
- C5 pad 1: GND_SHIP -> GND
- C5 pad 2: GND -> /NRST
- C6 pad 1: V_RAW -> /OSC_IN
- C6 pad 2: GND_SHIP -> GND
- C7 pad 1: +5V_SHIP -> GND
- C7 pad 2: GND_SHIP -> /OSC_OUT
- C8 pad 1: +5V -> GND_SHIP
- C8 pad 2: GND -> V_RAW
- C9 pad 1: +3.3V -> GND_SHIP
- C9 pad 2: GND -> +5V_SHIP
- DE1 pad 1: GND -> unconnected-(DE1-Pad1)
- DE1 pad 2: unconnected-(DE1-Pad2) -> /RS232_TX
- DE1 pad 3: Net-(U5-R1IN) -> /RS232_RX
- DE1 pad 4: Net-(U5-T1OUT) -> unconnected-(DE1-Pad4)
- DE1 pad 5: unconnected-(DE1-Pad5) -> GND
- DE2 pad 1: GND -> unconnected-(DE2-Pad1)
- DE2 pad 2: +3.3V -> unconnected-(DE2-Pad2)
- DE2 pad 6: /BRIGHTNESS_POT_IN_PLUG -> unconnected-(DE2-Pad6)
- DE2 pad 7: unconnected-(DE2-Pad7) -> GND
- R1 pad 1: +3.3V -> /NRST
- R1 pad 2: /NRST -> +3.3V
- R10 pad 2: GND -> +5V
- R11 pad 1: Net-(U4-R_EXT) -> /LCD_BL_RED_OUT
- R11 pad 2: GND -> Net-(Q8-G)
- R12 pad 1: +5V -> GND
- R12 pad 2: Net-(Q1-G) -> Net-(Q8-G)
- R14 pad 2: /LCD_BL_RED_OUT -> +5V
- R15 pad 1: +5V -> /LCD_BL_GREEN_OUT
- R15 pad 2: Net-(Q3-G) -> Net-(Q10-G)
- R16 pad 1: Net-(Q3-D) -> GND
- R16 pad 2: Net-(LCD1-A-GREEN) -> Net-(Q10-G)
- R17 pad 2: /LCD_BL_GREEN_OUT -> Net-(LCD2-A-BLUE)
- R18 pad 1: +5V -> Net-(Q11-G)
- R18 pad 2: Net-(Q5-G) -> +5V
- R19 pad 1: Net-(Q5-D) -> /LCD_BL_BLUE_OUT
- R19 pad 2: Net-(LCD1-A-BLUE) -> Net-(Q12-G)
- R20 pad 1: Net-(Q6-B) -> GND
- R20 pad 2: /LCD_BL_BLUE_OUT -> Net-(Q12-G)
- R21 pad 1: /LCD_PGUP_IN_PLUG -> Net-(LS1-EN)
- R21 pad 2: /LCD_PGUP_IN -> +5V
- R22 pad 1: /LCD_PGDOWN_IN_PLUG -> Net-(LCD2-SCL)
- R22 pad 2: /LCD_PGDOWN_IN -> +5V
- R23 pad 1: /DISPLAY_ON_IN_PLUG -> Net-(LCD2-SDA)
- R23 pad 2: /DISPLAY_ON_IN -> +5V
- R24 pad 1: +3.3V -> /IS31_INTB_OUT
- R24 pad 2: /IS31_I2C_SDA -> +3.3V
- R25 pad 1: +3.3V -> GND
- R25 pad 2: /IS31_I2C_SCL -> Net-(CPD1-R_EXT)
- R26 pad 1: +3.3V -> /IS31_I2C_SDA
- R26 pad 2: /BOARD_I2C_SDA -> +3.3V
- R27 pad 1: +3.3V -> /IS31_I2C_SCL
- R27 pad 2: /BOARD_I2C_SCL -> +3.3V
- R3 pad 1: /LCD_PGUP_IN -> /LCD_PGUP_IN_PLUG
- R3 pad 2: +3.3V -> /LCD_PGUP_IN
- R4 pad 1: /LCD_PGDOWN_IN -> +3.3V
- R4 pad 2: +3.3V -> /LCD_PGUP_IN
- R5 pad 1: /DISPLAY_ON_IN -> /LCD_PGDOWN_IN_PLUG
- R5 pad 2: +3.3V -> /LCD_PGDOWN_IN
- R6 pad 1: +5V -> +3.3V
- R6 pad 2: /IS31_INTB_OUT -> /LCD_PGDOWN_IN
- R7 pad 1: +3.3V -> /DISPLAY_ON_IN_PLUG
- R7 pad 2: /IS31_I2C_SCL -> /DISPLAY_ON_IN
- R8 pad 2: /IS31_I2C_SDA -> /DISPLAY_ON_IN
- R9 pad 1: /IS31_SHUTDOWN_OUT -> Net-(Q7-D)
- R9 pad 2: GND -> Net-(LCD2-A-RED)
- TP1 pad 1: V_RAW -> +5V_SHIP
- TP2 pad 1: GND_SHIP -> +3.3V
- TP3 pad 1: /N2K_TX -> /IS31_I2C_SDA
- TP4 pad 1: /N2K_RX -> /BOARD_I2C_SDA
- TVS1 pad 1: /BRIGHTNESS_POT_IN_PLUG -> Net-(SD1-A)
- TVS1 pad 2: GND -> GND_SHIP
- TVS2 pad 1: /LCD_PGUP_IN_PLUG -> /N2K_CAN_H
- TVS2 pad 2: GND -> /N2K_CAN_L
- TVS3 pad 1: /LCD_PGDOWN_IN_PLUG -> /LCD_PGUP_IN_PLUG
- TVS3 pad 2: GND -> /LCD_PGDOWN_IN_PLUG
- TVS4 pad 2: GND -> unconnected-(TVS4-IO2-Pad2)
Routing:
- net GND_SHIP: track 564.8 -> 8.02 mm, vias 6 -> 0
- net +5V: track 455.1 -> 0.00 mm
- net /LCD_PGUP_IN: track 262.0 -> 0.00 mm, vias 1 -> 0
- net /LCD_PGDOWN_IN: track 250.0 -> 0.00 mm, vias 1 -> 0
- net /DISPLAY_ON_IN: track 236.1 -> 0.00 mm, vias 1 -> 0
- net /LCD_BL_RED_OUT: track 220.7 -> 0.00 mm, vias 1 -> 0
- net +5V_SHIP: track 204.0 -> 0.00 mm, vias 29 -> 0
- net /LCD_BL_GREEN_OUT: track 200.8 -> 0.00 mm, vias 1 -> 0
- net +3.3V: track 194.1 -> 0.00 mm, vias 26 -> 0
- net /BRIGHTNESS_POT_IN: track 184.5 -> 0.00 mm, vias 2 -> 0
- net /BOARD_I2C_SCL: track 183.9 -> 0.00 mm, vias 4 -> 0
- net /BOARD_I2C_SDA: track 180.2 -> 0.00 mm, vias 3 -> 0
- net /LCD_BL_BLUE_OUT: track 179.8 -> 0.00 mm, vias 1 -> 0
- net V_RAW: track 137.6 -> 0.00 mm, vias 1 -> 0
- net /IS31_I2C_SDA: track 132.4 -> 0.00 mm, vias 2 -> 0
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- removed copper zone on B.Cu, net +3.3V
- removed copper zone on F.Cu, net +3.3V
- removed copper zone on B.Cu, net +5V_SHIP
- removed copper zone on F.Cu, net +5V_SHIP
Other:
- board text removed: "+3.3V"
- board text removed: "+5V"
- board text removed: "+5V_SHIP"
- board text removed: "-=] DE1 1 - Gnd 2 - nc 3 - RX 4 - TX 5~9 - nc"
- board text removed: "-=] DE2 1 - Gnd (Brightness Pot) 2 - 3.3V (Brightness Pot) 3 - Display On Switch 4 - LCD Page Down Switch 5 - LCD Page Up Switch 6 - Brightness Pot 7 - nc 8 - Gnd (Display On) 9 - Gnd (LCD Paging)"
- board text removed: "-=] Program Header"
- board text removed: "1"
- board text removed: "1 - NRST 2 - 3.3V 3 - SWDIO 4 - SWCLK 5 - Gnd"
- board text removed: "5"
- board text removed: "6"
- board text removed: "64KiB 0x55h"
- board text removed: "64KiB 0x57h"
- board text removed: "9"
- board text removed: "Board SCL"
- board text removed: "Board SDA"
- board text removed: "Boot"
- board text removed: "DE1"
- board text removed: "GND"
- board text removed: "GND_SHIP"
- board text removed: "IS31 SCL"
- board text removed: "IS31 SDA"
- board text removed: "N2K_RX"
- board text removed: "N2K_TX"
- board text removed: "NHD-0216K3Z-NS(RGB)-FBW-V3"
- board text removed: "NMEA2000 2x12 + 5x48 Battery Module v4 - Prototype - 01 © The Digital Mermaid - 2025"
- board text removed: "RS-232"
- board text removed: "RS232 115,200 baud"
- board text removed: "Reset"
- board text removed: "V_RAW"
- board text removed: "v4.0"
