File: Full Boards/Battery Display/Battery Display.kicad_pcb (KiCad board)
At the start: 4 copper layers, 110 x 175.2 mm, 195 parts, among them J3 Program Header, J4 Optional Bond, Q1 BSS314PE, Q2 DMN6075S, Q3 BSS314PE, Q4 DMN6075S, Q5 BSS314PE, Q6 DMN6075S, SW1 Boot, SW2 Reset

Commit message: Enabled additional tests and fixed some cosmetic / silkscreen issues.
Signed-off-by: digimer <digital.mermaid@gmail.com>
Parts:
- moved C11 0.10 mm to (47.1, 47.9)
Changed lines of the file:
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@@
 		(capping no)
 		(filling no)
+		(zone_defaults)
 		(pcbplotparams
 			(layerselection 0x00000000_00000000_55555555_575555ff)
@@
 		(tags "08051C105K4Z2A ")
 		(property "Reference" "C22"
-			(at 0 -2 270)
+			(at 3.1 0.1 90)
 			(unlocked yes)
 			(layer "F.SilkS")
@@
 		)
 	)
+	(footprint "mr-stuff:Knowles Syfer 2211JA25"
+		(layer "F.Cu")
+		(at 47.1 47.9 -90)
+		(property "Reference" "C11"
+			(at 0 -2.375 90)
+			(unlocked yes)
+			(layer "F.SilkS")
+			(effects
+				(font
+					(size 1 1)
+					(thickness 0.15)
+				)
+			)
+		)
+		(property "Value" "1nF"
+			(at 0 2.7 270)
+			(unlocked yes)
+			(layer "F.Fab")
+			(effects
+				(font
+					(size 1 1)
+					(thickness 0.15)
+				)
+			)
+		)
+		(property "Datasheet" "https://mm.digikey.com/Volume0/opasdata/d220001/medias/docus/3001/2211JA250102JKTSYX.pdf"
+			(at 0 0 270)
+			(unlocked yes)
+			(layer "F.Fab")
+			(hide yes)
+			(effects
+				(font
+					(size 1 1)
+					(thickness 0.15)
+				)
+			)
+		)
+		(property "Description" "1000 pF ±5% 250VAC Ceramic Capacitor C0G, NP0 (1B) 2211 (5728 Metric)"
+			(at 0 0 270)
+			(unlocked yes)
+			(layer "F.Fab")
+			(hide yes)
+			(effects
+				(font
+					(size 1 1)
+					(thickness 0.15)
+				)
+			)
+		)
+		(property "Part" "Knowles Syfer 2211JA250102JKTSYX"
+			(at 0 0 270)
+			(unlocked yes)
+			(layer "F.Fab")
+			(hide yes)
+			(effects
+				(font
+					(size 1 1)
+					(thickness 0.15)
+				)
+			)
+		)
+		(property ki_fp_filters "C_*")
+		(sheetname "/")
+		(sheetfile "Battery Display.kicad_sch")
+		(units
+			(unit
+				(name "A")
+				(pins "1" "2")
+			)
+		)
+		(attr smd dnp)
+		(duplicate_pad_numbers_are_jumpers no)
+		(fp_line
+			(start -1.431496 1.5)
+			(end 1.4 1.5)
+			(stroke
+				(width 0.12)
+				(type solid)
+			)
+			(layer "F.SilkS")
+		)
+		(fp_line
+			(start -1.431496 -1.5)
+			(end 1.4 -1.5)
+			(stroke
+				(width 0.12)
+				(type solid)
+			)
+			(layer "F.SilkS")
+		)
+		(fp_rect
+			(start -3.25 -1.75)
+			(end 3.25 1.75)
+			(stroke
+				(width 0.05)
+				(type solid)
+			)
+			(fill no)
+			(layer "F.CrtYd")
+		)
+		(fp_rect
+			(start -2.5 -1.5)
+			(end 2.5 1.5)
+			(stroke
+				(width 0.1)
+				(type solid)
+			)
+			(fill no)
+			(layer "F.Fab")
+		)
+		(fp_text user "${REFERENCE}"
+			(at 0 4.4 270)
+			(unlocked yes)
+			(layer "F.Fab")
+			(effects
+				(font
+					(size 1 1)
+					(thickness 0.15)
+				)
+			)
+		)
+		(pad "1" smd roundrect
+			(at -2.5 0 270)
+			(size 1.5 3)
+			(layers "F.Cu" "F.Mask" "F.Paste")
+			(roundrect_rratio 0.15)
+			(net "GND_SHIP")
+			(pintype "passive")
+		)
+		(pad "2" smd roundrect
+			(at 2.5 0 270)
+			(size 1.5 3)
+			(layers "F.Cu" "F.Mask" "F.Paste")
+			(roundrect_rratio 0.15)
+			(net "GND")
+			(pintype "passive")
+		)
+		(embedded_fonts no)
+	)
 	(footprint "mr-stuff:Stackpole RMCA0805"
 		(layer "F.Cu")
@@
 		(tags "08051C105K4Z2A ")
 		(property "Reference" "C29"
-			(at 0 -2 270)
+			(at -3.2 -0.1 90)
 			(unlocked yes)
 			(layer "F.SilkS")
@@
 		)
 	)
-	(footprint "mr-stuff:Knowles Syfer 2211JA25"
-		(layer "F.Cu")
-		(at 47.2 47.9 -90)
-		(property "Reference" "C11"
-			(at 4.2 0 0)
-			(unlocked yes)
-			(layer "F.SilkS")
-			(effects
-				(font
-					(size 1 1)
-					(thickness 0.15)
-				)
-			)
-		)
-		(property "Value" "1nF"
-			(at 0 2.7 270)
-			(unlocked yes)
-			(layer "F.Fab")
-			(effects
-				(font
-					(size 1 1)
-					(thickness 0.15)
-				)
-			)
-		)
-		(property "Datasheet" "https://mm.digikey.com/Volume0/opasdata/d220001/medias/docus/3001/2211JA250102JKTSYX.pdf"
-			(at 0 0 270)
-			(unlocked yes)
-			(layer "F.Fab")
-			(hide yes)
-			(effects
-				(font
-					(size 1 1)
-					(thickness 0.15)
-				)
-			)
-		)
-		(property "Description" "1000 pF ±5% 250VAC Ceramic Capacitor C0G, NP0 (1B) 2211 (5728 Metric)"
-			(at 0 0 270)
-			(unlocked yes)
-			(layer "F.Fab")
-			(hide yes)
-			(effects
-				(font
-					(size 1 1)
-					(thickness 0.15)
-				)
-			)
-		)
-		(property "MANUFACTURER" ""
-			(at 0 0 270)
-			(unlocked yes)
-			(layer "F.Fab")
-			(hide yes)
-			(effects
-				(font
-					(size 1 1)
-					(thickness 0.15)
-				)
-			)
-		)
-		(property "MAXIMUM_PACKAGE_HEIGHT" ""
-			(at 0 0 270)
-			(unlocked yes)
-			(layer "F.Fab")
-			(hide yes)
-			(effects
-				(font
-					(size 1 1)
-					(thickness 0.15)
-				)
-			)
-		)
-		(property "PARTREV" ""
-			(at 0 0 270)
-			(unlocked yes)
-			(layer "F.Fab")
-			(hide yes)
-			(effects
-				(font
-					(size 1 1)
-					(thickness 0.15)
-				)
-			)
-		)
-		(property "STANDARD" ""
-			(at 0 0 270)
-			(unlocked yes)
-			(layer "F.Fab")
-			(hide yes)
-			(effects
-				(font
-					(size 1 1)
-					(thickness 0.15)
-				)
-			)
-		)
-		(property ki_fp_filters "C_*")
-		(sheetname "/")
-		(sheetfile "Battery Display.kicad_sch")
-		(units
-			(unit
-				(name "A")
-				(pins "1" "2")
-			)
-		)
-		(attr smd dnp)
-		(duplicate_pad_numbers_are_jumpers no)
-		(fp_line
-			(start -1.431496 1.5)
-			(end 1.4 1.5)
-			(stroke
-				(width 0.12)
-				(type solid)
-			)
-			(layer "F.SilkS")
-		)
-		(fp_line
-			(start -1.431496 -1.5)
-			(end 1.4 -1.5)
-			(stroke
-				(width 0.12)
-				(type solid)
-			)
-			(layer "F.SilkS")
-		)
-		(fp_rect
-			(start -3.25 -1.75)
-			(end 3.25 1.75)
-			(stroke
-				(width 0.05)
-				(type solid)
-			)
-			(fill no)
-			(layer "F.CrtYd")
-		)
-		(fp_rect
-			(start -2.5 -1.5)
-			(end 2.5 1.5)
-			(stroke
-				(width 0.1)
-				(type solid)
-			)
-			(fill no)
-			(layer "F.Fab")
-		)
-		(fp_text user "${REFERENCE}"
-			(at 0 4.4 270)
-			(unlocked yes)
-			(layer "F.Fab")
-			(effects
-				(font
-					(size 1 1)
-					(thickness 0.15)
-				)
-			)
-		)
-		(pad "1" smd roundrect
-			(at -2.5 0 270)
-			(size 1.5 3)
-			(layers "F.Cu" "F.Mask" "F.Paste")
-			(roundrect_rratio 0.15)
-			(net "GND_SHIP")
-			(pintype "passive")
-		)
-		(pad "2" smd roundrect
-			(at 2.5 0 270)
-			(size 1.5 3)
-			(layers "F.Cu" "F.Mask" "F.Paste")
-			(roundrect_rratio 0.15)
-			(net "GND")
-			(pintype "passive")
-		)
-		(embedded_fonts no)
-	)
 	(footprint "mr-stuff:Kingbright WP383SURDTK"
 		(layer "F.Cu")
@@
 		(tags "08051C105K4Z2A ")
 		(property "Reference" "C17"
-			(at 0 -2 90)
+			(at 3.1 -0.015896 90)
 			(unlocked yes)
 			(layer "F.SilkS")
@@
 		(tags "08051C105K4Z2A ")
 		(property "Reference" "C30"
-			(at 0 -2 90)
+			(at 3 0 90)
 			(unlocked yes)
 			(layer "F.SilkS")
@@
 		(tags "08051C105K4Z2A ")
 		(property "Reference" "C32"
-			(at 0 -2 270)
+			(at 0 1.6 90)
 			(unlocked yes)
 			(layer "F.SilkS")
@@
 		(tags "08051C105K4Z2A ")
 		(property "Reference" "C31"
-			(at 0 -2 270)
+			(at 0 1.6 90)
 			(unlocked yes)
 			(layer "F.SilkS")
@@
 		(tags "08051C105K4Z2A ")
 		(property "Reference" "C2"
-			(at 0 -2 90)
+			(at 0 1.7017 90)
 			(unlocked yes)
 			(layer "F.SilkS")
@@
 		(tags "08051C105K4Z2A ")
 		(property "Reference" "C21"
-			(at 0 -2 270)
+			(at 3.1 0 90)
 			(unlocked yes)
 			(layer "F.SilkS")
@@
 		(tags "08051C105K4Z2A ")
 		(property "Reference" "C20"
-			(at 0 -2 270)
+			(at 3.1 0 90)
 			(unlocked yes)
 			(layer "F.SilkS")
@@
 	)
 	(segment
+		(start 45.6 41.54)
+		(end 47.1 40.04)
+		(width 0.4)
+		(layer "F.Cu")
+		(net "GND_SHIP")
+	)
+	(segment
+		(start 47.1 45.4)
+		(end 47.1 45.3)
+		(width 0.4)
+		(layer "F.Cu")
+		(net "GND_SHIP")
+	)
+	(segment
 		(start 59.5 68.8)
 		(end 58.3155 69.9845)
@@
 	)
 	(segment
-		(start 45.6 41.54)
-		(end 47.1 40.04)
+		(start 45.6 43.8)
+		(end 45.6 41.54)
 		(width 0.4)
 		(layer "F.Cu")
@@
 	)
 	(segment
+		(start 47.1 45.3)
+		(end 45.6 43.8)
+		(width 0.4)
+		(layer "F.Cu")
+		(net "GND_SHIP")
+	)
+	(segment
 		(start 70.1 68.9)
 		(end 73.482 72.282)
@@
 	)
 	(segment
-		(start 45.6 43.8)
-		(end 45.6 41.54)
-		(width 0.4)
-		(layer "F.Cu")
-		(net "GND_SHIP")
-	)
-	(segment
 		(start 88.36 26.7)
 		(end 88.36 31.765)
@@
 	)
 	(segment
-		(start 47.2 45.4)
-		(end 45.6 43.8)
-		(width 0.4)
-		(layer "F.Cu")
-		(net "GND_SHIP")
-	)
-	(segment
 		(start 73.482 76.9197)
 		(end 73.0017 77.4)
@@
 	)
 	(segment
-		(start 47.2 50.4)
-		(end 49.5 50.4)
-		(width 0.4)
-		(layer "F.Cu")
-		(net "GND")
-	)
-	(segment
 		(start 126.4 35.549999)
 		(end 126.4 27.995)
@@
 		(layer "F.Cu")
 		(net "GND")
+	)
+	(segment
+		(start 47.1 50.4)
+		(end 49.5 50.4)
+		(width 0.4)
+		(layer "F.Cu")
+		(net "GND")
