File: Full Boards/Battery Display/Battery Display.kicad_sch (KiCad schematic)
At the start: 194 parts, among them J3 Program Header, J4 Optional Bond, Q10 DMN6075S, Q11 BSS314PE, Q12 DMN6075S, Q7 BSS314PE, Q8 DMN6075S, Q9 BSS314PE, SW3 Boot, SW4 Reset

Commit message: Updated annotation.
Signed-off-by: digimer <digital.mermaid@gmail.com>
Parts:
- renumbered C30 to C1, C49 to C10, C50 to C11, C57 to C13, C59 to C14, C31 to C15, C34 to C16, C43 to C17, C33 to C18, C36 to C19, C42 to C2, C53 to C20, C54 to C21, C52 to C22, C51 to C23, C55 to C24, C29 to C25, C32 to C26, C35 to C27, C38 to C28, C39 to C29, C45 to C3, C37 to C30, C40 to C31, C41 to C32, C46 to C4, C47 to C5, C56 to C6, C58 to C7, C44 to C8, C48 to C9, R34 to R1, R39 to R10, R36 to R11, R38 to R12, R40 to R13, R43 to R14, R41 to R15, R42 to R16, R44 to R17, R47 to R18, R45 to R19, R37 to R2, R46 to R20, R51 to R21, R52 to R22, R53 to R23, R28 to R24, R29 to R25, R31 to R26, R33 to R27, R30 to R28, R32 to R29, R48 to R3, R54 to R4, R49 to R5, R55 to R6, R50 to R7, R56 to R8, R35 to R9, TP14 to TP1, TP17 to TP2, TP16 to TP3, TP15 to TP4, TVS5 to TVS1, TVS6 to TVS2, TVS7 to TVS3, TVS8 to TVS4

Commit message: Finished layout of the battery display PCB. Updated the silkscreen on the Compass Rose as well.
Signed-off-by: digimer <digital.mermaid@gmail.com>
Parts:
- DE2: footprint mr-stuff:Amphenol_L777SDE09PA4CH4F -> mr-stuff:Amphenol L777SDE09PA4CH4F
- renumbered LCD2 to LCD1, Q7 to Q1, Q8 to Q2, Q9 to Q3, Q10 to Q4, Q11 to Q5, Q12 to Q6, SW3 to SW1, SW4 to SW2
Connections:
- net +3.3V: now also R24.1; no longer R24.2
- net IS31_INTB_OUT: now also R24.2; no longer R24.1
Other:
- note added: "C11 provided for optional Common Mode EMI suppression If used: Knowles Syfer 2211JA250102JKTSYX"
- note removed: "C6 provided for optional Common Mode EMI suppression If used: Knowles Syfer 2211JA250102JKTSYX"
- moved on the sheet: R24
Changed lines of the file:
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@@
 		)
 	)
-	(text "C6 provided for optional \nCommon Mode EMI suppression\nIf used: Knowles Syfer 2211JA250102JKTSYX"
+	(text "C11 provided for optional \nCommon Mode EMI suppression\nIf used: Knowles Syfer 2211JA250102JKTSYX"
 		(exclude_from_sim no)
 		(at 190.246 106.934 0)
@@
 		(in_pos_files yes)
 		(dnp no)
-		(property "Reference" "SW4"
+		(property "Reference" "SW2"
 			(at 278.13 120.396 0)
 			(show_name no)
@@
 			(project "Battery Display"
 				(path "/66b9b57f-ad5a-4774-9c04-72011a45113c"
-					(reference "SW4")
+					(reference "SW2")
 					(unit 1)
 				)
@@
 			)
 		)
-		(property "Footprint" "mr-stuff:Amphenol_L777SDE09PA4CH4F"
+		(property "Footprint" "mr-stuff:Amphenol L777SDE09PA4CH4F"
 			(at 264.16 195.072 0)
 			(hide yes)
@@
 		(in_pos_files yes)
 		(dnp no)
-		(property "Reference" "Q10"
+		(property "Reference" "Q4"
 			(at 48.26 200.152 0)
 			(show_name no)
@@
 			(project "Battery Display"
 				(path "/66b9b57f-ad5a-4774-9c04-72011a45113c"
-					(reference "Q10")
+					(reference "Q4")
 					(unit 1)
 				)
@@
 		(in_pos_files yes)
 		(dnp no)
-		(property "Reference" "SW3"
+		(property "Reference" "SW1"
 			(at 278.13 111.506 0)
 			(show_name no)
@@
 			(project "Battery Display"
 				(path "/66b9b57f-ad5a-4774-9c04-72011a45113c"
-					(reference "SW3")
+					(reference "SW1")
 					(unit 1)
 				)
@@
 	(symbol
 		(lib_id "Device:R")
-		(at 177.8 185.42 270)
+		(at 177.8 185.42 90)
 		(unit 1)
 		(body_style 1)
@@
 		(dnp no)
 		(property "Reference" "R24"
-			(at 176.276 185.42 90)
+			(at 179.578 185.42 90)
 			(show_name no)
 			(do_not_autoplace no)
@@
 		)
 		(property "Value" "4.7k"
-			(at 176.022 187.706 90)
+			(at 179.832 187.452 90)
 			(show_name no)
 			(do_not_autoplace no)
@@
 		)
 		(property "Footprint" "mr-stuff:Stackpole RMCA0805"
-			(at 177.8 183.642 90)
+			(at 177.8 187.198 90)
 			(hide yes)
 			(show_name no)
@@
 		(in_pos_files yes)
 		(dnp no)
-		(property "Reference" "Q12"
+		(property "Reference" "Q6"
 			(at 67.31 200.152 0)
 			(show_name no)
@@
 			(project "Battery Display"
 				(path "/66b9b57f-ad5a-4774-9c04-72011a45113c"
-					(reference "Q12")
+					(reference "Q6")
 					(unit 1)
 				)
@@
 		(in_pos_files yes)
 		(dnp no)
-		(property "Reference" "LCD2"
+		(property "Reference" "LCD1"
 			(at 69.85 179.07 0)
 			(show_name no)
@@
 			(project "Battery Display"
 				(path "/66b9b57f-ad5a-4774-9c04-72011a45113c"
-					(reference "LCD2")
+					(reference "LCD1")
 					(unit 1)
 				)
@@
 		(in_pos_files yes)
 		(dnp no)
-		(property "Reference" "Q11"
+		(property "Reference" "Q5"
 			(at 62.992 194.056 0)
 			(show_name no)
@@
 			(project "Battery Display"
 				(path "/66b9b57f-ad5a-4774-9c04-72011a45113c"
-					(reference "Q11")
+					(reference "Q5")
 					(unit 1)
 				)
@@
 		(in_pos_files yes)
 		(dnp no)
-		(property "Reference" "Q9"
+		(property "Reference" "Q3"
 			(at 43.688 194.056 0)
 			(show_name no)
@@
 			(project "Battery Display"
 				(path "/66b9b57f-ad5a-4774-9c04-72011a45113c"
-					(reference "Q9")
+					(reference "Q3")
 					(unit 1)
 				)
@@
 		(in_pos_files yes)
 		(dnp no)
-		(property "Reference" "Q7"
+		(property "Reference" "Q1"
 			(at 24.638 194.056 0)
 			(show_name no)
@@
 			(project "Battery Display"
 				(path "/66b9b57f-ad5a-4774-9c04-72011a45113c"
-					(reference "Q7")
+					(reference "Q1")
 					(unit 1)
 				)
@@
 		(in_pos_files yes)
 		(dnp no)
-		(property "Reference" "Q8"
+		(property "Reference" "Q2"
 			(at 29.21 200.152 0)
 			(show_name no)
@@
 			(project "Battery Display"
 				(path "/66b9b57f-ad5a-4774-9c04-72011a45113c"
-					(reference "Q8")
+					(reference "Q2")
 					(unit 1)
 				)

Commit message: Added missing 'Part' metadata for C11.
Signed-off-by: digimer <digital.mermaid@gmail.com>
Parts:
- C11: Part (none) -> Knowles Syfer 2211JA250102JKTSYX
Changed lines of the file:
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@@
 			)
 		)
-		(property "MANUFACTURER" ""
+		(property "Part" "Knowles Syfer 2211JA250102JKTSYX"
 			(at 201.93 88.9 90)
 			(hide yes)
-			(show_name no)
-			(do_not_autoplace no)
-			(effects
-				(font
-					(size 1.27 1.27)
-				)
-			)
-		)
-		(property "MAXIMUM_PACKAGE_HEIGHT" ""
-			(at 201.93 88.9 90)
-			(hide yes)
-			(show_name no)
-			(do_not_autoplace no)
-			(effects
-				(font
-					(size 1.27 1.27)
-				)
-			)
-		)
-		(property "PARTREV" ""
-			(at 201.93 88.9 90)
-			(hide yes)
-			(show_name no)
-			(do_not_autoplace no)
-			(effects
-				(font
-					(size 1.27 1.27)
-				)
-			)
-		)
-		(property "STANDARD" ""
-			(at 201.93 88.9 90)
-			(hide yes)
