File: Full Boards/LED 1212 Al PCBs/LED 1212 Al PCBs.kicad_pcb (KiCad board)
At the start: 2 copper layers, 25 x 26.5 mm, 3 parts

Commit message: Started reworking the Relay Unit, not done. Updated the LED 1212 to create part-accurante iBOM for the three Rev. B colour variants.
Signed-off-by: digimer <digital.mermaid@gmail.com>
Parts:
- LED1: value LJ_CRBP.01 -> LUW CRBP.01-LYMY-G4J4-Y474
Changed lines of the file:
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@@
 			)
 		)
-		(property "Value" "LJ_CRBP.01"
+		(property "Value" "LUW CRBP.01-LYMY-G4J4-Y474"
 			(at 0 0 90)
 			(layer "F.SilkS")
@@
 			)
 		)
-		(property "Datasheet" "https://look.ams-osram.com/m/52bae5cfb8626588/original/LJ-CRBP-01.pdf"
+		(property "Datasheet" "https://look.ams-osram.com/m/71a3bd5830272549/original/LUW-CRBP-01.pdf"
 			(at 0 0 90)
 			(layer "F.Fab")
@@
 			)
 		)
-		(property "Part - Red" "ams OSRAM LJ CRBP.01-JZLX-27-3A4A-350-R18"
+		(property "Part - Red" "ams OSRAM LJ CRBP.01-JZLX-27-3A4A"
 			(at 0 0 270)
 			(unlocked yes)
@@
 			)
 		)
-		(property "Part - Green" "ams OSRAM LT CRBP.01-KZLZ-36-Q525-350-R18"
+		(property "Part - Green" "ams OSRAM LT CRBP.01-KZLZ-36-Q525"
 			(at 0 0 270)
 			(unlocked yes)
@@
 			)
 		)
-		(property "Part - White" "ams OSRAM LUW CRBP.01-LYMY-G4J4-Y474-350-R18"
+		(property "Part - White" "ams OSRAM LUW CRBP.01-LYMY-G4J4-Y474"
+			(at 0 0 270)
+			(unlocked yes)
+			(layer "F.Fab")
+			(hide yes)
+			(effects
+				(font
+					(size 1 1)
+					(thickness 0.15)
+				)
+			)
+		)
+		(property "Part" "ams OSRAM LUW CRBP.01-LYMY-G4J4-Y474"
 			(at 0 0 270)
 			(unlocked yes)
@@
 			)
 		)
+		(attr exclude_from_bom)
 		(duplicate_pad_numbers_are_jumpers no)
 		(fp_rect
@@
 			)
 		)
+		(attr exclude_from_bom)
 		(duplicate_pad_numbers_are_jumpers no)
 		(fp_rect
