File: Full Boards/LED 1212 Al PCBs/LED 1212 Al PCBs.kicad_sch (KiCad schematic)
At the start: 3 parts

Commit message: Removed the binning and packaging suffixes from the LED references.
Signed-off-by: digimer <digital.mermaid@gmail.com>
Parts:
- LED1: Part - Green ams OSRAM LT CRBP.01-KZLZ-36-Q525-350-R18 -> ams OSRAM LT CRBP.01-KZLZ-36-Q525; Part - Red ams OSRAM LJ CRBP.01-JZLX-27-3A4A-350-R18 -> ams OSRAM LJ CRBP.01-JZLX-27-3A4A; Part - White ams OSRAM LUW CRBP.01-LYMY-G4J4-Y474-350-R18 -> ams OSRAM LUW CRBP.01-LYMY-G4J4-Y474
Other:
- note added: "Red: ams OSRAM LJ CRBP.01-JZLX-27-3A4A Green: ams OSRAM LT CRBP.01-KZLZ-36-Q525 White: ams OSRAM LUW CRBP.01-LYMY-G4J4-Y474"
- note removed: "Red: ams OSRAM LJ CRBP.01-JZLX-27-3A4A-350-R18 Green: ams OSRAM LT CRBP.01-KZLZ-36-Q525-350-R18 White: ams OSRAM LUW CRBP.01-LYMY-G4J4-Y474-350-R18"
Changed lines of the file:
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@@
 		)
 	)
-	(text "Red: ams OSRAM LJ CRBP.01-JZLX-27-3A4A-350-R18\nGreen: ams OSRAM LT CRBP.01-KZLZ-36-Q525-350-R18\nWhite: ams OSRAM LUW CRBP.01-LYMY-G4J4-Y474-350-R18"
+	(text "Red: ams OSRAM LJ CRBP.01-JZLX-27-3A4A\nGreen: ams OSRAM LT CRBP.01-KZLZ-36-Q525\nWhite: ams OSRAM LUW CRBP.01-LYMY-G4J4-Y474"
 		(exclude_from_sim no)
 		(at 88.392 101.854 0)
@@
 			)
 		)
-		(property "Part - Red" "ams OSRAM LJ CRBP.01-JZLX-27-3A4A-350-R18"
+		(property "Part - Red" "ams OSRAM LJ CRBP.01-JZLX-27-3A4A"
 			(at 143.51 480.01 0)
 			(hide yes)
@@
 			)
 		)
-		(property "Part - Green" "ams OSRAM LT CRBP.01-KZLZ-36-Q525-350-R18"
+		(property "Part - Green" "ams OSRAM LT CRBP.01-KZLZ-36-Q525"
 			(at 127 85.09 0)
 			(hide yes)
@@
 			)
 		)
-		(property "Part - White" "ams OSRAM LUW CRBP.01-LYMY-G4J4-Y474-350-R18"
+		(property "Part - White" "ams OSRAM LUW CRBP.01-LYMY-G4J4-Y474"
 			(at 127 85.09 0)
 			(hide yes)

Commit message: Added Exlude from BoM flag to the SMD pads.
Signed-off-by: digimer <digital.mermaid@gmail.com>
Parts:
- SMD1, SMD2: now left out of the parts list
Changed lines of the file:
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@@
 		(body_style 1)
 		(exclude_from_sim no)
-		(in_bom yes)
+		(in_bom no)
 		(on_board yes)
 		(in_pos_files yes)
@@
 		(body_style 1)
 		(exclude_from_sim no)
-		(in_bom yes)
-		(on_board yes)
-		(in_pos_files yes)
+		(in_bom no)
+		(on_board yes)
+		(in_pos_files yes)

Commit message: Started reworking the Relay Unit, not done. Updated the LED 1212 to create part-accurante iBOM for the three Rev. B colour variants.
Signed-off-by: digimer <digital.mermaid@gmail.com>
Parts:
- LED1: value LJ_CRBP.01 -> LT CRBP.01-KZLZ-36-Q525; Part (none) -> ams OSRAM LT CRBP.01-KZLZ-36-Q525
Changed lines of the file:
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@@
 			)
 		)
-		(property "Value" "LJ_CRBP.01"
+		(property "Value" "LT CRBP.01-KZLZ-36-Q525"
 			(at 122.174 92.202 0)
 			(hide yes)
@@
 			)
 		)
-		(property "Datasheet" "https://look.ams-osram.com/m/52bae5cfb8626588/original/LJ-CRBP-01.pdf"
+		(property "Datasheet" "https://look.ams-osram.com/m/2df1c98d1ba04fa4/original/LT-CRBP-01.pdf"
 			(at 143.51 280.01 0)
 			(hide yes)
@@
 			(at 127 85.09 0)
 			(hide yes)
+			(show_name no)
+			(do_not_autoplace no)
+			(effects
+				(font
+					(size 1.27 1.27)
+				)
+			)
+		)
+		(property "Part" "ams OSRAM LT CRBP.01-KZLZ-36-Q525"
+			(at 127 85.09 0)
+			(hide yes)
