File: Full Boards/Relay Unit/Relay Unit.kicad_sch (KiCad schematic)
At the start: 140 parts, among them J1 Future Bond, J3 Program Header, SW1 Status Switch, SW3 SW_MEC_5G, SW4 SW_MEC_5G, U1 ISO1044BD, U10 FM24CL64B-G, U15 LM1117MP-5.0, U2 MAX3232, U3 STM32C092KCT6, U4 ULN2003A, U5 ULN2003A, U6 ULN2003A, U8 FM24CL64B-G, U9 IS31FL3731-SA

Commit message: Started reworking the Relay Unit, not done. Updated the LED 1212 to create part-accurante iBOM for the three Rev. B colour variants.
Signed-off-by: digimer <digital.mermaid@gmail.com>
Parts:
- removed C1, C10, C11, C12, C13, C2, C22, C23, C24, C7: 0.1uF, mr-stuff:RCE5C1H104J2A2H03B, symbol Device:C
- removed C16, C17, C18: 100μF, Capacitor_THT:CP_Radial_D8.0mm_P5.00mm, symbol Device:C_Polarized
- removed C19: 1μF, Capacitor_THT:C_Rect_L7.2mm_W7.2mm_P5.00mm_FKS2_FKP2_MKS2_MKP2, symbol Device:C
- removed C20, C21, C3, C4: 0.1μF, mr-stuff:RCE5C1H104J2A2H03B, symbol Device:C
- removed C5, C8, C9: 10uF, Capacitor_THT:CP_Radial_D8.0mm_P3.50mm, symbol Device:C_Polarized
- removed C6: TDK FA28NP01H152JNU06, mr-stuff:TDK CAPRB500W50L400T250H550, symbol mr-parts:TDK FA28NP01H152JNU06
- removed D145: 1N5822, Diode_THT:D_DO-201AD_P15.24mm_Horizontal, symbol Diode:1N5822
- removed D146: SLD22-018, mr-stuff:DIOAD4425W136L885D885, symbol mr-parts:SLD15-018
- removed DE1: ~, mr-stuff:Amphenol_L77SDE09SA4CH4F, symbol mr-parts:DE9_Socket
- removed H1, H2, H3, H4, H5: MountingHole_Pad, MountingHole:MountingHole_4mm_Pad_Via, symbol Mechanical:MountingHole_Pad
- removed J1: Future Bond, Connector_PinHeader_2.54mm:PinHeader_1x03_P2.54mm_Vertical, symbol Connector:Conn_01x03_Pin
- removed J3: Program Header, Connector_PinHeader_2.54mm:PinHeader_1x05_P2.54mm_Horizontal, symbol Connector:Conn_01x05_Pin
- removed L1: PA4340.103NLT, mr-stuff:Pulse PA4340.103NLT, symbol Device:L
- removed LR12: NCV8730ASN500T1G, mr-stuff:TSOP-5_483_OSI, symbol mr-parts:NCV8730ASN500T1G
- removed N2K1: ~, mr-stuff:M12B-05PMMR, symbol mr-parts:M12B-05PMMR
- removed PS2: SPBW06F-05, mr-stuff:SPBW06F05, symbol mr-parts:SPBW06F-05
- removed PTC2: PTC, mr-stuff:AHEF100, symbol mr-parts:AHEF100
- removed R1, R2, R3, R5: 4.7K, Resistor_THT:R_Axial_DIN0207_L6.3mm_D2.5mm_P7.62mm_Horizontal, symbol Device:R
- removed R10, R11, R6: 3.3K, Resistor_THT:R_Axial_DIN0207_L6.3mm_D2.5mm_P7.62mm_Horizontal, symbol Device:R
- removed R4: 100K, Resistor_THT:R_Axial_DIN0207_L6.3mm_D2.5mm_P7.62mm_Horizontal, symbol Device:R
- removed R7, R8: 10K, Resistor_THT:R_Axial_DIN0207_L6.3mm_D2.5mm_P7.62mm_Horizontal, symbol Device:R
- removed SW3, SW4: SW_MEC_5G, mr-stuff:SW_TS03-66-50-BK-160-LCR-D-67, symbol Switch:SW_MEC_5G
- removed TP1: TP_VRAW, Connector_PinHeader_2.54mm:PinHeader_1x01_P2.54mm_Vertical, symbol Connector:Conn_01x01_Pin
- removed TP12, TP5: +5V_SHIP, Connector_PinHeader_2.54mm:PinHeader_1x01_P2.54mm_Vertical, symbol Connector:Conn_01x01_Pin
- removed TP13, TP2, TP6: GND_SHIP, Connector_PinHeader_2.54mm:PinHeader_1x01_P2.54mm_Vertical, symbol Connector:Conn_01x01_Pin
- removed TP3: N2K_RX, Connector_PinHeader_2.54mm:PinHeader_1x01_P2.54mm_Vertical, symbol Connector:Conn_01x01_Pin
- removed TP4: N2K_TX, Connector_PinHeader_2.54mm:PinHeader_1x01_P2.54mm_Vertical, symbol Connector:Conn_01x01_Pin
- removed TP7: +5V, Connector_PinHeader_2.54mm:PinHeader_1x01_P2.54mm_Vertical, symbol Connector:Conn_01x01_Pin
- removed TP8: GND, Connector_PinHeader_2.54mm:PinHeader_1x01_P2.54mm_Vertical, symbol Connector:Conn_01x01_Pin
- removed TP9: +3.3V, Connector_PinHeader_2.54mm:PinHeader_1x01_P2.54mm_Vertical, symbol Connector:Conn_01x01_Pin
- removed U1: ISO1044BD, Package_SO:SOIC-8_3.9x4.9mm_P1.27mm, symbol Interface_CAN_LIN:ISO1044BD
- removed U10, U8: FM24CL64B-G, Package_SO:SOIC-8_3.9x4.9mm_P1.27mm, symbol Memory_NVRAM:FM24C64B
- removed U15: LM1117MP-5.0, Package_TO_SOT_SMD:SOT-223-3_TabPin2, symbol Regulator_Linear:LM1117MP-5.0
- removed U2: MAX3232, Package_SO:TSSOP-16_4.4x5mm_P0.65mm, symbol mr-parts:TI MAX3232EIPWRQ1
- removed U9: IS31FL3731-SA, Package_SO:SSOP-28_5.3x10.2mm_P0.65mm, symbol Driver_LED:IS31FL3731-SA
- added C26, C28, C29, C30, C32, C35, C36, C37, C39, C40, C44, C47, C48, C49: 0.1uF, mr-stuff:Kyocera AVX 0805, symbol Device:C
- added C27: 4.7uF, mr-stuff:Kyocera AVX 1206, symbol Device:C
- added C34, C38: 16pF, mr-stuff:Kemet C0603X, symbol Device:C
- added C41, C42, C43: 100uF, Capacitor_THT:CP_Radial_D8.0mm_P3.50mm, symbol Device:C_Polarized
- added C45: 1uF, mr-stuff:Kemet C1206C, symbol Device:C
- added C46, C53: 22uF, mr-stuff:Murata GCJ31CR71A, symbol Device:C
- added C50: 10uF, mr-stuff:Kyocera AVX 1206, symbol Device:C_Polarized
- added C51: 1nF, mr-stuff:Knowles Syfer 2211JA25, symbol Device:C
- added C52: 10uF, mr-stuff:TDK CGA5, symbol Device:C
- added CMC1: ACT12101012PTL00, mr-stuff:TDK ACT12101012PTL00, symbol mr-parts:TDK ACT1210-510-2P-TL00
- added CPD1: IS31FL3731-SA, Package_SO:SSOP-28_5.3x10.2mm_P0.65mm, symbol mr-parts:Lumissil IS31FL3731-SALS2-TR
- added DE2: L77SDE09SA4CH4F, mr-stuff:Amphenol_L77SDE09SA4CH4F, symbol mr-parts:Amphenol L77SDE09SA4CH4F
- added DE3: L777SDE09PA4CH4F, mr-stuff:Amphenol L777SDE09PA4CH4F, symbol mr-parts:DE9_Pins
- added FID1, FID2, FID3: Fiducial, Fiducial:Fiducial_0.5mm_Mask1.5mm, symbol Mechanical:Fiducial
- added H6, H7, H8, H9: MountingHole_Pad, MountingHole:MountingHole_4mm_Pad_Via, symbol Mechanical:MountingHole_Pad
- added ICT1: ISO1044BD, mr-stuff:TI ISO1044BDR, symbol mr-parts:TI_ISO1044BDR
- added IDCB1: SPBW06F-05, mr-stuff:Meanwell SPBW06F05, symbol mr-parts:Meanwell SPBW06F-05
- added J4: Optional Bond, Connector_PinHeader_2.54mm:PinHeader_1x02_P2.54mm_Vertical, symbol Connector:Conn_01x02_Pin
- added J5: Program Header, Connector_PinHeader_2.54mm:PinHeader_1x05_P2.54mm_Horizontal, symbol Connector:Conn_01x05_Pin
- added L2: PA4340.103NLT, mr-stuff:Pulse PA4340.103NLT, symbol Device:L
- added LVR1: BD450S5FP-CE2, mr-stuff:Rohm BD4xxS5 TO252-3, symbol mr-parts:Rohm BD450S5FP-CE2
- added LVR2: BD33C0AFP-CE2, mr-stuff:Rohm BD33C0, symbol mr-parts:BD33C0AFP-CE2
- added MCU1: STM32C092KCT6, mr-stuff:STM STM32C0 LQFP-32, symbol mr-parts:STM STM32C092KCT6
- added OX1: 12.60378, Crystal:Crystal_SMD_3225-4Pin_3.2x2.5mm, symbol mr-parts:Geyer 12.60378
- added PTC3: 0ZCG0110CF2B, mr-stuff:Bel Fuse 0ZCG, symbol mr-parts:Bel Fuse 0ZCG0110CF2B
- added R27: 4.7k, mr-stuff:Stackpole RMCA0805, symbol Device:R
- added R28: 20k, mr-stuff:Stackpole RMCA0805, symbol Device:R
- added R29, R30, R31, R32: 3.3k, mr-stuff:Stackpole RNCF0805, symbol Device:R
- added R33, R34: 10k, mr-stuff:Stackpole RMCA0805, symbol Device:R
- added ROM1, ROM2: M24C64, mr-stuff:STM M24C64-RMN6P, symbol mr-parts:STM_M24C64-RMN6P
- added RST1: MAX3232, mr-stuff:TI MAX3232EIPWRQ1, symbol mr-parts:TI MAX3232EIPWRQ1
- added SD1: VS-30MQ040HM3/5AT, Diode_SMD:D_SMA, symbol Device:D_Schottky
- added SW2: Boot, mr-stuff:Same Sky TS03-66, symbol mr-parts:Same Sky TS03-66-50-BK-160-LCR-D-67
- added SW5: Reset, mr-stuff:Same Sky TS03-66, symbol mr-parts:Same Sky TS03-66-50-BK-160-LCR-D-67
- added TB19: 1862440, mr-stuff:Phoenix Contact 1862440, symbol mr-parts:Phoenix Contact 1862440
- added TP10: Ship Power, Connector_PinHeader_2.54mm:PinHeader_1x03_P2.54mm_Vertical, symbol Connector:Conn_01x03_Pin
- added TP11: Board Power, Connector_PinHeader_2.54mm:PinHeader_1x03_P2.54mm_Vertical, symbol Connector:Conn_01x03_Pin
- added TP14: Board I2C, Connector_PinHeader_2.54mm:PinHeader_1x02_P2.54mm_Vertical, symbol Connector:Conn_01x02_Pin
- added TP15: IS31 I2C, Connector_PinHeader_2.54mm:PinHeader_1x02_P2.54mm_Vertical, symbol Connector:Conn_01x02_Pin
- added TVS2: SMBJ20A-Q, mr-stuff:Bourns SMBJ20, symbol mr-parts:Bouns SMBJ20A-Q
- added TVS3: PESD2CANFD54VT-QR, mr-stuff:Nexperia PESD2CANFD, symbol mr-parts:Nexperia PESD2CANFD54VT-QR
- LR1, LR2, LR3, LR4, LR5, LR6, LR7, LR8, LR9: value ~ -> (none)
Connections:
- net +3.3V: now also C26.2, C27.1, C28.2, C36.2, C40.2, C48.2, C49.2, C53.2, ICT1.1 (VCC1), J5.2 (Pin_2), LVR2.3 (Vout), MCU1.4 (VDD), R27.1, R29.2, R30.2, R31.2, R32.2, R33.2, ROM1.1 (E0), ROM1.3 (E2), ROM1.8 (VCC), ROM2.1 (E0), ROM2.2 (E1), ROM2.3 (E2), ROM2.8 (VCC), RST1.10 (T2IN), RST1.16 (VCC), SW2.1 (A), SW2.2 (A), TP11.1 (Pin_1)
- net +5V: now also C41.1, C42.1, C43.1, C45.1, C47.2, C52.2, CPD1.2 (VCC), CPD1.3 (~{SDB}), IDCB1.6 (+VOUT), LVR2.1 (Vcc), TP11.3 (Pin_3)
- net +5V_SHIP: now also C30.2, C46.2, ICT1.8 (VCC2), LVR1.3 (VOUT), TP10.1 (Pin_1)
- net BOARD_I2C_SCL: now also MCU1.14 (PA7), R31.1, ROM1.6 (SCL), ROM2.6 (SCL), TP14.2 (Pin_2)
- net BOARD_I2C_SDA: now also MCU1.13 (PA6), R29.1, ROM1.5 (SDA), ROM2.5 (SDA), TP14.1 (Pin_1)
- net CA1: now also CPD1.21 (CA1)
- net CA2: now also CPD1.22 (CA2)
- net CA3: now also CPD1.23 (CA3)
- net CA4: now also CPD1.24 (CA4)
- net CA5: now also CPD1.25 (CA5)
- net CA6: now also CPD1.26 (CA6)
- net CA7: now also CPD1.27 (CA7)
- net CA8: now also CPD1.28 (CA8)
- net CA9: now also CPD1.1 (CA9)
- net DEBUG_SWCLK: now also J5.4 (Pin_4), MCU1.25 (PA14), R34.1, SW2.3 (B), SW2.4 (B)
- net DEBUG_SWDIO: now also J5.3 (Pin_3), MCU1.24 (PA13)
- net GND: now also C26.1, C27.2, C28.1, C29.1, C34.2, C37.1, C38.1, C40.1, C41.2, C42.2, C43.2, C44.1, C45.2, C47.1, C48.1, C49.1, C51.2, C52.1, C53.1, CPD1.17 (IN), CPD1.18 (AD), CPD1.5 (GND), DE2.5, DE2.SH1, DE2.SH2, DE3.7, DE3.8, DE3.9, DE3.SH1, DE3.SH2, ICT1.4 (GND1), IDCB1.7 (-VOUT), J5.5 (Pin_5), LVR2.2 (Gnd), MCU1.5 (VSS), OX1.2, OX1.4, R28.1, R34.2, ROM1.2 (E1), ROM1.4 (VSS), ROM1.7 (~{WC}), ROM2.4 (VSS), ROM2.7 (~{WC}), RST1.15 (GND), SW5.3 (B), SW5.4 (B), TP11.2 (Pin_2)
- net GND_SHIP: now also C30.1, C39.1, C46.1, C50.2, C51.1, H6.1, H7.1, H8.1, H9.1, ICT1.7 (GND2), IDCB1.1 (-VIN), J4.2 (Pin_2), LVR1.4 (GND), TB19.5, TB19.6, TP10.2 (Pin_2), TVS2.2 (A), TVS3.3
- net NRST: now also C29.2, J5.1 (Pin_1), MCU1.6 (PF2), R33.1, SW5.1 (A), SW5.2 (A)
- net USART1_RX: now also MCU1.8 (PA1), RST1.12 (R1OUT)
- net USART1_TX: now also MCU1.7 (PA0), RST1.11 (T1IN)
- net V_RAW: now also C39.2, C50.1, L2.1, LVR1.1 (VCC), SD1.1 (K), TP10.3 (Pin_3)
- new net: C37.2, RST1.6 (VS-)
- new net: C32.2, RST1.1 (C1+)
- new net: C36.1, RST1.2 (VS+)
- new net: C32.1, RST1.3 (C1-)
- new net: C35.2, RST1.4 (C2+)
- new net: C35.1, RST1.5 (C2-)
- new net: CPD1.6 (R_EXT), R28.2
- new net: IDCB1.2 (+VIN), L2.2
- new net: CMC1.2 (I2), ICT1.5 (CANL)
- new net: CMC1.1 (I1), ICT1.6 (CANH)
- new net: J4.1 (Pin_1), TB19.1, TB19.2
- new net: PTC3.1, SD1.2 (A), TVS2.1 (K)
- new net: C44.2, CPD1.16 (C_FILT)
- new net: PTC3.2, TB19.3, TB19.4
- new net CB1: CPD1.7 (CB1)
- new net CB2: CPD1.8 (CB2)
- new net CB3: CPD1.9 (CB3)
- new net CB4: CPD1.10 (CB4)
- new net CB5: CPD1.11 (CB5)
- new net CB6: CPD1.12 (CB6)
- new net CB7: CPD1.13 (CB7)
- new net CB8: CPD1.14 (CB8)
- new net CB9: CPD1.15 (CB9)
- new net DISPLAY_ON_IN: MCU1.26 (PA15)
- new net DISPLAY_ON_IN_PLUG: DE3.3
- new net IS31_I2C_SCL: CPD1.20 (SCL), MCU1.19 (PA9), R32.1, TP15.2 (Pin_2)
- new net IS31_I2C_SDA: CPD1.19 (SDA), MCU1.21 (PA10), R30.1, TP15.1 (Pin_1)
- new net IS31_INTB_OUT: CPD1.4 (~{INTB}), MCU1.22 (PA11), R27.2
- new net LCD_PGDOWN_IN_PLUG: DE3.4
- new net LCD_PGUP_IN_PLUG: DE3.5
- new net N2K_CAN_H: CMC1.4 (O1), TB19.7, TB19.8, TVS3.1
- new net N2K_CAN_L: CMC1.3 (O2), TB19.10, TB19.9, TVS3.2
- new net N2K_FDCAN_RX: ICT1.3 (RXD), MCU1.15 (PB0)
- new net N2K_FDCAN_TX: ICT1.2 (TXD), MCU1.16 (PB1)
- new net OSC_IN: C34.1, MCU1.2 (PC14), OX1.1
- new net OSC_OUT: C38.2, MCU1.3 (PC15), OX1.3
- new net RS232_RX: DE2.3, RST1.13 (R1IN)
- new net RS232_TX: DE2.2, RST1.14 (T1OUT)
- no-connect marks 29 -> 20
Other:
- note added: "-=] DE2 1 - nc 2 - nc 3 - Display On Switch 4 - LCD Page Down Switch 5 - LCD Page Up Switch 6 - nc 7 - ESD Ground 8 - Ground (Display On) 9 - Ground (LCD Paging)"
- note added: "C11 provided for optional Common Mode EMI suppression If used: Knowles Syfer 2211JA250102JKTSYX"
- note added: "Charliplex LED Driver"
- note added: "Display Switches and Pot"
- note added: "High-Speed External Crystal"
- note added: "I2C Addr: 0x74"
- note added: "Isolated 5v to 3.3v"
- note added: "NOTE: IS31FL373Ω is powered from the +5V rail to allow for higher voltage LEDs. The I2C bus operates natively at 3.3V. This logic mismatch is validated. The minimum High-Level Input Voltage V{IH} of 1.4V. The 3.3V logic exceeds this threshold. A level shifter is intentionally omitted."
- note added: "Pin 4 tied to GND for thermal dissipation"
- note added: "Place as close to MCU pins as possible. Add ground ring with vias as Faraday cage."
- note added: "TB1 Pins: 1. Shield 2. V_RAW 3. GND_SHIP 4. CAN High 5. CAN Low"
- note added: "Use conductive tape on the back-side of the plexi and tie it to pin 7."
- note added: "V_RAW can be 10~16 VDC TB1 connect to Amphenol MSAS-05PMMC-SF8C15"
- note removed: "*V_RAW can vary from 10~16vDC"
- note removed: "1500pF"
- note removed: "5v to 3.3v"
- note removed: "Boot"
- note removed: "LED Driver"
- note removed: "Put close to MCU!"
- note removed: "Reset"
- moved on the sheet: C14, C15, C25, D1, D10, D11, D12, D13, D14, D15, D16, D17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
