File: Full Boards/N2K Transceiver/N2K Transceiver.kicad_sch (KiCad schematic)
At the start: 74 parts, among them J3 JTAG, SW1 SW_MEC_5G, SW2 SW_MEC_5G, SW3 SW_MEC_5G

Commit message: Added missing footprint to the new VIshay TVS
Signed-off-by: digimer <digital.mermaid@gmail.com>
Parts:
- TVS2: footprint (none) -> mr-stuff:Vishay VCAN33A2-03S
Changed lines of the file:
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@@
 			)
 		)
-		(property "Footprint" ""
+		(property "Footprint" "mr-stuff:Vishay VCAN33A2-03S"
 			(at 160.02 152.07 0)
 			(hide yes)

Commit message: Updated annotation.
Signed-off-by: digimer <digital.mermaid@gmail.com>
Parts:
- removed R26: 0R, mr-stuff:Vishay RCA-SR e3, symbol mr-parts:Vishay RCA08050000ZSEASR
- added R3: 0R, mr-stuff:Vishay RCA-SR e3, symbol mr-parts:Vishay RCA08050000ZSEASR
- renumbered C11 to C10, C12 to C11, C13 to C12, C14 to C13, C15 to C14, C16 to C15, C5 to C2, C8 to C3, C2 to C4, C3 to C5, C4 to C8, C10 to C9, R6 to R10, R7 to R11, R8 to R12, R9 to R13, R10 to R14, R11 to R15, R12 to R16, R13 to R17, R14 to R18, R15 to R19, R16 to R20, R17 to R21, R18 to R22, R19 to R23, R20 to R24, R21 to R25, R22 to R26, R23 to R27, R27 to R4, R25 to R5, R24 to R6, R3 to R7, R4 to R8, R5 to R9
Connections:
- net V_RAW: now also R3.1
- net at C3.1, C4.1, C5.1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: now also R3.2
Other:
- note removed: "Test Points"
- moved on the sheet: FID1, FID2, FID3, H1, H2, H3, H4, TP3

Commit message: More cleanup
Signed-off-by: digimer <digital.mermaid@gmail.com>
Other:
- moved on the sheet: TP1
Changed lines of the file:
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@@
 	(wire
 		(pts
-			(xy 87.63 104.14) (xy 107.95 104.14)
+			(xy 87.63 104.14) (xy 92.71 104.14)
 		)
 		(stroke
@@
 	(wire
 		(pts
-			(xy 105.41 90.17) (xy 105.41 92.71)
+			(xy 90.17 95.25) (xy 90.17 97.79)
 		)
 		(stroke
@@
 	(wire
 		(pts
-			(xy 105.41 92.71) (xy 100.33 92.71)
+			(xy 90.17 97.79) (xy 85.09 97.79)
 		)
 		(stroke
@@
 	(wire
 		(pts
-			(xy 107.95 104.14) (xy 107.95 90.17)
+			(xy 92.71 104.14) (xy 92.71 95.25)
 		)
 		(stroke
@@
 	(wire
 		(pts
-			(xy 110.49 106.68) (xy 110.49 90.17)
+			(xy 95.25 106.68) (xy 95.25 95.25)
 		)
 		(stroke
@@
 	(wire
 		(pts
-			(xy 100.33 92.71) (xy 100.33 90.17)
+			(xy 85.09 97.79) (xy 85.09 95.25)
 		)
 		(stroke
@@
 	(wire
 		(pts
-			(xy 113.03 90.17) (xy 113.03 92.71)
+			(xy 97.79 95.25) (xy 97.79 97.79)
 		)
 		(stroke
@@
 	(wire
 		(pts
-			(xy 87.63 106.68) (xy 110.49 106.68)
+			(xy 87.63 106.68) (xy 95.25 106.68)
 		)
 		(stroke
@@
 	(symbol
 		(lib_id "Connector:Conn_01x04_Pin")
-		(at 107.95 85.09 90)
+		(at 92.71 90.17 90)
 		(mirror x)
 		(unit 1)
@@
 		(dnp yes)
 		(property "Reference" "TP1"
-			(at 109.22 81.788 90)
+			(at 93.98 86.868 90)
 			(show_name no)
 			(do_not_autoplace no)
@@
 		)
 		(property "Value" "MCU Tx/Rx"
-			(at 109.22 83.82 90)
+			(at 93.98 88.9 90)
 			(show_name no)
 			(do_not_autoplace no)
@@
 		)
 		(property "Footprint" "Connector_PinHeader_2.54mm:PinHeader_1x04_P2.54mm_Vertical"
-			(at 107.95 85.09 0)
+			(at 92.71 90.17 0)
 			(hide yes)
 			(show_name no)
@@
 		)
 		(property "Datasheet" ""
-			(at 107.95 85.09 0)
+			(at 92.71 90.17 0)
 			(hide yes)
 			(show_name no)
@@
 		)
 		(property "Description" "Generic connector, single row, 01x04, script generated"
-			(at 107.95 85.09 0)
+			(at 92.71 90.17 0)
 			(hide yes)
 			(show_name no)
@@
 		)
 		(property "Part" "Amphenol 68001-416HLF"
-			(at 107.95 85.09 90)
+			(at 92.71 90.17 90)
 			(hide yes)
 			(show_name no)
@@
 	(symbol
 		(lib_id "power:+3.3V")
-		(at 100.33 90.17 0)
+		(at 85.09 95.25 0)
 		(unit 1)
 		(body_style 1)
@@
 		(dnp no)
 		(property "Reference" "#PWR077"
-			(at 100.33 93.98 0)
+			(at 85.09 99.06 0)
 			(hide yes)
 			(show_name no)
@@
 		)
 		(property "Value" "+3.3V"
-			(at 100.33 86.36 0)
+			(at 85.09 91.44 0)
 			(show_name no)
 			(do_not_autoplace no)
@@
 		)
 		(property "Footprint" ""
-			(at 100.33 90.17 0)
+			(at 85.09 95.25 0)
 			(hide yes)
 			(show_name no)
@@
 		)
 		(property "Datasheet" ""
-			(at 100.33 90.17 0)
+			(at 85.09 95.25 0)
 			(hide yes)
 			(show_name no)
@@
 		)
 		(property "Description" "Power symbol creates a global label with name \"+3.3V\""
-			(at 100.33 90.17 0)
+			(at 85.09 95.25 0)
 			(hide yes)
 			(show_name no)
@@
 	(symbol
 		(lib_id "power:GND")
-		(at 113.03 92.71 0)
+		(at 97.79 97.79 0)
 		(unit 1)
 		(body_style 1)
@@
 		(dnp no)
 		(property "Reference" "#PWR078"
-			(at 113.03 99.06 0)
+			(at 97.79 104.14 0)
 			(hide yes)
 			(show_name no)
@@
 		)
 		(property "Value" "GND"
-			(at 113.03 96.266 0)
+			(at 97.79 101.346 0)
 			(show_name no)
 			(do_not_autoplace no)
@@
 		)
 		(property "Footprint" ""
-			(at 113.03 92.71 0)
+			(at 97.79 97.79 0)
 			(hide yes)
 			(show_name no)
@@
 		)
 		(property "Datasheet" ""
-			(at 113.03 92.71 0)
+			(at 97.79 97.79 0)
 			(hide yes)
 			(show_name no)
@@
 		)
 		(property "Description" "Power symbol creates a global label with name \"GND\" , ground"
-			(at 113.03 92.71 0)
+			(at 97.79 97.79 0)
 			(hide yes)
 			(show_name no)
