File: projects/throttle-led-board/pcb/Throttle LED Board.kicad_pcb (KiCad board)
At the start: 4 copper layers, 45 x 184 mm, 54 parts

Commit message: Added switches to the N2K Transceiver
This is to allow for near-hardware overrides of the masthead light states if/when the MFD is unavailable.

Signed-off-by: digimer <digital.mermaid@gmail.com>
Parts:
- moved H4 20.2 mm to (237.7, 202.8)
- moved H3 17.3 mm to (165.2, 202.8)
- moved LED45 6.03 mm to (211.0, 144.3)
- moved LED44 5.97 mm to (189.0, 144.3)
Changed lines of the file:
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@@
 	(footprint "mr-stuff:Kingbright WP383SURDTK"
 		(layer "F.Cu")
-		(at 211.032618 62.6)
+		(at 211.03 62.6)
 		(property "Reference" "LED1"
 			(at 0 -2.286 0)
@@
 			(polygon
 				(pts
-					(xy 208.532618 61.35) (xy 213.532618 61.35) (xy 213.532618 63.85) (xy 208.532618 63.85)
+					(xy 208.53 61.35) (xy 213.53 61.35) (xy 213.53 63.85) (xy 208.53 63.85)
 				)
 			)
@@
 	(footprint "mr-stuff:Kingbright WP383SURDTK"
 		(layer "F.Cu")
-		(at 195 144.3)
+		(at 189.03 144.3)
 		(property "Reference" "LED44"
 			(at 3.4 0 90)
@@
 			(polygon
 				(pts
-					(xy 192.5 143.05) (xy 197.5 143.05) (xy 197.5 145.55) (xy 192.5 145.55)
+					(xy 186.53 143.05) (xy 191.53 143.05) (xy 191.53 145.55) (xy 186.53 145.55)
 				)
 			)
@@
 	(footprint "MountingHole:MountingHole_4mm_Pad_Via"
 		(layer "F.Cu")
-		(at 182.5 202.77868)
+		(at 165.2 202.77868)
 		(descr "Mounting Hole 4mm, generated by kicad-footprint-generator mountinghole.py")
 		(tags "mountinghole")
@@
 	(footprint "mr-stuff:Kingbright WP383SURDTK"
 		(layer "F.Cu")
-		(at 205 144.3)
+		(at 211.03 144.3)
 		(property "Reference" "LED45"
 			(at 3.4 0 90)
@@
 			(polygon
 				(pts
-					(xy 202.5 143.05) (xy 207.5 143.05) (xy 207.5 145.55) (xy 202.5 145.55)
+					(xy 208.53 143.05) (xy 213.53 143.05) (xy 213.53 145.55) (xy 208.53 145.55)
 				)
 			)
@@
 	(footprint "MountingHole:MountingHole_4mm_Pad_Via"
 		(layer "F.Cu")
-		(at 217.5 202.77868)
+		(at 237.7 202.77868)
 		(descr "Mounting Hole 4mm, generated by kicad-footprint-generator mountinghole.py")
 		(tags "mountinghole")
@@
 	(footprint "mr-stuff:Kingbright WP383SURDTK"
 		(layer "F.Cu")
-		(at 189.032618 62.6)
+		(at 189.03 62.6)
 		(property "Reference" "LED2"
 			(at 0 -2.286 0)
@@
 			(polygon
 				(pts
-					(xy 186.532618 61.35) (xy 191.532618 61.35) (xy 191.532618 63.85) (xy 186.532618 63.85)
+					(xy 186.53 61.35) (xy 191.53 61.35) (xy 191.53 63.85) (xy 186.53 63.85)
 				)
 			)
