File: projects/n2k-transceiver/N2K Transceiver.kicad_sch (KiCad schematic)
At the start: 82 parts, among them J1 JTAG, SW1 SW_MEC_5G, SW2 SW_MEC_5G, SW3 SW_MEC_5G, SW4 SW_MEC_5G

Commit message: Added switches to the N2K Transceiver
This is to allow for near-hardware overrides of the masthead light states if/when the MFD is unavailable.

Signed-off-by: digimer <digital.mermaid@gmail.com>
Parts:
- added C18, C19: 0.1uF, mr-stuff:Kyocera AVX 0805, symbol Device:C
- added C27, C28, C29, C30, C31, C32, C33, C34, C35, C36: 0.1uF, mr-stuff:Kyocera AVX 0805, symbol mr-parts:Kyocera 08051C104K4Z2A
- added HDR1, HDR2, HDR3, HDR4, HDR5, HDR6: 0022112032, mr-stuff:Molex 0022112032, symbol mr-parts:Molex 0022112032
- added IOX1: PI4IOE5V6416RQ2LEX, mr-stuff:Diodes Inc PI4IOE5V6416RQ2LEX, symbol mr-parts:Diodes Inc PI4IOE5V6416RQ2LEX
- added R49, R50, R56, R57, R60, R61, R64, R65, R68, R69: 475R, mr-stuff:Stackpole RNCP0805, symbol mr-parts:Stackpole RNCP0805FTD475R
- added R51, R55, R58, R59, R62, R63, R66, R67, R70, R71: 4.7kR, mr-stuff:Stackpole RMCA0805, symbol mr-parts:Stackpole RMCA0805FT4K70-HP
- added R72, R73: 10kR, mr-stuff:Stackpole RNCP0805, symbol mr-parts:Stackpole RNCP0805FTD10K0
- added TVS32, TVS33, TVS34, TVS35, TVS36: TPD2E2U06QDBZRQ1, mr-stuff:TI TPD2E2U06, symbol mr-parts:TVS TPD2E2U06QDBZRQ1
- ROM1, ROM2: symbol mr-parts:STM_M24C64-RMN6P -> mr-parts:STM M24C64-RMN6P
Connections:
- net +3.3V: now also C18.1, C19.1, IOX1.2 (VDD^{(I2C)}), IOX1.21 (ADDR), IOX1.24 (VDD^{(P)}), R51.2, R55.2, R58.2, R59.2, R62.2, R63.2, R66.2, R67.2, R70.2, R71.2, R72.2, R73.2
- net CAN_HIGH: now also TP1.5 (Pin_5); no longer TP1.4 (Pin_4)
- net CAN_LOW: now also TP1.6 (Pin_6); no longer TP1.5 (Pin_5)
- net CAN_RX_LOCAL: now also TP1.8 (Pin_8); no longer TP1.7 (Pin_7)
- net CAN_TX_LOCAL: now also TP1.7 (Pin_7); no longer TP1.6 (Pin_6)
- net GND: now also TP1.2 (Pin_2), C18.2, C19.2, C27.2, C28.1, C29.2, C30.1, C31.2, C32.1, C33.2, C34.1, C35.2, C36.1, HDR1.2 (Pin_2), HDR2.2 (Pin_2), HDR3.2 (Pin_2), HDR4.2 (Pin_2), HDR5.2 (Pin_2), HDR6.2 (Pin_2), IOX1.12 (VSS), TVS32.3 (GND), TVS33.3 (GND), TVS34.3 (GND), TVS35.3 (GND), TVS36.3 (GND); no longer TP1.10 (Pin_10)
- net I2C_SCL: now also TP1.9 (Pin_9), IOX1.22 (SCL); no longer TP1.8 (Pin_8)
- net I2C_SDA: now also TP1.10 (Pin_10), IOX1.23 (SDA); no longer TP1.9 (Pin_9)
- net RXD0: now also TP1.4 (Pin_4); no longer TP1.3 (Pin_3)
- net TXD0: now also TP1.3 (Pin_3); no longer TP1.2 (Pin_2)
- net IOX1_INT: now reaches MCU1.21 (IO13)
- net IOX1_INT: now also IOX1.1 (~{INT}), R72.1
- new net: IOX1.3 (~{RESET}), R73.1
- new net ANCHOR_OFF_IN: C28.2, IOX1.5 (P0_1), R50.2, R55.1
- new net ANCHOR_OFF_PLUG: HDR1.3 (Pin_3), R50.1, TVS32.2 (IO2)
- new net ANCHOR_ON_IN: C27.1, IOX1.4 (P0_0), R49.2, R51.1
- new net ANCHOR_ON_PLUG: HDR1.1 (Pin_1), R49.1, TVS32.1 (IO1)
- new net BEACON_ON_IN: C35.1, IOX1.13 (P1_0), R68.2, R70.1
- new net BEACON_ON_PLUG: HDR5.1 (Pin_1), R68.1, TVS36.1 (IO1)
- new net DECK_OFF_IN: C34.2, IOX1.11 (P0_7), R65.2, R67.1
- new net DECK_OFF_PLUG: HDR4.3 (Pin_3), R65.1, TVS35.2 (IO2)
- new net DECK_ON_IN: C33.1, IOX1.10 (P0_6), R64.2, R66.1
- new net DECK_ON_PLUG: HDR4.1 (Pin_1), R64.1, TVS35.1 (IO1)
- new net LOCATE_ON_IN: C36.2, IOX1.14 (P1_1), R69.2, R71.1
- new net LOCATE_ON_PLUG: HDR6.1 (Pin_1), R69.1, TVS36.2 (IO2)
- new net STEAMING_OFF_IN: C32.2, IOX1.9 (P0_5), R61.2, R63.1
- new net STEAMING_OFF_PLUG: HDR3.3 (Pin_3), R61.1, TVS34.2 (IO2)
- new net STEAMING_ON_IN: C31.1, IOX1.8 (P0_4), R60.2, R62.1
- new net STEAMING_ON_PLUG: HDR3.1 (Pin_1), R60.1, TVS34.1 (IO1)
- new net TRICOLOUR_OFF_IN: C30.2, IOX1.7 (P0_3), R57.2, R59.1
- new net TRICOLOUR_OFF_PLUG: HDR2.3 (Pin_3), R57.1, TVS33.2 (IO2)
- new net TRICOLOUR_ON_IN: C29.1, IOX1.6 (P0_2), R56.2, R58.1
- new net TRICOLOUR_ON_PLUG: HDR2.1 (Pin_1), R56.1, TVS33.1 (IO1)
- no-connect marks 12 -> 19
Other:
- note added: "I^{2}C IO Expander (at 0x21h)"
- note added: "Intended Switches; 1. on-off-on: Carlingtech 2M1-SP1-T1-B1-M1RE 2. on-on: E-Switch 100SP1T6B11M1REH If substituting - gold signal switches, not silver load switches. Cables use: * Molex 0022013037 housing * Molex 0008550102 contact pins Wire: * Alpha Wire AZ221934 family * TE Connectivity 55A0111-22 family If Substituting - ETFE jacket, 22AWG, 19/34+ fine strand, tinned"
- note added: "Light Override Switches"
- note added: "Light Switches ESD Protection"
- moved on the sheet: C64, C65, FID1, FID2, FID3, H1, H2, H3, H4, R24, R52, R53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

Commit message: Progressing on new N2K Transceiver PCB layout
Signed-off-by: digimer <digital.mermaid@gmail.com>
Parts:
- removed C64: 0.1uF, mr-stuff:Kyocera AVX 0805, symbol mr-parts:Kyocera 08051C104K4Z2A
- removed R10, R11, R12, R13, R17, R18, R2, R24, R8, R9: 10kR, mr-stuff:Stackpole_RNCP1206, symbol Device:R
- removed R52: 475R, mr-stuff:Stackpole RNCP0805, symbol mr-parts:Stackpole RNCP0805FTD475R
- removed SW3: SW_MEC_5G, mr-stuff:SW_TS03-66-50-BK-160-LCR-D-67, symbol Switch:SW_MEC_5G
- added C31: 0.1uF, mr-stuff:Kyocera AVX 0805, symbol mr-parts:Kyocera 08051C104K4Z2A
- added HDR7: 0022112032, mr-stuff:Molex 0022112032, symbol mr-parts:Molex 0022112032
- added R10, R11, R12, R13, R17, R18, R2, R8, R9: 10kR, mr-stuff:Stackpole RNCP0805, symbol mr-parts:Stackpole RNCP0805FTD10K0
- added R55: 475R, mr-stuff:Stackpole RNCP0805, symbol mr-parts:Stackpole RNCP0805FTD475R
- added R57: 4.7kR, mr-stuff:Stackpole RMCA0805, symbol mr-parts:Stackpole RMCA0805FT4K70-HP
- added TVS9: TPD2E2U06QDBZRQ1, mr-stuff:TI TPD2E2U06, symbol mr-parts:TVS TPD2E2U06QDBZRQ1
- C1, C12, C18, C4: value 0.1uF -> C; footprint mr-stuff:Kyocera AVX 0805 -> (none); Part Kyocera 08051C104K4Z2A -> (none)
- C10, C2, C3: value 10uF -> C; footprint mr-stuff:TDK CGA5 -> (none); Part TDK CGA5L1X7R1H106K160AE -> (none)
- C11, C14, C9: value 1uF -> C; footprint mr-stuff:Kyocera AVX 0805 -> (none); Part Kyocera 08051C105K4Z2A -> (none)
- C15: renamed from C16; value 0.1uF -> C; footprint mr-stuff:Kyocera AVX 0805 -> (none); Part Kyocera 08051C104K4Z2A -> (none)
- C16: renamed from C17; value 0.1uF -> C; footprint mr-stuff:Kyocera AVX 0805 -> (none); Part Kyocera 08051C104K4Z2A -> (none)
- C17: renamed from C19; value 0.1uF -> C; footprint mr-stuff:Kyocera AVX 0805 -> (none); Part Kyocera 08051C104K4Z2A -> (none)
- C7, C8: value 22uF -> C; footprint mr-stuff:Murata GCJ32ER71C -> (none); Part Murata GCJ32ER71C226KE01L -> (none)
- CMC1: value ACT12101012PTL00 -> ACT1210-101-2P-TL00
- FID1, FID2, FID3: footprint Fiducial:Fiducial_1mm_Mask2mm -> (none)
- H1, H2, H3, H4: value MountingHole_Pad -> MountingHole; footprint MountingHole:MountingHole_4.3mm_M4 -> (none)
- J1: value JTAG -> Conn_01x05_Pin; footprint Connector_PinHeader_2.54mm:PinHeader_1x05_P2.54mm_Vertical -> (none)
- R1: footprint mr-stuff:Stackpole_RNCP1206 -> mr-stuff:Stackpole RNCP0805; symbol Device:R -> mr-parts:Stackpole RNCP0805FTD10K0; Part Stackpole RNCP1206FTD10K0 -> Stackpole RNCP0805FTD10K0
- R14: value 15kR -> R; footprint mr-stuff:Stackpole_RNCP1206 -> (none); Part Stackpole RNCP1206FTD15K0 -> (none)
- R15, R16: value 5.11kR -> R; footprint mr-stuff:Stackpole_RNCP1206 -> (none); Part Stackpole RNCP1206FTD5K11 -> (none)
- R3, R4, R7: value 0R -> RCA08050000ZSEASR; Alternate Murata LQW21FT1R5M0HL -> (none); Note Placeholder if bench testing shows an inductor is needed fo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 -> (none)
- R5: value 470kR -> R; footprint mr-stuff:Wurth WRIS-RSKS -> (none); Part Wurth 560112120009 -> (none)
- R6: value 100kR -> R; footprint mr-stuff:Stackpole RMCA0805 -> (none); Part Stackpole RMCA0805FT100K-HP -> (none)
- ROM1, ROM2: value M24C64 -> STM_M24C64-RMN6P
- SD1: value VS-30MQ040HM3/5AT -> VS-30MQ040-M3_5AT
- SW1, SW2: footprint mr-stuff:SW_TS03-66-50-BK-160-LCR-D-67 -> (none); Part Same Sky TS03-66-50-BK-160-LCR-D-67 -> (none)
- SW3: renamed from SW4; footprint mr-stuff:SW_TS03-66-50-BK-160-LCR-D-67 -> (none); Part Same Sky TS03-66-50-BK-160-LCR-D-67 -> (none)
- TP1: value Comms TP -> Conn_01x10_Pin; footprint Connector_PinHeader_2.54mm:PinHeader_1x10_P2.54mm_Vertical -> (none)
- U1: renamed from MCU1; value ESP32-S3-WROOM-1-N16R2 -> ESP32-S3-WROOM-1; footprint mr-stuff:ESP32-S3-WROOM-1 -> RF_Module:ESP32-S3-WROOM-1; Part Espressif ESP32-S3-WROOM-1-N16R2 -> (none)
- renumbered C65 to C20, C27 to C21, C28 to C22, C29 to C23, C30 to C24, C31 to C25, C32 to C26, C33 to C27, C34 to C28, C35 to C29, C36 to C30, R49 to R29, R51 to R30, R50 to R31, R55 to R32, R56 to R33, R58 to R34, R57 to R35, R59 to R36, R60 to R37, R62 to R38, R61 to R39, R63 to R40, R64 to R41, R66 to R42, R65 to R43, R67 to R44, R68 to R45, R70 to R46, R69 to R47, R71 to R48, R73 to R49, R72 to R50, TVS32 to TVS4, TVS33 to TVS5, TVS34 to TVS6, TVS35 to TVS7, TVS36 to TVS8
Connections:
- net +3.3V: now also R1.1, R17.1, R18.1, R57.2, R8.1, R9.2; no longer R1.2
- net CAN_STANDBY: now also R2.1
- net CAN_TX_LOCAL: now also R1.2; no longer R1.1
- net GND: now also C31.2, HDR7.2 (Pin_2), R10.1, R11.1, R12.1, R2.2, TVS9.3 (GND)
- net N2K_TX_LED: now also U1.11 (IO18); no longer U1.6 (IO6)
- net POWER_LED: now also U1.6 (IO6); no longer U1.22 (IO14)
- net ROM1_WP: now also R17.2
- net ROM2_WP: now also R18.2
- net SRV_UP_LED: now also U1.8 (IO15); no longer U1.9 (IO16)
- net VBUS: now also R13.2
- net VBUS_MCU: now also U1.22 (IO14), R13.1; no longer U1.7 (IO7)
- net WIFI_RX_LED: now also U1.10 (IO17); no longer U1.11 (IO18)
- net WIFI_TX_LED: now also U1.9 (IO16); no longer U1.10 (IO17)
- net WIFI_UP_LED: now also U1.7 (IO7); no longer U1.8 (IO15)
- net at C13.2, SW2.3 (B), SW2.4 (B)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: now also R9.1
- net at U1.15 (IO3): now also R12.2
- net at C14.1, SW1.3 (B), SW1.4 (B)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: now also R8.2
- net at U1.39 (IO1): now also R10.2
- net at U1.38 (IO2): now also R11.2
- net LED_ENABLE renamed LED_ENABLE_IN
- net LED_ENABLE_IN: now also C31.1, R55.2, R57.1
- new net LED_ENABLE_PLUG: HDR7.1 (Pin_1), R55.1, TVS9.1 (IO1)
- no-connect marks 19 -> 21
Other:
- note added: "Config Switch"
- note added: "Intended Switches; 1. on-off-on: Carlingtech 2M1-SP1-T1-B1-M1RE 2. on-on: E-Switch 100SP1T6B11M1REH 3. on-(on): E-Switch 100SP2T6B11M1RE If substituting - gold signal switches, not silver load switches. Cables use: * Molex 0022013037 housing * Molex 0008550102 contact pins Wire: * Alpha Wire AZ221934 family * TE Connectivity 55A0111-22 family If Substituting - ETFE jacket, 22AWG, 19/34+ fine stra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"
- note removed: "Control Switches"
- note removed: "Intended Switches; 1. on-off-on: Carlingtech 2M1-SP1-T1-B1-M1RE 2. on-on: E-Switch 100SP1T6B11M1REH If substituting - gold signal switches, not silver load switches. Cables use: * Molex 0022013037 housing * Molex 0008550102 contact pins Wire: * Alpha Wire AZ221934 family * TE Connectivity 55A0111-22 family If Substituting - ETFE jacket, 22AWG, 19/34+ fine strand, tinned"
- note removed: "LEDs"
- note removed: "Replace R3 with a Murate LQW21FT1R5M0HL if bench testing shows an inductor is needed for VHF."
- moved on the sheet: C20, C21, C22, C23, C24, C25, C26, C27, C28, C29, C30, R1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

Commit message: Finished new PCB layout
Signed-off-by: digimer <digital.mermaid@gmail.com>
Parts:
- removed C1, C10, C11, C12, C14, C15, C16, C17, C18, C2, C3, C4, C7, C8, C9: C, symbol Device:C
- removed R14, R15, R16, R5, R6: R, symbol Device:R
- removed SW1, SW2, SW3: SW_MEC_5G, symbol Switch:SW_MEC_5G
- removed TP1: Conn_01x10_Pin, symbol Connector:Conn_01x10_Pin
- added C1, C12, C15, C16, C17, C18, C4: 0.1uF, mr-stuff:Kyocera AVX 0805, symbol mr-parts:Kyocera 08051C104K4Z2A
- added C10, C2, C3: 10uF, mr-stuff:TDK CGA5, symbol mr-parts:TDK CGA5L1X7R1H106K160AE
- added C11, C14, C9: 1uF, mr-stuff:Kyocera AVX 0805, symbol mr-parts:Kyocera 08051C105K4Z2A
- added C7, C8: 22uF, mr-stuff:Murata GCJ32ER71C, symbol mr-parts:Murata GCJ32ER71C226KE01L
- added R14: 15kR, mr-stuff:Stackpole RNCP0805, symbol mr-parts:Stackpole RNCP0805FTD15K0
- added R15, R16: 5.11kR, mr-stuff:Stackpole RNCP0805, symbol mr-parts:Stackpole RNCP0805FTD5K11
- added R5: 470kR, mr-stuff:Wurth WRIS-RSKS, symbol mr-parts:Wurth 560112120009
- added R6: 100kR, mr-stuff:Stackpole RMCA0805, symbol mr-parts:Stackpole RMCA0805FT100K-HP
- added SW1, SW2, SW3: TS03-66-50-BK-160-LCR-D-67, mr-stuff:Same Sky TS03-66, symbol mr-parts:Same Sky TS03-66-50-BK-160-LCR-D-67
- added TP1: Power/UART Test Point, Connector_PinHeader_2.54mm:PinHeader_1x04_P2.54mm_Vertical, symbol Connector:Conn_01x04_Pin
- added TP2: CAN Test Point, Connector_PinHeader_2.54mm:PinHeader_1x04_P2.54mm_Vertical, symbol Connector:Conn_01x04_Pin
- added TP3: I2C Test Point, Connector_PinHeader_2.54mm:PinHeader_1x02_P2.54mm_Vertical, symbol Connector:Conn_01x02_Pin
- FID1, FID2, FID3: footprint (none) -> Fiducial:Fiducial_1mm_Mask2mm
- H1, H2, H3, H4: footprint (none) -> MountingHole:MountingHole_4.3mm_M4
- JTAG1: renamed from J1; footprint (none) -> Connector_PinHeader_2.54mm:PinHeader_1x05_P2.54mm_Vertical; now left out of the parts list
- MCU1: renamed from U1; value ESP32-S3-WROOM-1 -> ESP32-S3-WROOM-1-N16R2; Part (none) -> Espressif ESP32-S3-WROOM-1-N16R2
- R3, R4, R7: value RCA08050000ZSEASR -> 0R
- ROM1, ROM2: value STM_M24C64-RMN6P -> M24C64
- SD1: value VS-30MQ040-M3_5AT -> VS-30MQ040HM3/5AT; Part Vishay VS-30MQ040-M3_5AT -> Vishay VS-30MQ040HM3/5AT
Connections:
- net +3.3V: now also C1.1, C10.1, C11.1, C12.1, C15.1, C16.1, C17.1, C18.1, C7.1, C8.1, TP1.1 (Pin_1)
- net ANCHOR_OFF_IN: now also IOX1.19 (P1_6); no longer IOX1.5 (P0_1)
- net ANCHOR_ON_IN: now also IOX1.20 (P1_7); no longer IOX1.4 (P0_0)
- net BEACON_ON_IN: now also IOX1.11 (P0_7); no longer IOX1.13 (P1_0)
- net CAN_HIGH: now also TP2.1 (Pin_1)
- net CAN_LOW: now also TP2.2 (Pin_2)
- net CAN_RX_LOCAL: now also TP2.4 (Pin_4)
- net CAN_TX_LOCAL: now also TP2.3 (Pin_3)
- net DECK_OFF_IN: now also IOX1.13 (P1_0); no longer IOX1.11 (P0_7)
- net DECK_ON_IN: now also IOX1.14 (P1_1); no longer IOX1.10 (P0_6)
- net GND: now also C1.2, C10.2, C11.2, C12.2, C14.2, C15.2, C16.2, C17.2, C18.2, C2.2, C3.2, C4.2, C7.2, C8.2, C9.1, R14.2, R15.1, R16.2, R6.1, SW1.1 (A), SW1.2 (A), SW2.1 (A), SW2.2 (A), SW3.3 (B), SW3.4 (B), TP1.2 (Pin_2)
- net I2C_SCL: now also TP3.1 (Pin_1)
- net I2C_SDA: now also TP3.2 (Pin_2)
- net LOCATE_ON_IN: now also IOX1.10 (P0_6); no longer IOX1.14 (P1_1)
- net RXD0: now also TP1.4 (Pin_4)
- net STEAMING_OFF_IN: now also IOX1.15 (P1_2); no longer IOX1.9 (P0_5)
- net STEAMING_ON_IN: now also IOX1.16 (P1_3); no longer IOX1.8 (P0_4)
- net TRICOLOUR_OFF_IN: now also IOX1.17 (P1_4); no longer IOX1.7 (P0_3)
- net TRICOLOUR_ON_IN: now also IOX1.18 (P1_5); no longer IOX1.6 (P0_2)
- net TXD0: now also TP1.3 (Pin_3)
- net VBUS_MCU: now also R14.1
- net V_RAW: now also R5.1
- net at C20.2, R53.2, R54.2: now also SW3.1 (A), SW3.2 (A)
- net at C13.2, MCU1.27 (IO0), R9.1: now also SW2.3 (B), SW2.4 (B)
- net at C5.1, R7.1, VR1.3 (VIN): now also C2.1, C3.1, C4.1
- net at MCU1.3 (EN), R8.2: now also C14.1, SW1.3 (B), SW1.4 (B)
- net at USBRV1.B5 (CC2): now also R16.1
- net at VR1.2 (EN): now also R5.2, R6.2
- net at USBRV1.A5 (CC1): now also R15.2
- net at VR1.8 (VCC): now also C9.2
Other:
- note added: "Test Points"
- note removed: "Test Point"
